File: schematics/board/SINS.sch (EAGLE design)
At the start: 48 parts

Commit message: Папка с платами
Parts:
- removed BSK2, BSK2A: (no value), pinheadCS:PINHD-1X8
- removed BSK3: (no value), pinheadCS:PINHD-1X12
- removed BSK4: (no value), pinheadCS:PINHD-1X14
- removed C1, C12, C33, C5: 0,1µ, rcl:C-USC0603
- removed C14: 2,2µ, rcl:C-USC0603
- removed C15, C6: 22µ, rcl:C-USC1206
- removed C16, C17: 47µ, rcl:C-EUC1210
- removed C3: 10µ, rcl:C-EUC1206
- removed C4: 1nF, rcl:C-USC0603
- removed JTAG: (no value), pinheadCS:PINHD-1X6
- removed LED-B#2, LED1: (no value), led:LEDCHIPLED_0603
- removed R10, R11, R6: 5k1, resistor:R-US_R0603
- removed R12: 73,2k, resistor:R-US_R0603
- removed R13: 45,3k, resistor:R-US_R0603
- removed R18, R21, R22, R23, R24: 3k3, resistor:R-US_R0603
- removed R2, R27: 2k, resistor:R-US_R0603
- removed R29, R8, R9: 10k, resistor:R-US_R0603
- removed R5: 12k, resistor:R-US_R0603
- removed RADIO: RADIO, CanCubeSat:RADIO
- removed SD: SD, CanCubeSat:SD
- removed U$10: LTC3633, CanCubeSat:LTC3633
- removed U$11: 1µH, CanCubeSat:B82498F
- removed U$12: B82498F, CanCubeSat:B82498F
- removed U$13: ESP32WROOM, CanCubeSat:ESP32WROOM
- removed U$18, U$19, U$20: 74HC595, CanCubeSat:74HC595
- removed U$5: DS18B20Z, CanCubeSat:DS18B20Z
- removed U$6: USB-C, CanCubeSat:USB-C
- removed U$7: EM_HEAT, CanCubeSat:EM_HEAT
- removed U$8: L293DD, CanCubeSat:L293DD
- added BT1: 6.8MM_COIN_CELL, SparkFun-Batteries:BATTERY-6.8MM_SMD
- added C10, C11: 10pF, rcl:C-EUC0603
- added C13, C9: 2,2µ, rcl:C-USC0603
- added C18, C2, C20, C53, C54, C55: 100nF, rcl:C-EUC0603
- added C19: 10µ, rcl:C-USC1206
- added C7, C8: 27pF, rcl:C-EUC0603
- added D1: BB141, diode:BB141
- added GPS: GPSNEO6M, CanCubeSat:GPSNEO6M
- added LED2, LED3: (no value), led:LEDCHIPLED_0603
- added MAG: (no value), pinheadCS:PINHD-1X4
- added Q1: 8MHz, 9C-8.000MEEJ-T:9C-8.000MEEJ-T
- added Q2: 32,768KHz, CanCubeSat:C005R
- added R1, R14, R3, R7: 10k, resistor:R-US_R0603
- added R15, R16: 2k, resistor:R-US_R0603
- added R17: 1M, resistor:R-US_R0603
- added R25, R26: 5k1, resistor:R-US_R0603
- added R4: 620R, resistor:R-US_R0603
- added U$4: USB-C, CanCubeSat:USB-C
- added U1: STM32F405RGT6, STM32F405RGT6:STM32F405RGT6
Connections:
- removed net 1W: BSK2.6, BSK2A.6, BSK3.8, BSK4.14, U$13.IO21, U$5.DQ
- removed net AUX: RADIO.AUX, U$13.SVP
- removed net B1_KEM+: U$18.Q2, U$8.IN1
- removed net B1_KEM-: U$18.Q3, U$8.IN2
- removed net B1_KHEAT: U$18.Q1, U$8.IN4
- removed net B2A_KEM+: BSK2A.3, U$19.Q2
- removed net B2A_KEM-: BSK2A.2, U$19.Q3
- removed net B2A_KHEAT: BSK2A.4, U$19.Q1
- removed net B2A_KVCC: BSK2A.5, U$19.Q0
- removed net B2_KEM+: BSK2.3, U$19.Q6
- removed net B2_KEM-: BSK2.2, U$19.Q7
- removed net B2_KHEAT: BSK2.4, U$19.Q5
- removed net B2_KVCC: BSK2.5, U$19.Q4
- removed net B3_KEM+: BSK3.5, U$20.Q6
- removed net B3_KEM-: BSK3.4, U$20.Q7
- removed net B3_KHEAT: BSK3.6, U$20.Q5
- removed net B3_KVCC: BSK3.7, U$20.Q4
- removed net B4_KEM+: BSK4.11, U$18.Q6
- removed net B4_KEM-: BSK4.10, U$18.Q7
- removed net B4_KHEAT: BSK4.12, U$18.Q5
- removed net B4_KVCC: BSK4.13, U$18.Q4
- removed net B5_KEM+: BSK3.2, U$20.Q2
- removed net B5_KEM-: BSK3.1, U$20.Q3
- removed net B5_KHEAT: BSK3.11, U$20.Q1
- removed net B5_KVCC: BSK3.12, U$20.Q0
- removed net BUS+: BSK2.8, BSK2A.8, BSK3.10, BSK4.3, C16.1, C17.1, U$10.RUN1, U$10.RUN2, U$10.VIN1, U$10.VIN2, U$6.3V3/BUS
- removed net DAT0: JP1.2, R23.2, SD.DAT0, U$13.IO2
- removed net DAT1: R24.2, SD.DAT1, U$13.IO4
- removed net DS: U$13.IO25, U$18.DS
- removed net EN: C4.1, R5.1, U$13.EN, U$6.NRST/EN
- removed net I2CINT: BSK4.5, U$13.IO18
- removed net IO0-E: R6.1, U$13.IO0, U$6.NC/GPIO
- removed net IO1: R2.1, U$13.IO5
- removed net M1: R29.1, RADIO.M1, U$13.IO34, U$6.NC/M1
- removed net MTCK: JTAG.5, R21.2, SD.DAT3, U$13.IO13
- removed net MTDI: JTAG.6, R18.2, SD.DAT2, U$13.IO12
- removed net MTDO: JTAG.3, R22.2, SD.CMD, U$13.IO15
- removed net MTMS: JTAG.4, SD.CLK, U$13.IO14
- removed net N$17: U$18.Q7S, U$19.DS
- removed net N$18: U$19.Q7S, U$20.DS
- removed net N$24: C14.2, U$10.INTVCC, U$10.ITH1, U$10.ITH2, U$10.MODE, U$10.PHMODE, U$10.RT, U$10.V2P5
- removed net N$25: R13.1, R8.1, U$10.VFB1
- removed net N$28: C5.1, U$10.SW1, U$11.1
- removed net N$3: LED-B#2.A, U$7.5V, U$8.OUT4
- removed net N$31: C5.2, U$10.BOOST1
- removed net N$32: C1.1, U$10.BOOST2
- removed net N$33: C1.2, U$10.SW2, U$12.1
- removed net N$39: R12.1, R9.1, U$10.VFB2
- removed net N$4: LED1.C, R2.2
- removed net N$51: LED-B#2.C, R27.1
- removed net PL_KVCC: BSK4.8, U$13.IO33
- removed net RX-E: U$13.RXD0, U$6.SWD/RXD
- removed net RX-R: RADIO.TXD, U$13.IO35, U$6.RX0
- removed net SCLTM: BSK4.7, R10.2, U$13.IO16
- removed net SDATM: BSK4.6, R11.2, U$13.IO17
- removed net SHCP: U$13.IO27, U$18.SHCP, U$19.SHCP, U$20.SHCP
- removed net STCP: U$13.IO26, U$18.STCP, U$19.STCP, U$20.STCP
- removed net TIME: BSK4.4, U$13.IO19
- removed net TX-E: U$13.TXD0, U$6.SWC/TXD
- removed net TX-R: RADIO.RXD, U$13.IO32, U$6.TX0
- new net N$1: BT1.+, R4.1
- new net N$15: C8.1, Q1.1, R17.1, U1.PH1/OSC_OUT
- new net N$2: D1.C, R4.2, U1.VBAT
- new net N$30: C7.1, Q1.2, R17.2, U1.PH0/OSC_IN
- new net N$34: C10.1, Q2.2, U1.PC14/OSC32_IN
- new net N$35: C11.1, Q2.1, U1.PC15/OSC32_OUT
- new net N$37: LED2.C, R15.2
- new net N$38: R15.1, U1.PC12
- new net N$40: LED3.C, R16.2
- new net N$41: GPS.RX, U1.PA2/USART2_TX
- new net N$42: GPS.TX, U1.PA3/USART2_RX
- new net N$5: JP1.2, R14.1, U1.PB9
- new net N$6: U1.PB6, U1.PD2
- new net N$7: C9.2, U1.VCAP_1
- new net N$8: C13.2, U1.VCAP_2
- new net NRST: R7.1, U$4.NRST/EN, U1.NRST
- new net RX-S: U$4.RX0, U1.PC10
- new net SCL: MAG.3, R25.2, U1.PB10
- new net SDA: MAG.4, R26.2, U1.PB11
- new net SWC: R3.1, U$4.SWC/TXD, U1.PA14/JTCK-SWCLK
- new net SWD: R1.1, U$4.SWD/RXD, U1.PA13/JMS-SWDIO
- new net TIME-G: GPS.PPS, U1.PA0/WKUP, U1.PA7/SPI1_MOSI, U1.PB7
- new net TX-S: U$4.TX0, U1.PC11
- net 5V: now also GPS.UCC; no longer BSK2.7, BSK2A.7, BSK3.9, BSK4.2, C15.1, R12.2, RADIO.VCC, U$10.VON2, U$12.2, U$5.VDD, U$8.EN1, U$8.EN2, U$8.VS, U$8.VSS
- net GND: now also BT1.-, C10.2, C11.2, C13.1, C18.1, C19.1, C2.2, C20.1, C53.1, C54.1, C55.1, C7.2, C8.2, C9.1, GPS.GND, MAG.1, R14.2, R16.1, U$4.GND, U1.BOOT0, U1.PB2/BOOT1, U1.VSS, U1.VSSA; no longer BSK2.1, BSK2A.1, BSK3.3, BSK4.9, C12.1, C14.1, C15.2, C16.2, C17.2, C3.2, C33.2, C4.2, C6.2, JP1.1, JTAG.1, R27.2, R29.2, R8.2, R9.2, RADIO.GND, RADIO.M0, SD.VSS, U$10.HEAT, U$10.SGND, U$13.GND, U$13.HEAT, U$18.GND, U$18.OE, U$19.GND, U$19.OE, U$20.GND, U$20.OE, U$5.GND, U$5.HEAT, U$6.GND, U$7.GND, U$8.GND, U$8.HEAT
- net RX-ES: now also U1.PA9; no longer U$13.IO22
- net TIME-ES: now also U1.PA6/SPI1_MISO; no longer U$13.SVN
- net TX-ES: now also U1.PA10; no longer U$13.IO23
- net VDD: now also C18.2, C19.2, C2.1, C20.2, C53.2, C54.2, C55.2, D1.A, JP1.1, LED2.A, LED3.A, MAG.2, R1.2, R25.1, R26.1, R3.2, R7.2, U$4.3V3/BUS, U1.VDD, U1.VDDA; no longer BSK4.1, C12.2, C3.1, C33.1, C6.1, JTAG.2, LED1.A, R10.1, R11.1, R13.2, R18.1, R21.1, R22.1, R23.1, R24.1, R5.2, R6.2, SD.VDD, U$10.VON1, U$11.2, U$13.3V3, U$18.MR, U$18.VCC, U$19.MR, U$19.VCC, U$20.MR, U$20.VCC, U$6.NC/3V3
Other:
- note removed: "1.5µH"
- note removed: "1µH"
- note removed: "HEAT"
- moved on the sheet: JP1
