File: schematics/board/ARKnew.brd (EAGLE design)
At the start: 89 x 89 mm, 211 parts, among them IC2 STM32F103C8T, Q5 8MHz

Commit message: Папка с платами
Routing:
- net NRST: track 53.1 -> 52.0 mm
- net VDD: track 314.5 -> 315.4 mm, vias 21 -> 20
Changed lines of the file:
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@@
 <drawing>
 <settings>
-<setting alwaysvectorfont="yes"/>
+<setting alwaysvectorfont="no"/>
 <setting verticaltext="up"/>
 </settings>
@@
 <layer number="14" name="Route14" color="22" fill="1" visible="no" active="no"/>
 <layer number="15" name="Route15" color="23" fill="1" visible="no" active="no"/>
-<layer number="16" name="Bottom" color="1" fill="1" visible="no" active="yes"/>
+<layer number="16" name="Bottom" color="1" fill="1" visible="yes" active="yes"/>
 <layer number="17" name="Pads" color="2" fill="1" visible="yes" active="yes"/>
 <layer number="18" name="Vias" color="2" fill="1" visible="yes" active="yes"/>
@@
 <layer number="54" name="bGND_GNDA" color="1" fill="9" visible="no" active="no"/>
 <layer number="56" name="wert" color="7" fill="1" visible="no" active="no"/>
+<layer number="57" name="tCAD" color="7" fill="1" visible="no" active="no"/>
+<layer number="59" name="tCarbon" color="7" fill="1" visible="no" active="no"/>
+<layer number="60" name="bCarbon" color="7" fill="1" visible="no" active="no"/>
 <layer number="88" name="SimResults" color="9" fill="1" visible="no" active="no"/>
 <layer number="89" name="SimProbes" color="9" fill="1" visible="no" active="no"/>
@@
 <layer number="112" name="tSilk" color="7" fill="1" visible="no" active="no"/>
 <layer number="113" name="IDFDebug" color="7" fill="1" visible="no" active="yes"/>
+<layer number="114" name="Badge_Outline" color="7" fill="1" visible="no" active="no"/>
+<layer number="115" name="ReferenceISLANDS" color="7" fill="1" visible="no" active="no"/>
 <layer number="116" name="Patch_BOT" color="9" fill="4" visible="no" active="no"/>
 <layer number="118" name="Rect_Pads" color="7" fill="1" visible="no" active="no"/>
@@
 <layer number="127" name="_tValues" color="7" fill="1" visible="no" active="no"/>
 <layer number="128" name="_bValues" color="7" fill="1" visible="no" active="no"/>
+<layer number="129" name="Mask" color="7" fill="1" visible="no" active="no"/>
 <layer number="131" name="tAdjust" color="7" fill="1" visible="no" active="no"/>
 <layer number="132" name="bAdjust" color="7" fill="1" visible="no" active="no"/>
 <layer number="144" name="DrillLegend" color="7" fill="1" visible="no" active="no"/>
+<layer number="150" name="Notes" color="7" fill="1" visible="no" active="no"/>
 <layer number="151" name="HeatSink" color="14" fill="1" visible="no" active="no"/>
 <layer number="152" name="_bDocu" color="7" fill="1" visible="no" active="no"/>
+<layer number="153" name="FabDoc1" color="7" fill="1" visible="no" active="no"/>
+<layer number="154" name="FabDoc2" color="7" fill="1" visible="no" active="no"/>
+<layer number="155" name="FabDoc3" color="7" fill="1" visible="no" active="no"/>
 <layer number="199" name="Contour" color="7" fill="1" visible="no" active="no"/>
 <layer number="200" name="200bmp" color="1" fill="10" visible="no" active="no"/>
@@
 <layer number="227" name="227bmp" color="7" fill="1" visible="no" active="yes"/>
 <layer number="228" name="228bmp" color="7" fill="1" visible="no" active="yes"/>
+<layer number="229" name="229bmp" color="7" fill="1" visible="no" active="no"/>
 <layer number="230" name="230bmp" color="7" fill="1" visible="no" active="yes"/>
+<layer number="231" name="231bmp" color="7" fill="1" visible="no" active="no"/>
+<layer number="232" name="Eagle3D_PG2" color="7" fill="1" visible="no" active="no"/>
+<layer number="233" name="Eagle3D_PG3" color="7" fill="1" visible="no" active="no"/>
 <layer number="248" name="Housing" color="7" fill="1" visible="no" active="no"/>
 <layer number="249" name="Edge" color="7" fill="1" visible="no" active="no"/>
@@
 <layer number="251" name="SMDround" color="7" fill="1" visible="no" active="yes"/>
 <layer number="254" name="OrgLBR" color="13" fill="1" visible="no" active="no"/>
+<layer number="255" name="routoute" color="7" fill="1" visible="no" active="no"/>
 </layers>
 <board>
@@
 <contactref element="IC2" pad="36"/>
 <wire x1="49.155" y1="16.32" x2="45.885" y2="13.05" width="0.3" layer="16"/>
-<wire x1="49.155" y1="16.32" x2="54.495" y2="16.32" width="0.3" layer="16"/>
+<wire x1="49.155" y1="16.32" x2="52.5" y2="16.32" width="0.3" layer="16"/>
+<wire x1="52.5" y1="16.32" x2="54.495" y2="16.32" width="0.3" layer="16"/>
 <wire x1="43.425" y1="13.05" x2="45.885" y2="13.05" width="0.3" layer="16"/>
 <wire x1="41.4" y1="15.075" x2="43.425" y2="13.05" width="0.3" layer="16"/>
@@
 <wire x1="32.4" y1="17.55" x2="38.025" y2="17.55" width="0.3" layer="16"/>
 <wire x1="41.175" y1="15.3" x2="41.31" y2="15.2" width="0.3" layer="16"/>
-<via x="54.495" y="16.32" extent="1-16" drill="0.35"/>
 <via x="78.775" y="39.575" extent="1-16" drill="0.35"/>
 <via x="32.4" y="17.55" extent="1-16" drill="0.35"/>
@@
 <wire x1="69.39" y1="32.25" x2="69.39" y2="35.2632" width="0.3" layer="16"/>
 <wire x1="69.39" y1="35.2632" x2="68.2" y2="36.4532" width="0.3" layer="16"/>
-<wire x1="56.75" y1="12.1" x2="56.75" y2="15.995" width="0.3" layer="1"/>
-<wire x1="56.75" y1="15.995" x2="56.5" y2="16.245" width="0.3" layer="1"/>
-<via x="56.5" y="16.245" extent="1-16" drill="0.35"/>
 <wire x1="62.06016875" y1="32.0718" x2="61.88196875" y2="32.25" width="0.3" layer="1"/>
 <wire x1="61.88196875" y1="32.25" x2="61.05" y2="32.25" width="0.3" layer="1"/>
@@
 <wire x1="69.55" y1="36.25" x2="68.4032" y2="36.25" width="0.3" layer="1"/>
 <wire x1="68.4032" y1="36.25" x2="68.2" y2="36.4532" width="0.3" layer="1"/>
-<wire x1="54.495" y1="16.32" x2="54.25" y2="16.075" width="0.3" layer="1"/>
-<wire x1="54.25" y1="16.075" x2="54.25" y2="12.1" width="0.3" layer="1"/>
 <wire x1="80.8438" y1="41.6438" x2="78.775" y2="39.575" width="0.3" layer="16"/>
 <wire x1="27.85" y1="42.3" x2="29.24773125" y2="42.3" width="0.3" layer="1"/>
@@
 <wire x1="30.3225" y1="39.8225" x2="30.3225" y2="39.8275" width="0.3" layer="16"/>
 <wire x1="30.3225" y1="39.8275" x2="27.85" y2="42.3" width="0.3" layer="16"/>
+<wire x1="57.9" y1="12.1" x2="57.9" y2="14.67874375" width="0.5" layer="1"/>
+<wire x1="57.9" y1="14.67874375" x2="57.8718" y2="14.70694375" width="0.5" layer="1"/>
+<wire x1="57.8718" y1="14.70694375" x2="57.8718" y2="15.39305625" width="0.5" layer="1"/>
+<wire x1="57.8718" y1="15.39305625" x2="58.35694375" y2="15.8782" width="0.5" layer="1"/>
+<wire x1="59.0782" y1="15.8782" x2="59.25" y2="16.05" width="0.5" layer="1"/>
+<wire x1="58.35694375" y1="15.8782" x2="59.0782" y2="15.8782" width="0.5" layer="1"/>
+<wire x1="53.1" y1="12.1" x2="53.1" y2="15.72" width="0.5" layer="1"/>
+<wire x1="53.1" y1="15.72" x2="52.5" y2="16.32" width="0.5" layer="1"/>
+<via x="52.5" y="16.32" extent="1-16" drill="0.35"/>
 </signal>
 <signal name="GND">
@@
 <wire x1="73.375" y1="35.3" x2="73.3125" y2="35.3625" width="0.3" layer="1"/>
 <via x="73.375" y="35.3" extent="1-16" drill="0.35"/>
-<wire x1="53.1" y1="12.1" x2="53.1" y2="14.0718" width="0.25" layer="1"/>
-<wire x1="53.1" y1="14.0718" x2="53.0218" y2="14.15" width="0.25" layer="1"/>
-<via x="53.0218" y="14.15" extent="1-16" drill="0.35"/>
-<wire x1="53.0218" y1="14.15" x2="53.8218" y2="14.95" width="0.25" layer="16"/>
-<wire x1="53.8218" y1="14.95" x2="57.805525" y2="14.95" width="0.25" layer="16"/>
 <via x="66.4" y="16.25" extent="1-16" drill="0.35"/>
 <wire x1="57.805525" y1="14.95" x2="58.408725" y2="14.3468" width="0.25" layer="16"/>
@@
 <contactref element="IC2" pad="7"/>
 <wire x1="69.55" y1="35.25" x2="73.2" y2="35.25" width="0.3" layer="1"/>
+<wire x1="54.25" y1="12.1" x2="54.25" y2="14.5218" width="0.3" layer="1"/>
+<wire x1="54.25" y1="14.5218" x2="54.5" y2="14.7718" width="0.3" layer="1"/>
+<via x="54.5" y="14.7718" extent="1-16" drill="0.35"/>
+<wire x1="54.5" y1="14.7718" x2="54.6782" y2="14.95" width="0.3" layer="16"/>
+<wire x1="54.6782" y1="14.95" x2="57.805525" y2="14.95" width="0.3" layer="16"/>
 </signal>
 <signal name="N$5">

Commit message: Плата АБ
Parts:
- removed AB1, AB2, AB3: (no value), pinheadCS:1X08
- removed C1, C10, C11, C12, C17, C18, C19, C2, C20, C21, C22, C23, C24, C25, C26, C27, C28, C3, C4, C5, C6, C7, C8, C9: 0,1µ, rcl:C0603
- removed R1, R17, R33, R41, R49, R9: 2k, resistor:R0603
- removed R10, R11, R18, R19, R2, R3, R34, R35, R42, R43, R50, R51: 330R, resistor:R0603
- removed R12, R13, R14, R15, R20, R21, R22, R23, R36, R37, R38, R39, R4, R44, R45, R46, R47, R5, R52, R53, R54, R55, R6, R7, R88, R89, R90, R91, R92, R93, R94, R95, R96, R97, R98, R99: 100R, resistor:R0603
- removed R16, R24, R40, R48, R56, R8: R05, rcl:R2512
- removed U$1, U$15, U$22, U$24, U$25, U$26, U$27, U$28, U$29, U$30, U$8, U$9: FS8205A-, CanCubeSat:FS8205A-
- removed U$10, U$17, U$3, U$31, U$38, U$45: HY2120, CanCubeSat:HY2120
- removed U$11, U$12, U$18, U$19, U$32, U$33, U$39, U$4, U$40, U$46, U$47, U$5: HY2213, CanCubeSat:HY2213
- removed U$13, U$14, U$20, U$21, U$34, U$35, U$41, U$42, U$48, U$49, U$6, U$7: SI2302CDS, CanCubeSat:SI2302CDS
Connections:
- removed net B-1: AB1.6, C1.2, C2.2, C4.2, R8.2, U$3.6, U$5.3, U$7.2
- removed net B-2: AB1.1, C25.2, C26.2, C28.2, R56.2, U$45.6, U$47.3, U$49.2
- removed net B-3: AB2.6, C5.2, C6.2, C8.2, R16.2, U$10.6, U$12.3, U$14.2
- removed net B-4: AB2.1, C21.2, C22.2, C24.2, R48.2, U$38.6, U$40.3, U$42.2
- removed net B-5: AB3.6, C10.2, C12.2, C9.2, R24.2, U$17.6, U$19.3, U$21.2
- removed net B-6: AB3.1, C17.2, C18.2, C20.2, R40.2, U$31.6, U$33.3, U$35.2
- removed net N$1: C1.1, R2.1, U$3.5
- removed net N$10: R5.1, U$7.3
- removed net N$100: U$46.6, U$48.1
- removed net N$102: U$47.6, U$49.1
- removed net N$104: R49.2, R56.1, U$1.67
- removed net N$107: C26.1, R51.1, U$45.4
- removed net N$108: C28.1, R55.1, U$47.2
- removed net N$110: AB1.2, C27.2, R51.2, R53.2, R55.2, U$46.3, U$48.2
- removed net N$13: R1.2, R8.1, U$26.67
- removed net N$15: C2.1, R3.1, U$3.4
- removed net N$16: C5.1, R10.1, U$10.5
- removed net N$18: R9.1, U$10.3
- removed net N$19: C7.1, R14.1, U$11.2
- removed net N$2: C4.1, R7.1, U$5.2
- removed net N$20: U$11.6, U$13.1
- removed net N$21: R12.1, U$13.3
- removed net N$22: U$12.6, U$14.1
- removed net N$23: R13.1, U$14.3
- removed net N$24: R16.1, R9.2, U$25.67
- removed net N$27: C6.1, R11.1, U$10.4
- removed net N$28: C8.1, R15.1, U$12.2
- removed net N$3: R1.1, U$3.3
- removed net N$30: AB2.7, C7.2, R11.2, R13.2, R15.2, U$11.3, U$13.2
- removed net N$31: R91.2, U$9.5
- removed net N$33: C9.1, R18.1, U$17.5
- removed net N$34: R17.1, U$17.3
- removed net N$35: C11.1, R22.1, U$18.2
- removed net N$36: U$18.6, U$20.1
- removed net N$37: R20.1, U$20.3
- removed net N$38: U$19.6, U$21.1
- removed net N$39: R21.1, U$21.3
- removed net N$4: C3.1, R6.1, U$4.2
- removed net N$40: R17.2, R24.1, U$24.67
- removed net N$43: C10.1, R19.1, U$17.4
- removed net N$44: C12.1, R23.1, U$19.2
- removed net N$45: R90.2, U$9.4
- removed net N$46: AB3.7, C11.2, R19.2, R21.2, R23.2, U$18.3, U$20.2
- removed net N$49: U$15.23, U$22.67
- removed net N$50: U$24.23, U$9.67
- removed net N$53: R88.2, U$22.4
- removed net N$57: R36.1, U$34.3
- removed net N$58: R37.1, U$35.3
- removed net N$59: R44.1, U$41.3
- removed net N$6: U$4.6, U$6.1
- removed net N$61: R89.2, U$22.5
- removed net N$62: U$25.23, U$27.67
- removed net N$63: R93.2, U$27.5
- removed net N$64: R92.2, U$27.4
- removed net N$65: C17.1, R34.1, U$31.5
- removed net N$66: R33.1, U$31.3
- removed net N$67: C19.1, R38.1, U$32.2
- removed net N$68: U$32.6, U$34.1
- removed net N$69: R45.1, U$42.3
- removed net N$7: R4.1, U$6.3
- removed net N$70: U$33.6, U$35.1
- removed net N$71: R52.1, U$48.3
- removed net N$72: R33.2, R40.1, U$15.67
- removed net N$73: U$28.67, U$8.23
- removed net N$74: R97.2, U$28.5
- removed net N$75: C18.1, R35.1, U$31.4
- removed net N$76: C20.1, R39.1, U$33.2
- removed net N$77: R96.2, U$28.4
- removed net N$78: AB3.2, C19.2, R35.2, R37.2, R39.2, U$32.3, U$34.2
- removed net N$79: U$26.23, U$29.67
- removed net N$8: AB1.7, C3.2, R3.2, R5.2, R7.2, U$4.3, U$6.2
- removed net N$80: R95.2, U$29.5
- removed net N$81: C21.1, R42.1, U$38.5
- removed net N$82: R41.1, U$38.3
- removed net N$83: C23.1, R46.1, U$39.2
- removed net N$84: U$39.6, U$41.1
- removed net N$85: R53.1, U$49.3
- removed net N$86: U$40.6, U$42.1
- removed net N$88: R41.2, R48.1, U$8.67
- removed net N$89: R94.2, U$29.4
- removed net N$9: U$5.6, U$7.1
- removed net N$90: U$1.23, U$30.67
- removed net N$91: C22.1, R43.1, U$38.4
- removed net N$92: C24.1, R47.1, U$40.2
- removed net N$93: R99.2, U$30.5
- removed net N$94: AB2.2, C23.2, R43.2, R45.2, R47.2, U$39.3, U$41.2
- removed net N$95: R98.2, U$30.4
- removed net N$97: C25.1, R50.1, U$45.5
- removed net N$98: R49.1, U$45.3
- removed net N$99: C27.1, R54.1, U$46.2
- removed net OC1: U$26.5, U$3.2
- removed net OC2: U$1.5, U$45.2
- removed net OC3: U$10.2, U$25.5
- removed net OC4: U$38.2, U$8.5
- removed net OC5: U$17.2, U$24.5
- removed net OC6: U$15.5, U$31.2
- removed net OD1: U$26.4, U$3.1
- removed net OD2: U$1.4, U$45.1
- removed net OD3: U$10.1, U$25.4
- removed net OD4: U$38.1, U$8.4
- removed net OD5: U$17.1, U$24.4
- removed net OD6: U$15.4, U$31.1
- net 1W: no longer AB1.5, AB2.5, AB3.5
- net BMS+: no longer AB1.8, AB2.8, AB3.8, R10.2, R12.2, R14.2, R18.2, R2.2, R20.2, R22.2, R34.2, R36.2, R38.2, R4.2, R42.2, R44.2, R46.2, R50.2, R52.2, R54.2, R6.2
- net BMS1: no longer R94.1, R95.1
- net BMS2: no longer R98.1, R99.1
- net BMS3: no longer R92.1, R93.1
- net BMS4: no longer R96.1, R97.1
- net BMS5: no longer R90.1, R91.1
- net BMS6: no longer R88.1, R89.1
- net GND: no longer AB1.4, AB2.4, AB3.4, U$22.23, U$27.23, U$28.23, U$29.23, U$30.23, U$9.23
- net VDD: no longer AB1.3, AB2.3, AB3.3
Routing:
- net 1W: track 212.3 -> 146.0 mm
- net GND: track 580.9 -> 520.3 mm
- net VDD: track 315.4 -> 259.4 mm
- net BMS+: track 235.1 -> 204.3 mm
- net B-6: track 30.6 -> 0.00 mm
- net B-2: track 30.5 -> 0.00 mm
- net B-4: track 30.5 -> 0.00 mm
- net B-5: track 30.5 -> 0.00 mm
- net B-3: track 30.4 -> 0.00 mm
- net B-1: track 30.4 -> 0.00 mm
- net N$110: track 24.3 -> 0.00 mm
- net N$94: track 24.3 -> 0.00 mm
- net N$78: track 24.2 -> 0.00 mm
- net N$46: track 24.1 -> 0.00 mm
- net N$8: track 24.1 -> 0.00 mm
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