File: schematics/board/BSK4new.brd (EAGLE design)
At the start: 82 x 100 mm, 34 parts

Commit message: Сделаны платы CROSSnew, SPIDERnew, BSK2
Parts:
- removed DS18B20Z1: DS18B20Z, CanCubeSat:SOIC8+HEAT_S
- removed LED6, LED7: (no value), led:CHIPLED_0603
- removed R12: 2M, resistor:R0603
- removed R13: 1k5, resistor:R0603
- removed R14, R8, R9: 1M, resistor:R0603
- removed R94, R95: 2k26, resistor:R0603
- removed U$10, U$11, U$12, U$9: KCONNECT, CanCubeSat:KCONNECT
- removed U$13, U$8: SI2302CDS, CanCubeSat:SOT23-3
- removed U$14: EM_HEAT, CanCubeSat:EM_HEAT
- removed U$26: FS8205A+, CanCubeSat:FS8205A+
- removed YELLOW: LAP4-BOTTOM, led:P47F-BOTTOM
- added BSK5: (no value), pinheadCS:1X08
- added DS18B20Z: DS18B20Z, CanCubeSat:DS18B20Z
- added JP1, JP2, JP3, JP4, JP5, JP6: (no value), pinheadCS:2X10
- added LAP2: LAP4-BOTTOM, led:P47F-BOTTOM
- added LED1, LED2: (no value), led:CHIPLED_0603
- added R1, R2: 2k26, resistor:R0603
- added R10, R11: 2k, resistor:R0603
- added R18, R20, R3: 1M, resistor:R0603
- added R19: 1k5, resistor:R0603
- added U$17: FS8205A+, CanCubeSat:FS8205A+
- added U$18, U$19, U$20, U$21: KCONNECT, CanCubeSat:KCONNECT
- added U$22: MOCD217M, CanCubeSat:SOIC8
- added U$23, U$25: SI2302CDS, CanCubeSat:SOT23-3
- added U$24: EM_HEAT, CanCubeSat:EM_HEAT
- BKU: device pinheadCS:1X08 -> pinheadCS:1X20
- R4, R7: value 2k -> 2M
- R6: value 2M -> 1M
- U$5: value MOCD217M -> SI2302CDS; device CanCubeSat:SOIC8 -> CanCubeSat:SOT23-3
- moved U$5 211.5 mm to (3.60, -120.5)
- moved R6 207.9 mm to (1.50, -116.6), turned to 0 degrees
- moved R5 201.8 mm to (37.9, -111.7), turned to 0 degrees
- moved R7 182.2 mm to (41.8, -111.7), turned to 0 degrees
- moved R4 136.4 mm to (34.0, -111.7), turned to 0 degrees
- moved BKU 9.00 mm to (41.0, 98.8)
- moved U$2 0.65 mm to (21.1, 69.9)
- moved U$4 0.65 mm to (60.9, 69.9)
- moved U$3 0.65 mm to (69.4, 78.4)
- moved U$1 0.65 mm to (12.6, 78.4)
- renumbered U$15 to U$28, U$16 to U$29, U$6 to U$30, U$7 to U$27
Connections:
- net B2-CMD renamed B1-CMD
- removed net 1: R7.2, U$14.2, U$8.3
- removed net 2: R13.2, U$13.3, U$27.P$1, U$28.P$1, U$29.P$1, U$30.P$1
- removed net B2-KHEAT: BKU.1, R8.1, U$8.1
- removed net B2-KVCC: BKU.2, R94.2, R95.2, U$5.1, U$5.3
- removed net B2-ROZE: BKU.3, R14.1, U$13.1
- removed net N$26: R5.1, R6.2, U$26.5
- removed net N$29: LED7.C, R13.1
- removed net N$31: LED6.C, R7.1
- removed net OC1: R9.2, U$5.6
- removed net OD1: R5.2, U$5.8
- new net 3: R11.2, U$23.3, U$24.2
- new net 3V3: BKU.8, BSK5.3, JP1.9, JP2.9, JP3.9, JP4.9, JP5.9, JP6.9
- new net 4: R19.2, U$25.3, U$27.P$1, U$28.P$1, U$29.P$1, U$30.P$1
- new net B1-KHEAT: BKU.1, R18.1, U$23.1
- new net B1-KVCC: BKU.2, R1.2, R2.2, U$22.1, U$22.3
- new net B1-ROZE: BKU.3, R20.1, U$25.1
- new net BMS1: JP1.1, JP2.1, JP3.1, JP4.5, JP5.3, JP6.3
- new net BMS2: JP1.2, JP2.2, JP3.2, JP4.6, JP5.4, JP6.4
- new net BMS3: JP1.3, JP2.3, JP3.3, JP4.1, JP5.5, JP6.5
- new net BMS4: JP1.4, JP2.4, JP3.4, JP4.2, JP5.6, JP6.6
- new net BMS5: JP1.5, JP2.5, JP3.5, JP4.3, JP5.1, JP6.1
- new net BMS6: JP1.6, JP2.6, JP3.6, JP4.4, JP5.2, JP6.2
- new net INT: JP1.16, JP2.16, JP3.16, JP4.16, JP5.16, JP6.16
- new net N$1: R4.2, R5.1, U$17.5
- new net N$2: LED1.C, R11.1
- new net N$3: LED2.C, R19.1
- new net N$4: DS18B20Z.HEAT, U$17.HEAT
- new net OC2: R3.2, U$22.6
- new net OD2: R5.2, U$22.8
- new net PL1: JP1.17, JP2.17, JP3.17, JP4.17, JP5.17, JP6.17
- new net PL1-GND: U$5.3
- new net PL1-KVCC: BKU.15, R6.1, U$5.1
- new net PL2: JP1.19, JP2.19, JP3.19, JP4.19, JP5.19, JP6.19
- new net PL2-KVCC: BKU.16
- new net PL3: JP1.18, JP2.18, JP3.18, JP4.18, JP5.18, JP6.18
- new net PL3-KVCC: BKU.17
- new net PL4: JP1.20, JP2.20, JP3.20, JP4.20, JP5.20, JP6.20
- new net PL4-KVCC: BKU.18
- new net PL5-KVCC: BKU.19
- new net PL6-KVCC: BKU.20
- new net SCL: BKU.10, BSK5.5, JP1.13, JP2.13, JP3.13, JP4.13, JP5.13, JP6.13
- new net SDA: BKU.12, BSK5.7, JP1.14, JP2.14, JP3.14, JP4.14, JP5.14, JP6.14
- new net TIME: BKU.14, JP1.15, JP2.15, JP3.15, JP4.15, JP5.15, JP6.15
- new net TIME-ES: BKU.13, BSK5.8
- net 1W: now also DS18B20Z.4, JP1.7, JP2.7, JP3.7, JP4.7, JP5.7, JP6.7; no longer DS18B20Z1.4
- net 5V: now also BSK5.2, DS18B20Z.3, JP1.10, JP2.10, JP3.10, JP4.10, JP5.10, JP6.10, LED1.A, R10.1, U$24.1; no longer DS18B20Z1.3, LED6.A, R4.1, U$14.1
- net BUS+: now also JP1.8, JP2.8, JP3.8, JP4.8, JP5.8, JP6.8, LED2.A, R4.1, R7.2; no longer LED7.A, R12.2, R6.1
- net BUS+2: now also U$18.1, U$18.2, U$18.3, U$18.4, U$18.P$1, U$18.P$2; no longer U$9.1, U$9.2, U$9.3, U$9.4, U$9.P$1, U$9.P$2
- net BUS+3: now also U$20.1, U$20.2, U$20.3, U$20.4, U$20.P$1, U$20.P$2; no longer U$11.1, U$11.2, U$11.3, U$11.4, U$11.P$1, U$11.P$2
- net BUS-: now also LAP2.C, U$17.67, U$22.7; no longer U$26.67, U$5.7, YELLOW.C
- net BUS-2: now also U$19.1, U$19.2, U$19.3, U$19.4, U$19.P$1, U$19.P$2; no longer U$10.1, U$10.2, U$10.3, U$10.4, U$10.P$1, U$10.P$2
- net BUS-3: now also U$21.1, U$21.2, U$21.3, U$21.4, U$21.P$1, U$21.P$2; no longer U$12.1, U$12.2, U$12.3, U$12.4, U$12.P$1, U$12.P$2
- net GND: now also BKU.11, BKU.9, BSK5.1, BSK5.4, BSK5.6, DS18B20Z.5, JP1.11, JP1.12, JP2.11, JP2.12, JP3.11, JP3.12, JP4.11, JP4.12, JP5.11, JP5.12, JP6.11, JP6.12, R1.1, R18.2, R2.1, R20.2, R6.2, U$17.23, U$22.2, U$22.4, U$22.5, U$23.2, U$25.2; no longer BKU.8, DS18B20Z1.5, DS18B20Z1.HEAT, R14.2, R8.2, R94.1, R95.1, U$13.2, U$26.23, U$26.HEAT, U$5.4, U$5.5, U$8.2
- net N$27: now also R3.1, R7.1, U$17.4; no longer R12.1, R9.1, U$26.4
- net N$28: now also LAP2.A, R10.2; no longer R4.2, YELLOW.A
Routing:
- net BUS+: track 226.1 -> 0.00 mm, vias 2 -> 0
- net 2: track 160.0 -> 0.00 mm, vias 2 -> 0
- net BUS-: track 117.3 -> 0.00 mm, vias 2 -> 0
- net 5V: track 112.3 -> 0.00 mm, vias 6 -> 0
- net B1-CMD: track 74.1 -> 0.00 mm, vias 2 -> 0
- net B2-ROZE: track 72.6 -> 0.00 mm, vias 2 -> 0
- net B2-KHEAT: track 50.0 -> 0.00 mm, vias 1 -> 0
- net B2-KVCC: track 35.1 -> 0.00 mm
- net 1W: track 30.4 -> 0.00 mm, vias 2 -> 0
- net BUS-1: track 23.4 -> 0.00 mm
- net BUS-2: track 23.4 -> 0.00 mm
- net BUS-3: track 23.3 -> 0.00 mm
- net BUS+1: track 22.1 -> 0.00 mm
- net BUS+2: track 22.1 -> 0.00 mm
- net BUS+3: track 22.0 -> 0.00 mm
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- added copper zone on layer 1, net GND4
Other:
- outline, holes or cut-outs redrawn
- board text added: "BSK1 "Концерн ИТС""
- board text added: "to BSK5"
- board text removed: "BSK2 "Концерн ИТС""
