File: schematics/board/BSK4new.sch (EAGLE design)
At the start: 29 parts

Commit message: Сделаны платы CROSSnew, SPIDERnew, BSK2
Parts:
- removed BSK3: (no value), pinheadCS:PINHD-1X8
- removed LAP1: LAP4-BOTTOM, led:LAP4-BOTTOM
- removed LED6, LED7: (no value), led:LEDCHIPLED_0603
- removed R12: 2M, resistor:R-US_R0603
- removed R13: 1k5, resistor:R-US_R0603
- removed R14, R8, R9: 1M, resistor:R-US_R0603
- removed R94, R95: 2k26, resistor:R-US_R0603
- removed U$10, U$11, U$12, U$9: KCONNECT, CanCubeSat:KCONNECT
- removed U$13, U$8: SI2302CDS, CanCubeSat:SI2302CDS
- removed U$14: EM_HEAT, CanCubeSat:EM_HEAT
- removed U$26: FS8205A+, CanCubeSat:FS8205A+
- added BKU: (no value), pinheadCS:PINHD-1X20
- added BSK5: (no value), pinheadCS:PINHD-1X8
- added CMD: KCONNECTQUAD, CanCubeSat:KCONNECTQUAD
- added JP1, JP2, JP3, JP4, JP5, JP6: (no value), pinheadCS:PINHD-2X10
- added LAP2: LAP4-BOTTOM, led:LAP4-BOTTOM
- added LED1, LED2: (no value), led:LEDCHIPLED_0603
- added R1, R2: 2k26, resistor:R-US_R0603
- added R10, R11: 2k, resistor:R-US_R0603
- added R18, R20, R3: 1M, resistor:R-US_R0603
- added R19: 1k5, resistor:R-US_R0603
- added U$17: FS8205A+, CanCubeSat:FS8205A+
- added U$18, U$19, U$20, U$21: KCONNECT, CanCubeSat:KCONNECT
- added U$22: MOCD217M, CanCubeSat:MOCD217M
- added U$23, U$25: SI2302CDS, CanCubeSat:SI2302CDS
- added U$24: EM_HEAT, CanCubeSat:EM_HEAT
- added U$27, U$28, U$29, U$30: GRAFITGRAFIT3_1, CanCubeSat:GRAFITGRAFIT3_1
- R4, R7: value 2k -> 2M
- R6: value 2M -> 1M
- U$5: value MOCD217M -> SI2302CDS; device CanCubeSat:MOCD217M -> CanCubeSat:SI2302CDS
Connections:
- removed net 1: R7.2, U$14.GND, U$8.D
- removed net 2: R13.2, U$13.D
- removed net B5-KHEAT: R8.1, U$8.G
- removed net B5-KVCC: R94.2, R95.2, U$5.AN1, U$5.AN2
- removed net B5-ROZE: R14.1, U$13.G
- removed net KEM7: BSK3.3
- removed net KEM8: BSK3.2
- removed net KHEAT4: BSK3.4
- removed net KVCC4: BSK3.5
- removed net N$30: R5.1, R6.2, U$26.G2
- removed net N$31: R12.1, R9.1, U$26.G1
- removed net N$32: LAP1.A, R4.2
- removed net N$33: LED6.C, R7.1
- removed net N$34: LED7.C, R13.1
- removed net N$35: DS18B20Z.HEAT, U$26.HEAT
- removed net OC1: R9.2, U$5.COL2
- removed net OD1: R5.2, U$5.COL1
- new net 3: R11.2, U$23.D, U$24.GND
- new net 3V3: BKU.8, BSK5.3, JP1.9, JP2.9, JP3.9, JP4.9, JP5.9, JP6.9
- new net 4: R19.2, U$25.D, U$27.P$1, U$28.P$1, U$29.P$1, U$30.P$1
- new net B1-CMD: BKU.4, CMD.P$1
- new net B1-KHEAT: BKU.1, R18.1, U$23.G
- new net B1-KVCC: BKU.2, R1.2, R2.2, U$22.AN1, U$22.AN2
- new net B1-ROZE: BKU.3, R20.1, U$25.G
- new net BMS1: JP1.1, JP2.1, JP3.1, JP4.5, JP5.3, JP6.3
- new net BMS2: JP1.2, JP2.2, JP3.2, JP4.6, JP5.4, JP6.4
- new net BMS3: JP1.3, JP2.3, JP3.3, JP4.1, JP5.5, JP6.5
- new net BMS4: JP1.4, JP2.4, JP3.4, JP4.2, JP5.6, JP6.6
- new net BMS5: JP1.5, JP2.5, JP3.5, JP4.3, JP5.1, JP6.1
- new net BMS6: JP1.6, JP2.6, JP3.6, JP4.4, JP5.2, JP6.2
- new net INT: JP1.16, JP2.16, JP3.16, JP4.16, JP5.16, JP6.16
- new net N$1: R4.2, R5.1, U$17.G2
- new net N$2: LED1.C, R11.1
- new net N$27: R3.1, R7.1, U$17.G1
- new net N$28: LAP2.A, R10.2
- new net N$3: LED2.C, R19.1
- new net N$4: DS18B20Z.HEAT, U$17.HEAT
- new net OC2: R3.2, U$22.COL2
- new net OD2: R5.2, U$22.COL1
- new net PL1: JP1.17, JP2.17, JP3.17, JP4.17, JP5.17, JP6.17
- new net PL1-GND: U$5.D
- new net PL1-KVCC: BKU.15, R6.1, U$5.G
- new net PL2: JP1.19, JP2.19, JP3.19, JP4.19, JP5.19, JP6.19
- new net PL2-KVCC: BKU.16
- new net PL3: JP1.18, JP2.18, JP3.18, JP4.18, JP5.18, JP6.18
- new net PL3-KVCC: BKU.17
- new net PL4: JP1.20, JP2.20, JP3.20, JP4.20, JP5.20, JP6.20
- new net PL4-KVCC: BKU.18
- new net PL5-KVCC: BKU.19
- new net PL6-KVCC: BKU.20
- new net SCL: BKU.10, BSK5.5, JP1.13, JP2.13, JP3.13, JP4.13, JP5.13, JP6.13
- new net SDA: BKU.12, BSK5.7, JP1.14, JP2.14, JP3.14, JP4.14, JP5.14, JP6.14
- new net TIME: BKU.14, JP1.15, JP2.15, JP3.15, JP4.15, JP5.15, JP6.15
- new net TIME-ES: BKU.13, BSK5.8
- net 1W: now also BKU.5, JP1.7, JP2.7, JP3.7, JP4.7, JP5.7, JP6.7; no longer BSK3.6
- net 5V: now also BKU.7, BSK5.2, JP1.10, JP2.10, JP3.10, JP4.10, JP5.10, JP6.10, LED1.A, R10.1, U$24.5V; no longer BSK3.7, LED6.A, R4.1, U$14.5V
- net BUS+: now also BKU.6, JP1.8, JP2.8, JP3.8, JP4.8, JP5.8, JP6.8, LED2.A, R4.1, R7.2, U$27.P$2, U$28.P$2, U$29.P$2, U$30.P$2; no longer BSK3.8, LED7.A, R12.2, R6.1
- net BUS+2: now also U$18.P$1; no longer U$9.P$1
- net BUS+3: now also U$20.P$1; no longer U$11.P$1
- net BUS-: now also LAP2.C, U$17.S2, U$22.EM1; no longer LAP1.C, U$26.S2, U$5.EM1
- net BUS-2: now also U$19.P$1; no longer U$10.P$1
- net BUS-3: now also U$21.P$1; no longer U$12.P$1
- net GND: now also BKU.11, BKU.9, BSK5.1, BSK5.4, BSK5.6, JP1.11, JP1.12, JP2.11, JP2.12, JP3.11, JP3.12, JP4.11, JP4.12, JP5.11, JP5.12, JP6.11, JP6.12, R1.1, R18.2, R2.1, R20.2, R6.2, U$17.S1, U$22.CAT1, U$22.CAT2, U$22.EM2, U$23.S, U$25.S, U$5.S; no longer BSK3.1, R14.2, R8.2, R94.1, R95.1, U$13.S, U$26.S1, U$5.CAT1, U$5.CAT2, U$5.EM2, U$8.S
Other:
- moved on the sheet: R4, R5, R6, R7, U$1, U$2, U$3, U$4
