File: schematics/board/BMSnew.brd (EAGLE design)
At the start: 78 x 21 mm, 61 parts

Commit message: Плата АБ
Parts:
- removed B+, B-, BC: BATTERY, CanCubeSat:BATTERY
- added B+2, B-2, BC2: BATTERY, CanCubeSat:BATTERY
- moved BC1 39.8 mm to (19.0, 12.0)
- moved B+1 39.5 mm to (9.00, 12.0)
- moved B-1 39.5 mm to (29.5, 12.0)
- moved R17 3.01 mm to (52.3, 19.0)
- moved R16 3.01 mm to (55.8, 19.0)
- moved R18 2.52 mm to (52.3, 16.5)
- moved R15 2.51 mm to (55.8, 16.5)
- moved R56 1.80 mm to (71.4, 12.4)
- moved U$1 1.50 mm to (63.0, 12.4)
- moved R55 1.28 mm to (74.4, 7.80)
- moved R54 1.28 mm to (74.4, 4.10)
- moved R51 1.28 mm to (60.1, 7.80)
- moved R50 1.28 mm to (60.1, 4.10)
- moved C28 1.28 mm to (72.1, 7.80), turned to 90 degrees
- moved R53 1.28 mm to (62.4, 7.80)
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Connections:
- removed net BUS+: AB1.4
- removed net N$98: R49.1, U$45.3
- new net N$13: R1.2, U$3.3
- net B-1: now also B-1.P$1; no longer B-.P$1
- net B-2: now also B-2.P$1; no longer B-1.P$1
- net BC1: now also BC1.P$1; no longer BC.P$1
- net BC2: now also BC2.P$1; no longer BC1.P$1
- net BMS+: now also AB1.4, B+2.P$1; no longer B+.P$1
- net GND: now also R1.1, R49.1
- net N$16: no longer R49.2
- net N$3: no longer R1.2
- net N$5: now also R49.2, U$45.3; no longer R1.1, U$3.3
Routing:
- net BMS+: track 60.4 -> 141.5 mm, vias 1 -> 3
- net 1W: track 22.4 -> 73.7 mm, vias 0 -> 4
- net BMS2: track 0.00 -> 49.9 mm, vias 0 -> 3
- net 3V3: track 23.3 -> 66.6 mm, vias 0 -> 3
- net B-2: track 0.00 -> 34.2 mm, vias 0 -> 1
- net BC2: track 0.00 -> 29.0 mm, vias 0 -> 1
- net OD2: track 0.00 -> 26.4 mm, vias 0 -> 4
- net BMS1: track 36.3 -> 62.1 mm, vias 2 -> 4
- net OC2: track 0.00 -> 24.7 mm, vias 0 -> 2
- net GND: track 19.0 -> 43.7 mm, vias 2 -> 4
- net N$10: track 0.00 -> 17.2 mm, vias 0 -> 2
- net N$107: track 0.00 -> 15.7 mm
- net N$3: track 24.2 -> 10.2 mm
- net N$14: track 0.00 -> 9.74 mm
- net N$97: track 0.00 -> 9.52 mm, vias 0 -> 2
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- added copper zone on layer 1, net BMS+
Other:
- board text added: "1W"
- board text added: "3V3"
- board text added: "BMS+"
- board text added: "BMS1"
- board text added: "BMS2"
- board text added: "GND"

Commit message: Сделал платку BMSnew лучше, но не совсем
Parts:
- R11, R12: value 100R -> 100k
Changed lines of the file:
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@@
 <drawing>
 <settings>
-<setting alwaysvectorfont="no"/>
+<setting alwaysvectorfont="yes"/>
 <setting verticaltext="up"/>
 </settings>
@@
 <attribute name="VALUE" x="22.635" y="3.905" size="1.27" layer="27" rot="R180"/>
 </element>
-<element name="R11" library="resistor" library_urn="urn:adsk.eagle:library:348" package="R0603" package3d_urn="urn:adsk.eagle:package:23555/3" value="100R" x="26" y="2" smashed="yes" rot="R180">
+<element name="R11" library="resistor" library_urn="urn:adsk.eagle:library:348" package="R0603" package3d_urn="urn:adsk.eagle:package:23555/3" value="100k" x="26" y="2" smashed="yes" rot="R180">
 <attribute name="VALUE" x="26.635" y="3.905" size="1.27" layer="27" rot="R180"/>
 </element>
-<element name="R12" library="resistor" library_urn="urn:adsk.eagle:library:348" package="R0603" package3d_urn="urn:adsk.eagle:package:23555/3" value="100R" x="26" y="4.5" smashed="yes">
+<element name="R12" library="resistor" library_urn="urn:adsk.eagle:library:348" package="R0603" package3d_urn="urn:adsk.eagle:package:23555/3" value="100k" x="26" y="4.5" smashed="yes">
 <attribute name="VALUE" x="25.365" y="2.595" size="1.27" layer="27"/>
 </element>

Commit message: платы DC-DC и AB
Parts:
- added R13, R14, R19, R20: 2k26, resistor:R0603
- R17, R18: value 100R -> 100k
- R94, R95, R98, R99: value 2k26 -> 200k
- moved U$1 0.50 mm to (63.0, 12.9)
- moved R94 0.30 mm to (26.8, 10.3)
- moved U$3 0.22 mm to (23.6, 11.6)
Connections:
- removed net N$16: R56.1, U$1.67, U$10.7
- new net N$17: R14.1, R94.2, U$2.1
- new net N$18: R13.1, R95.2, U$2.3
- new net N$19: R19.1, R99.2, U$10.3
- new net NO_GND1: R8.1, R94.1, R95.1, U$2.2, U$2.4, U$2.7, U$26.67
- new net NO_GND2: R56.1, R98.1, R99.1, U$1.67, U$10.2, U$10.4, U$10.7
- net BMS1: now also R13.2, R14.2; no longer R94.2, R95.2, U$2.1, U$2.3
- net BMS2: now also R19.2, R20.2; no longer R98.2, R99.2, U$10.1, U$10.3
- net GND: no longer R94.1, R95.1, R98.1, R99.1, U$10.2, U$10.4, U$2.2, U$2.4
- net N$3: now also R20.1, R98.2, U$10.1; no longer R8.1, U$2.7, U$26.67
Routing:
- net N$19: track 0.00 -> 48.5 mm, vias 0 -> 2
- net NO_GND1: track 0.00 -> 48.4 mm, vias 0 -> 2
- net N$17: track 0.00 -> 48.0 mm, vias 0 -> 4
- net NO_GND2: track 0.00 -> 37.5 mm, vias 0 -> 1
- net N$18: track 0.00 -> 31.6 mm, vias 0 -> 2
- net N$3: track 10.2 -> 40.4 mm, vias 0 -> 2
- net GND: track 43.7 -> 27.0 mm, vias 4 -> 3
- net BMS2: track 49.9 -> 35.9 mm
- net N$16: track 8.00 -> 0.00 mm
- net BMS1: track 62.1 -> 54.3 mm, vias 4 -> 2
- net BMS+: track 141.5 -> 145.5 mm
- net N$1: track 17.2 -> 18.0 mm
- net B-1: track 36.2 -> 36.8 mm
