File: schematics/board/BMSnew.sch (EAGLE design)
At the start: 61 parts

Commit message: Плата АБ
Parts:
- removed B+, B-, BC: BATTERY, CanCubeSat:BATTERY
- added B+2, B-2, BC2: BATTERY, CanCubeSat:BATTERY
Connections:
- removed net BUS+: AB1.4
- removed net N$98: R49.1, U$45.CS
- new net N$13: R1.2, U$3.CS
- net B-1: now also B-1.P$1; no longer B-.P$1
- net B-2: now also B-2.P$1; no longer B-1.P$1
- net BC1: now also BC1.P$1; no longer BC.P$1
- net BC2: now also BC2.P$1; no longer BC1.P$1
- net BMS+: now also AB1.4, B+2.P$1; no longer B+.P$1
- net GND: now also R1.1, R49.1
- net N$16: no longer R49.2
- net N$3: no longer R1.2
- net N$5: now also R49.2, U$45.CS; no longer R1.1, U$3.CS
Other:
- moved on the sheet: B+1, B-1, BC1, R1, R49

Commit message: Сделал платку BMSnew лучше, но не совсем
Parts:
- R11, R12: value 100R -> 100k
Changed lines of the file:
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@@
 <drawing>
 <settings>
-<setting alwaysvectorfont="no"/>
+<setting alwaysvectorfont="yes"/>
 <setting verticaltext="up"/>
 </settings>
@@
 <part name="R9" library="resistor" library_urn="urn:adsk.eagle:library:348" deviceset="R-US_" device="R0603" package3d_urn="urn:adsk.eagle:package:23555/3" value="100R"/>
 <part name="R10" library="resistor" library_urn="urn:adsk.eagle:library:348" deviceset="R-US_" device="R0603" package3d_urn="urn:adsk.eagle:package:23555/3" value="100R"/>
-<part name="R11" library="resistor" library_urn="urn:adsk.eagle:library:348" deviceset="R-US_" device="R0603" package3d_urn="urn:adsk.eagle:package:23555/3" value="100R"/>
-<part name="R12" library="resistor" library_urn="urn:adsk.eagle:library:348" deviceset="R-US_" device="R0603" package3d_urn="urn:adsk.eagle:package:23555/3" value="100R"/>
+<part name="R11" library="resistor" library_urn="urn:adsk.eagle:library:348" deviceset="R-US_" device="R0603" package3d_urn="urn:adsk.eagle:package:23555/3" value="100k"/>
+<part name="R12" library="resistor" library_urn="urn:adsk.eagle:library:348" deviceset="R-US_" device="R0603" package3d_urn="urn:adsk.eagle:package:23555/3" value="100k"/>
 <part name="U$10" library="CanCubeSat" deviceset="MOCD217M" device="" package3d_urn="urn:adsk.eagle:package:8087957/1"/>
 <part name="R15" library="resistor" library_urn="urn:adsk.eagle:library:348" deviceset="R-US_" device="R0603" package3d_urn="urn:adsk.eagle:package:23555/3" value="100R"/>
@@
 <wire x1="116.84" y1="137.16" x2="101.6" y2="137.16" width="0.1524" layer="91"/>
 <wire x1="101.6" y1="137.16" x2="101.6" y2="121.92" width="0.1524" layer="91"/>
-<label x="81.28" y="121.92" size="1.778" layer="95"/>
+<label x="68.58" y="121.92" size="1.778" layer="95"/>
 <pinref part="DS18B20" gate="G$1" pin="2"/>
 <pinref part="DS18B20C" gate="G$1" pin="2"/>
@@
 <pinref part="DS18B20A" gate="G$1" pin="3"/>
 <pinref part="DS18B20B" gate="G$1" pin="3"/>
-<label x="81.28" y="127" size="1.778" layer="95"/>
+<label x="68.58" y="127" size="1.778" layer="95"/>
 <wire x1="66.04" y1="127" x2="104.14" y2="127" width="0.1524" layer="91"/>
 </segment>
@@
 <wire x1="99.06" y1="139.7" x2="99.06" y2="124.46" width="0.1524" layer="91"/>
 <wire x1="66.04" y1="124.46" x2="99.06" y2="124.46" width="0.1524" layer="91"/>
-<label x="88.9" y="124.46" size="1.778" layer="95"/>
-</segment>
-<segment>
+<label x="68.58" y="124.46" size="1.778" layer="95"/>
+</segment>
+<segment>

Commit message: платы DC-DC и AB
Parts:
- added R13, R14, R19, R20: 2k26, resistor:R-US_R0603
- R17, R18: value 100R -> 100k
- R94, R95, R98, R99: value 2k26 -> 200k
Connections:
- removed net N$16: R56.1, U$1.S2, U$10.EM1
- new net N$17: R14.1, R94.2, U$2.AN1
- new net N$18: R13.1, R95.2, U$2.AN2
- new net N$19: R19.1, R99.2, U$10.AN2
- new net NO_GND1: R8.1, R94.1, R95.1, U$2.CAT1, U$2.CAT2, U$2.EM1, U$26.S2
- new net NO_GND2: R56.1, R98.1, R99.1, U$1.S2, U$10.CAT1, U$10.CAT2, U$10.EM1
- net BMS1: now also R13.2, R14.2; no longer R94.2, R95.2, U$2.AN1, U$2.AN2
- net BMS2: now also R19.2, R20.2; no longer R98.2, R99.2, U$10.AN1, U$10.AN2
- net GND: no longer R94.1, R95.1, R98.1, R99.1, U$10.CAT1, U$10.CAT2, U$2.CAT1, U$2.CAT2
- net N$3: now also R20.1, R98.2, U$10.AN1; no longer R8.1, U$2.EM1, U$26.S2
Other:
- moved on the sheet: C25, C26, C27, C28, R15, R16, R17, R18, R49, R50, R51, R52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
