File: schematics/board/DC-DC.sch (EAGLE design)
At the start: 48 parts

Commit message: Папка с платами
Parts:
- removed BSK2, BSK2A: (no value), pinheadCS:PINHD-1X8
- removed BSK3: (no value), pinheadCS:PINHD-1X12
- removed BSK4: (no value), pinheadCS:PINHD-1X14
- removed JTAG: (no value), pinheadCS:PINHD-1X6
- removed LED-B#2: (no value), led:LEDCHIPLED_0603
- removed RADIO: RADIO, CanCubeSat:RADIO
- removed SD: SD, CanCubeSat:SD
- added C10, C2, C25, C26, C7, C8: 0,1µ, rcl:C-USC0603
- added C11: 33p, rcl:C-USC0603
- added C13, C29, C30, C31, C32, C9: 22µ, rcl:C-USC1206
- added C18, C19, C36: 220p, rcl:C-USC0603
- added C20, C22, C23: 1µ, rcl:C-USC0603
- added C21, C24, C35, C37: 4.7nF, rcl:C-USC0603
- added C27, C28: 10p, rcl:C-USC0603
- added C34: 10µ, rcl:C-USC1206
- added C38, C39: 47µ, rcl:C-EUC1210
- added D1: MBR0520LT, diode:MBR0520LT
- added JP10, JP11, JP4, JP5, JP6, JP7, JP8, JP9: (no value), pinheadCS:PINHD-1X3
- added JP12, JP13, JP14, JP15, JP16, JP17, JP18, JP19, JP20, JP21, JP22, JP23, JP24, JP25, JP26, JP27, JP28, JP29, JP30, JP31, JP32, JP33, JP34, JP35, JP36, JP37: (no value), pinheadCS:PINHD-1X1
- added JP2, JP3: (no value), pinheadCS:PINHD-1X2
- added LED2: (no value), led:LEDCHIPLED_0603
- added R1: 162k, resistor:R-US_R0603
- added R14: 8k87, resistor:R-US_R0603
- added R15, R4: 40k2, resistor:R-US_R0603
- added R16: 10k, resistor:R-US_R0603
- added R17, R19: 13k, resistor:R-US_R0603
- added R20: 1M, resistor:R-US_R0603
- added R25: 11k5, resistor:R-US_R0603
- added R26: 18k7, resistor:R-US_R0603
- added R3: 200k, resistor:R-US_R0603
- added R31: 2k, resistor:R-US_R0603
- added R7: 24k9, resistor:R-US_R0603
- added U$1: MP1584+VIA, CanCubeSat:MP1584+VIA
- added U$14: GRAFITGRAFIT2, CanCubeSat:GRAFITGRAFIT2
- added U$15: GRAFITGRAFIT2_1, CanCubeSat:GRAFITGRAFIT2_1
- added U$16: GRAFITGRAFIT2_2, CanCubeSat:GRAFITGRAFIT2_2
- added U$17: GRAFITGRAFIT3, CanCubeSat:GRAFITGRAFIT3
- added U$2: L_10MKH, CanCubeSat:L_10MKH
- added U$21: GRAFITGRAFIT4_1, CanCubeSat:GRAFITGRAFIT4_1
- added U$22: GRAFITGRAFIT4_2, CanCubeSat:GRAFITGRAFIT4_2
- added U$3: MP2225, CanCubeSat:MP2225
- added U$4: L_3.3MKH, CanCubeSat:L_3.3MKH_5X5
- added U$9: GRAFITGRAFIT1_1, CanCubeSat:GRAFITGRAFIT1_1
- C12: value 0,1µ -> 22µ; device rcl:C-USC0603 -> rcl:C-USC1206
- C3: value 10µ -> 22µ; device rcl:C-EUC1206 -> rcl:C-USC1206
- C33: value 0,1µ -> 10µ; device rcl:C-USC0603 -> rcl:C-USC1206
- C4: value 1nF -> 10µ; device rcl:C-USC0603 -> rcl:C-USC1206
- R10: value 5k1 -> 68k1
- R11, R6: value 5k1 -> 100k
- R18: value 3k3 -> 324k
- R21, R22: value 3k3 -> 100k
- R23, R24: value 3k3 -> 1M
- R27: value 2k -> 84k5
- R29: value 10k -> 84k5
- R5: value 12k -> 124k
- U$10: value LTC3633 -> LTC3633+VIA; device CanCubeSat:LTC3633 -> CanCubeSat:LTC3633+VIA
- U$11: device CanCubeSat:B82498F -> CanCubeSat:VLS3012HBX
- U$12: value B82498F -> SPM4020; device CanCubeSat:B82498F -> CanCubeSat:SPM4020
- U$13: value ESP32WROOM -> GRAFITGRAFIT1_2; device CanCubeSat:ESP32WROOM -> CanCubeSat:GRAFITGRAFIT1_2
- U$18: value 74HC595 -> GRAFITGRAFIT3_1; device CanCubeSat:74HC595 -> CanCubeSat:GRAFITGRAFIT3_1
- U$19: value 74HC595 -> GRAFITGRAFIT3_2; device CanCubeSat:74HC595 -> CanCubeSat:GRAFITGRAFIT3_2
- U$20: value 74HC595 -> GRAFITGRAFIT4; device CanCubeSat:74HC595 -> CanCubeSat:GRAFITGRAFIT4
- U$5: value DS18B20Z -> LTC3633+VIA; device CanCubeSat:DS18B20Z -> CanCubeSat:LTC3633+VIA
- U$6: value USB-C -> L_2.2MKH; device CanCubeSat:USB-C -> CanCubeSat:L_2.2MKH
- U$7: value EM_HEAT -> L_2.2MKH; device CanCubeSat:EM_HEAT -> CanCubeSat:L_2.2MKH
- U$8: value L293DD -> GRAFITGRAFIT1; device CanCubeSat:L293DD -> CanCubeSat:GRAFITGRAFIT1
Connections:
- removed net 1W: BSK2.6, BSK2A.6, BSK3.8, BSK4.14, U$13.IO21, U$5.DQ
- removed net AUX: RADIO.AUX, U$13.SVP
- removed net B1_KEM+: U$18.Q2, U$8.IN1
- removed net B1_KEM-: U$18.Q3, U$8.IN2
- removed net B1_KHEAT: U$18.Q1, U$8.IN4
- removed net B2A_KEM+: BSK2A.3, U$19.Q2
- removed net B2A_KEM-: BSK2A.2, U$19.Q3
- removed net B2A_KHEAT: BSK2A.4, U$19.Q1
- removed net B2A_KVCC: BSK2A.5, U$19.Q0
- removed net B2_KEM+: BSK2.3, U$19.Q6
- removed net B2_KEM-: BSK2.2, U$19.Q7
- removed net B2_KHEAT: BSK2.4, U$19.Q5
- removed net B2_KVCC: BSK2.5, U$19.Q4
- removed net B3_KEM+: BSK3.5, U$20.Q6
- removed net B3_KEM-: BSK3.4, U$20.Q7
- removed net B3_KHEAT: BSK3.6, U$20.Q5
- removed net B3_KVCC: BSK3.7, U$20.Q4
- removed net B4_KEM+: BSK4.11, U$18.Q6
- removed net B4_KEM-: BSK4.10, U$18.Q7
- removed net B4_KHEAT: BSK4.12, U$18.Q5
- removed net B4_KVCC: BSK4.13, U$18.Q4
- removed net B5_KEM+: BSK3.2, U$20.Q2
- removed net B5_KEM-: BSK3.1, U$20.Q3
- removed net B5_KHEAT: BSK3.11, U$20.Q1
- removed net B5_KVCC: BSK3.12, U$20.Q0
- removed net DAT0: JP1.2, R23.2, SD.DAT0, U$13.IO2
- removed net DAT1: R24.2, SD.DAT1, U$13.IO4
- removed net DS: U$13.IO25, U$18.DS
- removed net EN: C4.1, R5.1, U$13.EN, U$6.NRST/EN
- removed net I2CINT: BSK4.5, U$13.IO18
- removed net IO0-E: R6.1, U$13.IO0, U$6.NC/GPIO
- removed net IO1: R2.1, U$13.IO5
- removed net M1: R29.1, RADIO.M1, U$13.IO34, U$6.NC/M1
- removed net MTCK: JTAG.5, R21.2, SD.DAT3, U$13.IO13
- removed net MTDI: JTAG.6, R18.2, SD.DAT2, U$13.IO12
- removed net MTDO: JTAG.3, R22.2, SD.CMD, U$13.IO15
- removed net MTMS: JTAG.4, SD.CLK, U$13.IO14
- removed net PL_KVCC: BSK4.8, U$13.IO33
- removed net RX-E: U$13.RXD0, U$6.SWD/RXD
- removed net RX-ES: U$13.IO22
- removed net RX-R: RADIO.TXD, U$13.IO35, U$6.RX0
- removed net SCLTM: BSK4.7, R10.2, U$13.IO16
- removed net SDATM: BSK4.6, R11.2, U$13.IO17
- removed net SHCP: U$13.IO27, U$18.SHCP, U$19.SHCP, U$20.SHCP
- removed net STCP: U$13.IO26, U$18.STCP, U$19.STCP, U$20.STCP
- removed net TIME: BSK4.4, U$13.IO19
- removed net TIME-ES: U$13.SVN
- removed net TX-E: U$13.TXD0, U$6.SWC/TXD
- removed net TX-ES: U$13.IO23
- removed net TX-R: RADIO.RXD, U$13.IO32, U$6.TX0
- new net 3V3: C3.1, R5.1, U$2.1
- new net FB1: C28.1, R26.1, R29.2, U$5.VFB1
- new net FB2: C27.1, R25.1, R27.2, U$5.VFB2
- new net INTVCC: C22.2, C23.2, JP1.2, JP10.1, JP4.3, JP5.3, JP6.3, R21.2, R22.2, U$5.INTVCC
- new net N$1: R1.1, U$10.RT
- new net N$10: C4.2, R6.2, U$1.VIN
- new net N$11: C36.1, R10.1
- new net N$12: C36.2, U$1.COMP
- new net N$13: C7.2, U$3.BST
- new net N$14: C7.1, U$3.SW, U$4.2
- new net N$15: R11.2, U$3.EN
- new net N$16: C8.2, U$3.VCC
- new net N$19: C11.1, C12.2, C13.2, R15.2, U$4.1
- new net N$2: LED1.C, R31.2
- new net N$20: JP1.1, JP2.1, JP3.1, U$5.MODE
- new net N$21: JP4.1, JP4.2, R17.2, U$5.ITH2
- new net N$22: C18.2, R17.1
- new net N$23: JP2.2, R16.1
- new net N$26: JP5.1, JP5.2, R18.1, U$5.RT
- new net N$27: C20.2, U$5.V2P5
- new net N$29: JP6.1, JP6.2, R19.2, U$5.ITH1
- new net N$30: C19.2, R19.1
- new net N$34: C25.1, U$5.SW2, U$5._SW2, U$6.2
- new net N$35: C26.1, U$5.SW1, U$5._SW1, U$7.2
- new net N$36: R22.1, U$5.PGOOD1
- new net N$37: JP8.2, U$5.SS2
- new net N$38: JP7.2, R20.1, U$5.RUN2
- new net N$40: R21.1, U$5.PGOOD2
- new net N$41: JP9.2, R23.1, U$5.RUN1
- new net N$42: JP11.2, U$5.SS1
- new net N$43: C21.2, JP8.1
- new net N$44: JP10.2, R24.1, U$5.PHMODE
- new net N$45: C24.2, JP11.1
- new net N$46: C25.2, U$5.BOOST2
- new net N$47: LED1.A, U$10.PGOOD1
- new net N$48: C26.2, U$5.BOOST1
- new net N$49: JP13.1, JP8.3
- new net N$5: C2.2, U$1.BST
- new net N$50: JP11.3, JP12.1
- new net N$52: C37.2, U$10.SS2
- new net N$53: JP14.1, U$14.P$1
- new net N$54: JP15.1, U$15.P$1
- new net N$55: JP16.1, U$16.P$1
- new net N$56: JP17.1, U$14.P$2
- new net N$57: JP18.1, U$15.P$2
- new net N$58: JP19.1, U$16.P$2
- new net N$59: JP20.1, U$17.P$1
- new net N$6: C2.1, D1.C, U$1.SW, U$2.2
- new net N$60: JP21.1, U$18.P$1
- new net N$61: JP22.1, U$19.P$1
- new net N$62: JP23.1, U$17.P$2
- new net N$63: JP24.1, U$18.P$2
- new net N$64: JP25.1, U$19.P$2
- new net N$65: JP26.1, U$20.P$1
- new net N$66: JP27.1, U$21.P$1
- new net N$67: JP28.1, U$22.P$1
- new net N$68: JP29.1, U$20.P$2
- new net N$69: JP30.1, U$21.P$2
- new net N$7: R3.2, U$1.FREQ
- new net N$70: JP31.1, U$22.P$2
- new net N$71: JP32.1, U$8.P$1
- new net N$72: JP33.1, U$9.P$1
- new net N$73: JP34.1, U$13.P$1
- new net N$74: JP35.1, U$8.P$2
- new net N$75: JP36.1, U$9.P$2
- new net N$76: JP37.1, U$13.P$2
- new net N$8: R4.1, R5.2, U$1.FB
- new net N$9: R6.1, R7.1, U$1.EN
- new net VIN: C38.2, C39.2, JP7.1, JP9.1, U$5.VIN1, U$5.VIN2, U$5._VIN1, U$5._VIN2
- new net VON1: C28.2, C31.2, C32.2, C34.2, R29.1, U$5.VON1, U$7.1
- new net VON2: C27.2, C29.2, C30.2, C33.2, R27.1, U$5.VON2, U$6.1
- net 5V: no longer BSK2.7, BSK2A.7, BSK3.9, BSK4.2, RADIO.VCC, U$5.VDD, U$8.EN1, U$8.EN2, U$8.VS, U$8.VSS
- net BUS+: now also U$10._VIN1, U$10._VIN2; no longer BSK2.8, BSK2A.8, BSK3.10, BSK4.3, U$6.3V3/BUS
- net GND: now also C10.1, C13.1, C18.1, C19.1, C20.1, C21.1, C22.1, C23.1, C24.1, C29.1, C30.1, C31.1, C32.1, C33.1, C34.1, C35.1, C37.1, C38.1, C39.1, C4.1, C8.1, C9.1, D1.A, JP10.3, JP3.2, JP7.3, JP9.3, R1.2, R10.2, R14.2, R16.2, R18.2, R2.1, R20.2, R23.2, R24.2, R25.2, R26.2, R3.1, R31.1, R4.2, R7.2, U$1.GND, U$1.HEAT, U$3.AGND, U$3.GND, U$5.SGND; no longer BSK2.1, BSK2A.1, BSK3.3, BSK4.9, C33.2, C4.2, JP1.1, JTAG.1, R27.2, R29.2, RADIO.GND, RADIO.M0, SD.VSS, U$13.GND, U$13.HEAT, U$18.GND, U$18.OE, U$19.GND, U$19.OE, U$20.GND, U$20.OE, U$5.GND, U$6.GND, U$7.GND, U$8.GND, U$8.HEAT
- net N$17: now also C10.2, C9.2, R11.1, U$3.IN; no longer U$18.Q7S, U$19.DS
- net N$18: now also C11.2, R14.1, R15.1, U$3.FB; no longer U$19.Q7S, U$20.DS
- net N$24: no longer U$10.RT
- net N$28: now also U$10._SW1
- net N$3: now also LED2.A, U$10.PGOOD2; no longer LED-B#2.A, U$7.5V, U$8.OUT4
- net N$33: now also U$10._SW2
- net N$4: now also LED2.C; no longer LED1.C
- net N$51: now also C35.2, U$10.SS1; no longer LED-B#2.C, R27.1
- net VDD: no longer BSK4.1, C12.2, C3.1, C33.1, JTAG.2, LED1.A, R10.1, R11.1, R18.1, R21.1, R22.1, R23.1, R24.1, R5.2, R6.2, SD.VDD, U$13.3V3, U$18.MR, U$18.VCC, U$19.MR, U$19.VCC, U$20.MR, U$20.VCC, U$6.NC/3V3
Other:
- note removed: "HEAT"
- moved on the sheet: C1, C12, C14, C15, C16, C17, C3, C33, C4, C5, C6, JP1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

Commit message: Плата DC-DC
Parts:
- added 3,3µH: 3,3µ, CanCubeSat:B82472G6
- added 3,3µH1: 3,3µH, CanCubeSat:B82472G6
- added C40, C41, C49, C50, C56: 0,1µ, rcl:C-USC0603
- added C44, C52: 680p, rcl:C-USC0603
- added C45, C53: 4.7µ, rcl:C-USC1206
- added C46: 3,3n, rcl:C-USC0603
- added C47, C54: 150µ, CanCubeSat:ECAPECAP150
- added C48, C55: 220µ, CanCubeSat:ECAPECAP220
- added C57: 10µ, rcl:C-USC1206
- added INVERT: INVERTER, CanCubeSat:INVERTER
- added LED_G1, LED_G2, LED_R1, LED_R2: (no value), led:LEDCHIPLED_0603
- added OPA: OPA333, CanCubeSat:OPA333
- added R100, R32, R33, R57: 2k, resistor:R-US_R0603
- added R28, R30, R37, R39, R67, R68, R69: 150k, resistor:R-US_R0603
- added R34, R35: 51k, resistor:R-US_R0603
- added R36, R38, R66: 10k, resistor:R-US_R0603
- added R40: 910k, resistor:R-US_R0603
- added R41: 330k, resistor:R-US_R0603
- added R65: 1M, resistor:R-US_R0603
- added R70: 24k3, resistor:R-US_R0603
- added R72: 232k, resistor:R-US_R0603
- added U$23, U$59: LTC31191, CanCubeSat:LTC31191
- added U$25: 32961, CanCubeSat:32961
Connections:
- new net 1.65: R34.2, R35.1, R36.2
- new net 3.3: INVERT.VCC, OPA.V+, R35.2
- new net 90: R65.1, R66.2, R67.2, U$59.MPPC
- new net A: INVERT.A, OPA.OUT, R32.1, R37.2, R39.2, U$59.RUN
- new net INA_BMS+: C47.1, C55.1, R72.2, U$23.PVIN, U$23.VIN, U$59.PVOUT
- new net INA_BUS+: C48.1, C54.1, R40.1, R65.2, U$23.PVOUT, U$25.CW, U$59.PVIN, U$59.VIN
- new net N$129: C41.2, U$59.BST2
- new net N$131: 3,3µH.2, C40.1, U$59.SW1
- new net N$132: 3,3µH.1, C41.1, U$59.SW2
- new net N$135: R69.1, U$59.VC
- new net N$136: C44.1, R69.2
- new net N$139: C46.1, R66.1
- new net N$142: R68.2, U$59.RT
- new net N$144: C40.2, U$59.BST1
- new net N$215: C53.1, C56.1, C57.1, LED_G2.A, U$23.MPPC, U$23.SVCC, U$23.VCC
- new net N$234: C45.1, LED_G1.A, U$59.SVCC, U$59.VCC
- new net N$302: OPA.IN-, R36.1, R37.1
- new net N$77: 3,3µH1.2, C49.1, U$23.SW1
- new net N$78: 3,3µH1.1, C50.1, U$23.SW2
- new net N$79: R28.2, U$23.RT
- new net N$80: C49.2, U$23.BST1
- new net N$81: R30.1, U$23.VC
- new net N$82: C52.1, R30.2
- new net N$84: C50.2, U$23.BST2
- new net N$85: LED_R1.A, R32.2
- new net N$86: U$23.FB, U$25.WIP
- new net N$87: LED_R2.A, R57.2
- new net N$89: R70.1, R72.1, U$59.FB
- new net N$90: OPA.IN+, R38.1, R39.1
- new net N$91: LED_G1.C, R100.2
- new net N$92: LED_G2.C, R33.2
- new net PGOOD1: LED_R1.C, U$59.PGOOD
- new net PGOOD2: LED_R2.C, U$23.PGOOD
- new net RUN: R38.2, R40.2, R41.1
- new net Y: INVERT.Y, R57.1, U$23.RUN
- net GND: now also C44.2, C45.2, C46.2, C47.2, C48.2, C52.2, C53.2, C54.2, C55.2, C56.2, C57.2, INVERT.GND, OPA.V-, R100.1, R28.1, R33.1, R34.1, R41.2, R67.1, R68.1, R70.2, U$23.PGND, U$23.PWM, U$23.SGND, U$25.CCW, U$59.PGND, U$59.PWM, U$59.SGND
Other:
- note added: "Charge DC-DC"
- note added: "Discharge DC-DC"

Commit message: платы DC-DC и AB
Parts:
- removed D1: MBR0520LT, diode:MBR0520LT
- added D2: (no value), diode:SCHOTTKY-DIODESMC
Connections:
- net GND: now also D2.A; no longer D1.A
- net N$6: now also D2.C; no longer D1.C
Changed lines of the file:
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@@
 <part name="C2" library="rcl" library_urn="urn:adsk.eagle:library:334" deviceset="C-US" device="C0603" package3d_urn="urn:adsk.eagle:package:23616/2" value="0,1µ"/>
 <part name="R3" library="resistor" library_urn="urn:adsk.eagle:library:348" deviceset="R-US_" device="R0603" package3d_urn="urn:adsk.eagle:package:23555/3" value="200k"/>
-<part name="D1" library="diode" library_urn="urn:adsk.eagle:library:210" deviceset="MBR0520LT" device="" package3d_urn="urn:adsk.eagle:package:43420/1"/>
 <part name="U$2" library="CanCubeSat" deviceset="L_10MKH" device=""/>
 <part name="C3" library="rcl" library_urn="urn:adsk.eagle:library:334" deviceset="C-US" device="C1206" package3d_urn="urn:adsk.eagle:package:23618/2" value="22µ"/>
@@
 <part name="LED_R1" library="led" library_urn="urn:adsk.eagle:library:259" deviceset="LED" device="CHIPLED_0603" package3d_urn="urn:adsk.eagle:package:15822/2"/>
 <part name="LED_R2" library="led" library_urn="urn:adsk.eagle:library:259" deviceset="LED" device="CHIPLED_0603" package3d_urn="urn:adsk.eagle:package:15822/2"/>
+<part name="D2" library="diode" library_urn="urn:adsk.eagle:library:210" deviceset="SCHOTTKY-DIODE" device="SMC" package3d_urn="urn:adsk.eagle:package:43425/2"/>
 </parts>
 <sheets>
@@
 <attribute name="NAME" x="-72.39" y="-39.5986" size="1.778" layer="95" rot="R180"/>
 <attribute name="VALUE" x="-72.39" y="-34.798" size="1.778" layer="96" rot="R180"/>
-</instance>
-<instance part="D1" gate="G$1" x="-132.08" y="-17.78" smashed="yes" rot="R270">
-<attribute name="NAME" x="-131.5974" y="-20.32" size="1.778" layer="95" rot="R270"/>
 </instance>
 <instance part="U$2" gate="G$1" x="-147.32" y="-27.94" smashed="yes" rot="R90">
@@
 <attribute name="VALUE" x="14.605" y="-221.488" size="1.778" layer="96" rot="R270"/>
 </instance>
+<instance part="D2" gate="G$1" x="-132.08" y="-17.78" smashed="yes" rot="R270">
+<attribute name="NAME" x="-130.175" y="-15.494" size="1.778" layer="95" rot="R270"/>
+<attribute name="VALUE" x="-135.509" y="-15.494" size="1.778" layer="96" rot="R270"/>
+</instance>
 </instances>
 <busses>
@@
 </segment>
 <segment>
-<pinref part="D1" gate="G$1" pin="A"/>
 <wire x1="-132.08" y1="-15.24" x2="-132.08" y2="-7.62" width="0.1524" layer="91"/>
 <label x="-132.08" y="-12.7" size="1.778" layer="95" rot="R90"/>
+<pinref part="D2" gate="G$1" pin="A"/>
 </segment>
 <segment>
@@
 <wire x1="-124.46" y1="-27.94" x2="-132.08" y2="-27.94" width="0.1524" layer="91"/>
 <junction x="-124.46" y="-27.94"/>
-<pinref part="D1" gate="G$1" pin="C"/>
 <wire x1="-132.08" y1="-27.94" x2="-139.7" y2="-27.94" width="0.1524" layer="91"/>
 <wire x1="-132.08" y1="-20.32" x2="-132.08" y2="-27.94" width="0.1524" layer="91"/>
 <junction x="-132.08" y="-27.94"/>
 <pinref part="U$2" gate="G$1" pin="2"/>
-</segment>
-</net>
+<pinref part="D2" gate="G$1" pin="C"/>
+</segment>
+</net>
