File: schematics/board/AB+DC-DC.brd (EAGLE design)
At the start: 91 x 117 mm, 242 parts

Commit message: Плата АB+DC-DC
Parts:
- moved B+2 0.50 mm to (48.5, 11.5)
Connections:
- net GND: now also R94.1, R95.1, R98.1, R99.1, U$10.2, U$10.4, U$2.2, U$2.4
- net NO_GND1: no longer R94.1, R95.1, U$2.2, U$2.4
- net NO_GND2: no longer R98.1, R99.1, U$10.2, U$10.4
Routing:
- net NO_GND1: track 48.8 -> 10.2 mm, vias 2 -> 0
- net NO_GND2: track 37.7 -> 8.21 mm, vias 1 -> 0
- net GND: track 27.0 -> 54.1 mm
- net N$10: track 17.3 -> 16.7 mm
- net OC2: track 25.6 -> 25.1 mm
- net N$30: track 14.1 -> 14.6 mm
