File: schematics/board/SPout.brd (EAGLE design)
At the start: 82 x 82 mm, 45 parts

Commit message: Платы СБ
Parts:
- removed U$1, U$2, U$20, U$21: KCONNECT3, CanCubeSat:KCONNECT-3
- removed U$18, U$3, U$4: KCONNECT4, CanCubeSat:KCONNECT-4
- removed U$19: KCONNECT1, CanCubeSat:KCONNECT-1
- added U$6: GRAFITGRAFIT3_1, CanCubeSat:GRAFIT3_1
- moved S1 76.0 mm to (21.0, 79.0), turned to 0 degrees
Connections:
- net BUS+: no longer U$1.1, U$1.2, U$1.4, U$18.1, U$18.2, U$18.3, U$20.1, U$20.2, U$20.4, U$3.1, U$3.2, U$3.3
- net BUS-: no longer U$19.2, U$19.3, U$19.4, U$2.1, U$2.2, U$2.4, U$21.1, U$21.2, U$21.4, U$4.1, U$4.2, U$4.3
Routing:
- net N$7: track 23.6 -> 90.6 mm, vias 1 -> 3
- net BUS-: track 76.0 -> 23.3 mm
- net N$1: track 31.3 -> 26.4 mm
- net N$18: track 32.5 -> 33.4 mm
