File: schematics/board/SPout.brd (EAGLE design)
At the start: 82 x 82 mm, 40 parts

Commit message: Добавлены герберы плат BSK1-4, PL, SP и SPIDER
Changed lines of the file:
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@@
 <text x="16.25" y="78.5" size="1.2" layer="26" ratio="20" rot="MR0">ON</text>
 <text x="28.75" y="78.5" size="1.2" layer="26" ratio="20" rot="MR0">OFF</text>
-<text x="19" y="15" size="1.2" layer="26" ratio="20" rot="MR0">BUS+</text>
-<text x="68" y="16" size="1.2" layer="26" ratio="20" rot="MR0">BUS+</text>
-<text x="68" y="65" size="1.2" layer="26" ratio="20" rot="MR0">BUS+</text>
-<text x="19" y="65" size="1.2" layer="26" ratio="20" rot="MR0">BUS+</text>
+<text x="18" y="14" size="1.2" layer="26" ratio="20" rot="MR0">BUS+</text>
+<text x="68" y="15" size="1.2" layer="26" ratio="20" rot="MR0">BUS+</text>
+<text x="69" y="66" size="1.2" layer="26" ratio="20" rot="MR0">BUS+</text>
+<text x="19" y="66" size="1.2" layer="26" ratio="20" rot="MR0">BUS+</text>
 <text x="27" y="56" size="1.2" layer="26" ratio="20" rot="MR0">BUS-</text>
-<text x="60" y="56" size="1.2" layer="26" ratio="20" rot="MR0">BUS-</text>
+<text x="59" y="55" size="1.2" layer="26" ratio="20" rot="MR0">BUS-</text>
 <text x="60" y="24" size="1.2" layer="26" ratio="20" rot="MR0">BUS-</text>
-<text x="27" y="24" size="1.2" layer="26" ratio="20" rot="MR0">BUS-</text>
+<text x="28" y="26" size="1.2" layer="26" ratio="20" rot="MR0">BUS-</text>
 <wire x1="6" y1="13.071" x2="30.395" y2="37.466" width="0.1" layer="22"/>
 <wire x1="37.466" y1="30.395" x2="13.071" y2="6" width="0.1" layer="22"/>
@@
 <signal name="BUS+">
 <polygon width="0.5" layer="1" isolate="0.5">
-<vertex x="84.2" y="-1.8"/>
-<vertex x="84.2" y="85.1"/>
-<vertex x="-2.7" y="85.1"/>
-<vertex x="-2.7" y="-1.8"/>
+<vertex x="81.95" y="0.2"/>
+<vertex x="81.95" y="82.1"/>
+<vertex x="0.3" y="82.1"/>
+<vertex x="0.3" y="0.2"/>
 </polygon>
 <contactref element="S1" pad="2"/>
@@
 <wire x1="45" y1="3" x2="45.17" y2="3" width="0.5" layer="16"/>
 <polygon width="0.5" layer="16" isolate="0.5">
-<vertex x="-14.1" y="-8.2"/>
-<vertex x="89.7" y="-8.2"/>
-<vertex x="89.7" y="91.3"/>
-<vertex x="-14.1" y="91.3"/>
+<vertex x="0.15" y="0.3"/>
+<vertex x="81.7" y="0.3"/>
+<vertex x="81.7" y="82.3"/>
+<vertex x="0.15" y="82.3"/>
 </polygon>
 <wire x1="45.17" y1="3" x2="51" y2="3" width="0.5" layer="16"/>
@@
 <mfgpreviewcolor name="substratecolor" color="0xFF786E46"/>
 </mfgpreviewcolors>
+<errors>
+</errors>
 </board>
 </drawing>
