File: schematics/board/SPIDERnew.brd (EAGLE design)
At the start: 68 x 100 mm, 9 parts

Commit message: плата БСК5
Connections:
- net CMD: now also U$5.2, U$5.3, U$5.4
Changed lines of the file:
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@@
 <signal name="CMD">
 <contactref element="U$5" pad="1"/>
+<contactref element="U$5" pad="2"/>
+<contactref element="U$5" pad="3"/>
+<contactref element="U$5" pad="4"/>
 </signal>
 </signals>
