File: schematics/board/BSK1.sch (EAGLE design)
At the start: 80 parts

Commit message: Две линии i2c на платах БСК заменены на одну
Parts:
- BSK5: device pinheadCS:PINHD-1X10 -> pinheadCS:PINHD-1X8
Connections:
- removed net SCL-INA: BSK5.9, U$57.SCL
- removed net SDA-INA: BSK5.10, U$57.SDA
- net SCL-TM: now also U$57.SCL
- net SDA-TM: now also U$57.SDA
Changed lines of the file:
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@@
 <drawing>
 <settings>
-<setting alwaysvectorfont="yes"/>
+<setting alwaysvectorfont="no"/>
 <setting verticaltext="up"/>
 </settings>
@@
 <part name="U$29" library="CanCubeSat" deviceset="GRAFIT" device="GRAFIT3_1"/>
 <part name="U$30" library="CanCubeSat" deviceset="GRAFIT" device="GRAFIT3_1"/>
-<part name="BSK5" library="pinheadCS" deviceset="PINHD-1X10" device=""/>
+<part name="BSK5" library="pinheadCS" deviceset="PINHD-1X8" device=""/>
 <part name="U$5" library="CanCubeSat" deviceset="SI2302CDS" device=""/>
 <part name="R6" library="resistor" deviceset="R-US_" device="R0603" package3d_urn="urn:adsk.eagle:package:23555/3" value="1M"/>
@@
 </segment>
 </net>
-<net name="SCL-INA" class="0">
-<segment>
-<pinref part="BSK5" gate="A" pin="9"/>
-<wire x1="139.7" y1="309.88" x2="139.7" y2="327.66" width="0.1524" layer="91"/>
-<label x="139.7" y="317.5" size="1.778" layer="95" rot="R90"/>
+<net name="SCL-TM" class="0">
+<segment>
+<pinref part="BSK5" gate="A" pin="5"/>
+<wire x1="129.54" y1="309.88" x2="129.54" y2="327.66" width="0.1524" layer="91"/>
+<label x="129.54" y="317.5" size="1.778" layer="95" rot="R90"/>
+</segment>
+<segment>
+<pinref part="BKU" gate="A" pin="10"/>
+<wire x1="129.54" y1="345.44" x2="129.54" y2="363.22" width="0.1524" layer="91"/>
+<label x="129.54" y="353.06" size="1.778" layer="95" rot="R90"/>
+</segment>
+<segment>
+<pinref part="JP1" gate="A" pin="13"/>
+<wire x1="279.4" y1="342.9" x2="279.4" y2="358.14" width="0.1524" layer="91"/>
+<label x="279.4" y="353.06" size="1.778" layer="95" rot="R90"/>
+</segment>
+<segment>
+<pinref part="JP2" gate="A" pin="13"/>
+<wire x1="279.4" y1="281.94" x2="279.4" y2="297.18" width="0.1524" layer="91"/>
+<label x="279.4" y="292.1" size="1.778" layer="95" rot="R90"/>
+</segment>
+<segment>
+<pinref part="JP3" gate="A" pin="13"/>
+<wire x1="279.4" y1="223.52" x2="279.4" y2="238.76" width="0.1524" layer="91"/>
+<label x="279.4" y="233.68" size="1.778" layer="95" rot="R90"/>
+</segment>
+<segment>
+<pinref part="JP4" gate="A" pin="13"/>
+<wire x1="279.4" y1="165.1" x2="279.4" y2="180.34" width="0.1524" layer="91"/>
+<label x="279.4" y="175.26" size="1.778" layer="95" rot="R90"/>
+</segment>
+<segment>
+<pinref part="JP5" gate="A" pin="13"/>
+<wire x1="279.4" y1="104.14" x2="279.4" y2="119.38" width="0.1524" layer="91"/>
+<label x="279.4" y="114.3" size="1.778" layer="95" rot="R90"/>
+</segment>
+<segment>
+<pinref part="JP6" gate="A" pin="13"/>
+<wire x1="279.4" y1="38.1" x2="279.4" y2="53.34" width="0.1524" layer="91"/>
+<label x="279.4" y="48.26" size="1.778" layer="95" rot="R90"/>
 </segment>
 <segment>
@@
 </segment>
 </net>
-<net name="SDA-INA" class="0">
-<segment>
-<pinref part="BSK5" gate="A" pin="10"/>
-<wire x1="142.24" y1="309.88" x2="142.24" y2="327.66" width="0.1524" layer="91"/>
-<label x="142.24" y="317.5" size="1.778" layer="95" rot="R90"/>
+<net name="SDA-TM" class="0">
+<segment>
+<pinref part="BSK5" gate="A" pin="7"/>
+<wire x1="134.62" y1="309.88" x2="134.62" y2="327.66" width="0.1524" layer="91"/>
+<label x="134.62" y="317.5" size="1.778" layer="95" rot="R90"/>
+</segment>
+<segment>
+<pinref part="BKU" gate="A" pin="12"/>
+<wire x1="134.62" y1="345.44" x2="134.62" y2="363.22" width="0.1524" layer="91"/>
+<label x="134.62" y="353.06" size="1.778" layer="95" rot="R90"/>
+</segment>
+<segment>
+<pinref part="JP1" gate="A" pin="14"/>
+<wire x1="279.4" y1="335.28" x2="279.4" y2="320.04" width="0.1524" layer="91"/>
+<label x="279.4" y="320.04" size="1.778" layer="95" rot="R90"/>
+</segment>
+<segment>
+<pinref part="JP2" gate="A" pin="14"/>
+<wire x1="279.4" y1="274.32" x2="279.4" y2="259.08" width="0.1524" layer="91"/>
+<label x="279.4" y="259.08" size="1.778" layer="95" rot="R90"/>
+</segment>
+<segment>
+<pinref part="JP3" gate="A" pin="14"/>
+<wire x1="279.4" y1="215.9" x2="279.4" y2="200.66" width="0.1524" layer="91"/>
+<label x="279.4" y="200.66" size="1.778" layer="95" rot="R90"/>
+</segment>
+<segment>
+<pinref part="JP4" gate="A" pin="14"/>
+<wire x1="279.4" y1="157.48" x2="279.4" y2="142.24" width="0.1524" layer="91"/>
+<label x="279.4" y="142.24" size="1.778" layer="95" rot="R90"/>
+</segment>
+<segment>
+<pinref part="JP5" gate="A" pin="14"/>
+<wire x1="279.4" y1="96.52" x2="279.4" y2="81.28" width="0.1524" layer="91"/>
+<label x="279.4" y="81.28" size="1.778" layer="95" rot="R90"/>
+</segment>
+<segment>
+<pinref part="JP6" gate="A" pin="14"/>
+<wire x1="279.4" y1="30.48" x2="279.4" y2="15.24" width="0.1524" layer="91"/>
+<label x="279.4" y="15.24" size="1.778" layer="95" rot="R90"/>
 </segment>
 <segment>
@@
 </segment>
 </net>
-<net name="SCL-TM" class="0">
-<segment>
-<pinref part="BSK5" gate="A" pin="5"/>
-<wire x1="129.54" y1="309.88" x2="129.54" y2="327.66" width="0.1524" layer="91"/>
-<label x="129.54" y="317.5" size="1.778" layer="95" rot="R90"/>
-</segment>
-<segment>
-<pinref part="BKU" gate="A" pin="10"/>
-<wire x1="129.54" y1="345.44" x2="129.54" y2="363.22" width="0.1524" layer="91"/>
-<label x="129.54" y="353.06" size="1.778" layer="95" rot="R90"/>
-</segment>
-<segment>
-<pinref part="JP1" gate="A" pin="13"/>
-<wire x1="279.4" y1="342.9" x2="279.4" y2="358.14" width="0.1524" layer="91"/>
-<label x="279.4" y="353.06" size="1.778" layer="95" rot="R90"/>
-</segment>
-<segment>
-<pinref part="JP2" gate="A" pin="13"/>
-<wire x1="279.4" y1="281.94" x2="279.4" y2="297.18" width="0.1524" layer="91"/>
-<label x="279.4" y="292.1" size="1.778" layer="95" rot="R90"/>
-</segment>
-<segment>
-<pinref part="JP3" gate="A" pin="13"/>
-<wire x1="279.4" y1="223.52" x2="279.4" y2="238.76" width="0.1524" layer="91"/>
-<label x="279.4" y="233.68" size="1.778" layer="95" rot="R90"/>
-</segment>
-<segment>
-<pinref part="JP4" gate="A" pin="13"/>
-<wire x1="279.4" y1="165.1" x2="279.4" y2="180.34" width="0.1524" layer="91"/>
-<label x="279.4" y="175.26" size="1.778" layer="95" rot="R90"/>
-</segment>
-<segment>
-<pinref part="JP5" gate="A" pin="13"/>
-<wire x1="279.4" y1="104.14" x2="279.4" y2="119.38" width="0.1524" layer="91"/>
-<label x="279.4" y="114.3" size="1.778" layer="95" rot="R90"/>
-</segment>
-<segment>
-<pinref part="JP6" gate="A" pin="13"/>
-<wire x1="279.4" y1="38.1" x2="279.4" y2="53.34" width="0.1524" layer="91"/>
-<label x="279.4" y="48.26" size="1.778" layer="95" rot="R90"/>
-</segment>
-</net>
-<net name="SDA-TM" class="0">
-<segment>
-<pinref part="BSK5" gate="A" pin="7"/>
-<wire x1="134.62" y1="309.88" x2="134.62" y2="327.66" width="0.1524" layer="91"/>
-<label x="134.62" y="317.5" size="1.778" layer="95" rot="R90"/>
-</segment>
-<segment>
-<pinref part="BKU" gate="A" pin="12"/>
-<wire x1="134.62" y1="345.44" x2="134.62" y2="363.22" width="0.1524" layer="91"/>
-<label x="134.62" y="353.06" size="1.778" layer="95" rot="R90"/>
-</segment>
-<segment>
-<pinref part="JP1" gate="A" pin="14"/>
-<wire x1="279.4" y1="335.28" x2="279.4" y2="320.04" width="0.1524" layer="91"/>
-<label x="279.4" y="320.04" size="1.778" layer="95" rot="R90"/>
-</segment>
-<segment>
-<pinref part="JP2" gate="A" pin="14"/>
-<wire x1="279.4" y1="274.32" x2="279.4" y2="259.08" width="0.1524" layer="91"/>
-<label x="279.4" y="259.08" size="1.778" layer="95" rot="R90"/>
-</segment>
-<segment>
-<pinref part="JP3" gate="A" pin="14"/>
-<wire x1="279.4" y1="215.9" x2="279.4" y2="200.66" width="0.1524" layer="91"/>
-<label x="279.4" y="200.66" size="1.778" layer="95" rot="R90"/>
-</segment>
-<segment>
-<pinref part="JP4" gate="A" pin="14"/>
-<wire x1="279.4" y1="157.48" x2="279.4" y2="142.24" width="0.1524" layer="91"/>
-<label x="279.4" y="142.24" size="1.778" layer="95" rot="R90"/>
-</segment>
-<segment>
-<pinref part="JP5" gate="A" pin="14"/>
-<wire x1="279.4" y1="96.52" x2="279.4" y2="81.28" width="0.1524" layer="91"/>
-<label x="279.4" y="81.28" size="1.778" layer="95" rot="R90"/>
-</segment>
-<segment>
-<pinref part="JP6" gate="A" pin="14"/>
-<wire x1="279.4" y1="30.48" x2="279.4" y2="15.24" width="0.1524" layer="91"/>
-<label x="279.4" y="15.24" size="1.778" layer="95" rot="R90"/>
-</segment>
-</net>
