File: schematics/board/BSK2.sch (EAGLE design)
At the start: 27 parts

Commit message: Сделаны платы CROSSnew, SPIDERnew, BSK2
Parts:
- removed DS18B20Z: DS18B20Z, CanCubeSat:DS18B20Z
- removed FS8205A: FS8205A+, CanCubeSat:FS8205A+
- removed L293DD: L293DD, CanCubeSat:L293DD
- removed LAP4: LAP4-BOTTOM, led:LAP4-BOTTOM
- removed LED1, LED2, LED3, LED4: (no value), led:LEDCHIPLED_0603
- removed R1, R2, R3, R81: 2k, resistor:R-US_R0603
- removed R10, R11: 100R, resistor:R-US_R0603
- removed R19: 1M, resistor:R-US_R0603
- removed R20: 510k, resistor:R-US_R0603
- added CMD: KCONNECTQUAD, CanCubeSat:KCONNECTQUAD
- added DS18B20Z1: DS18B20Z, CanCubeSat:DS18B20Z
- added LED6, LED7: (no value), led:LEDCHIPLED_0603
- added R12, R6: 2M, resistor:R-US_R0603
- added R13: 1k5, resistor:R-US_R0603
- added R14, R5, R8, R9: 1M, resistor:R-US_R0603
- added R4, R7: 2k, resistor:R-US_R0603
- added R94, R95: 2k26, resistor:R-US_R0603
- added U$13, U$8: SI2302CDS, CanCubeSat:SI2302CDS
- added U$14: EM_HEAT, CanCubeSat:EM_HEAT
- added U$15, U$16: GRAFITGRAFIT3_1, CanCubeSat:GRAFITGRAFIT3_1
- added U$26: FS8205A+, CanCubeSat:FS8205A+
- added U$5: MOCD217M, CanCubeSat:MOCD217M
- added YELLOW: LAP4-BOTTOM, led:LAP4-BOTTOM
- U$6, U$7: value EM_HEAT -> GRAFITGRAFIT3_1; device CanCubeSat:EM_HEAT -> CanCubeSat:GRAFITGRAFIT3_1
- renumbered BSK1 to BKU
Connections:
- removed net B2_KEM+: BKU.3, L293DD.IN1
- removed net B2_KEM-: BKU.2, L293DD.IN2
- removed net B2_KHEAT: BKU.4, L293DD.IN4
- removed net B2_KVCC: BKU.5, R10.1, R11.1, R19.1, R20.1
- removed net N$1: L293DD.OUT1, LED1.C, LED2.A, U$6.5V
- removed net N$2: L293DD.OUT2, R1.1, R81.1, U$6.GND
- removed net N$22: LED2.C, R81.2
- removed net N$23: LED1.A, R1.2
- removed net N$24: LED3.C, R2.1
- removed net N$25: LAP4.A, LED4.A, R3.2
- removed net N$3: L293DD.OUT4, LED3.A, U$7.5V
- removed net N$8: FS8205A.G1, R10.2
- removed net N$9: FS8205A.G2, R11.2
- new net 1: R7.2, U$14.GND, U$8.D
- new net 2: R13.2, U$13.D, U$15.P$1, U$16.P$1, U$6.P$1, U$7.P$1
- new net B2-CMD: BKU.4, CMD.P$1
- new net B2-KHEAT: BKU.1, R8.1, U$8.G
- new net B2-KVCC: BKU.2, R94.2, R95.2, U$5.AN1, U$5.AN2
- new net B2-ROZE: BKU.3, R14.1, U$13.G
- new net N$26: R5.1, R6.2, U$26.G2
- new net N$27: R12.1, R9.1, U$26.G1
- new net N$28: R4.2, YELLOW.A
- new net N$29: LED7.C, R13.1
- new net N$31: LED6.C, R7.1
- new net OC1: R9.2, U$5.COL2
- new net OD1: R5.2, U$5.COL1
- net 1W: now also BKU.5, DS18B20Z1.DQ; no longer BKU.6, DS18B20Z.DQ
- net 5V: now also DS18B20Z1.VDD, LED6.A, R4.1, U$14.5V; no longer DS18B20Z.VDD, L293DD.EN1, L293DD.EN2, L293DD.VS, L293DD.VSS, R3.1
- net BUS+: now also BKU.6, LED7.A, R12.2, R6.1, U$15.P$2, U$16.P$2, U$6.P$2, U$7.P$2; no longer BKU.8, R19.2
- net BUS-: now also U$26.S2, U$5.EM1, YELLOW.C; no longer FS8205A.S1, LAP4.C, LED4.C, R20.2
- net GND: now also BKU.8, DS18B20Z1.GND, DS18B20Z1.HEAT, R14.2, R8.2, R94.1, R95.1, U$13.S, U$26.HEAT, U$26.S1, U$5.CAT1, U$5.CAT2, U$5.EM2, U$8.S; no longer BKU.1, DS18B20Z.GND, DS18B20Z.HEAT, FS8205A.HEAT, FS8205A.S2, L293DD.GND, L293DD.HEAT, R2.2, U$7.GND
Other:
- note removed: "EM"

Commit message: Исправлена БСК1
Parts:
- added C41: 0,1µ, rcl:C-USC0603
- added R1, R2: 2k26, resistor:R-US_R0603
- added R75: R01, rcl:R-US_R2512
- added R76, R77: 10R, resistor:R-US_R0603
- added U$57: INA219AID, CanCubeSat:INA219AID
- BKU: device pinheadCS:PINHD-1X8 -> pinheadCS:PINHD-1X11
- R12, R6: value 2M -> 100k
- R5, R9: value 1M -> 100R
- R94, R95: value 2k26 -> 200k
Connections:
- net BUS+1 renamed SP+1
- net BUS+2 renamed SP+2
- net BUS+3 renamed SP+3
- net BUS- renamed SP-
- net BUS-1 renamed SP-1
- net BUS-2 renamed SP-2
- net BUS-3 renamed SP-3
- new net 3V3: BKU.8, U$57.VS
- new net N$150: C41.1, R76.2, U$57.IN+
- new net N$151: C41.2, R77.2, U$57.IN-
- new net N$17: R1.1, R94.2, U$5.AN1
- new net N$18: R2.1, R95.2, U$5.AN2
- new net SCL-INA: BKU.10, U$57.SCL
- new net SDA-INA: BKU.11, U$57.A0, U$57.SDA
- new net SP+: R75.1, R77.1, U$3.P$1
- net B2-KVCC: now also R1.2, R2.2; no longer R94.2, R95.2, U$5.AN1, U$5.AN2
- net BUS+: now also R75.2, R76.1; no longer U$3.P$1
- net GND: now also BKU.9, U$57.A1, U$57.GND; no longer BKU.8

Commit message: Плата АB+DC-DC
Other:
- moved on the sheet: C41, R75, R76, R77

Commit message: Изменен номинал резисторов
Parts:
- R13: value 1k5 -> 3k3
Changed lines of the file:
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@@
 <part name="R8" library="resistor" library_urn="urn:adsk.eagle:library:348" deviceset="R-US_" device="R0603" package3d_urn="urn:adsk.eagle:package:23555/3" value="1M"/>
 <part name="U$13" library="CanCubeSat" deviceset="SI2302CDS" device=""/>
-<part name="R13" library="resistor" library_urn="urn:adsk.eagle:library:348" deviceset="R-US_" device="R0603" package3d_urn="urn:adsk.eagle:package:23555/3" value="1k5"/>
+<part name="R13" library="resistor" library_urn="urn:adsk.eagle:library:348" deviceset="R-US_" device="R0603" package3d_urn="urn:adsk.eagle:package:23555/3" value="3k3"/>
 <part name="LED7" library="led" library_urn="urn:adsk.eagle:library:259" deviceset="LED" device="CHIPLED_0603" package3d_urn="urn:adsk.eagle:package:15822/2"/>
 <part name="R14" library="resistor" library_urn="urn:adsk.eagle:library:348" deviceset="R-US_" device="R0603" package3d_urn="urn:adsk.eagle:package:23555/3" value="1M"/>

Commit message: Внесены правки в платы БСК
Parts:
- added R3, R32: 100R, resistor:R-US_R0603
Connections:
- new net N$19: R32.1, R8.1, U$8.G
- new net N$20: R14.1, R3.1, U$13.G
- net B2-KHEAT: now also R32.2; no longer R8.1, U$8.G
- net B2-ROZE: now also R3.2; no longer R14.1, U$13.G
Changed lines of the file:
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@@
 <part name="R1" library="resistor" library_urn="urn:adsk.eagle:library:348" deviceset="R-US_" device="R0603" package3d_urn="urn:adsk.eagle:package:23555/3" value="2k26"/>
 <part name="R2" library="resistor" library_urn="urn:adsk.eagle:library:348" deviceset="R-US_" device="R0603" package3d_urn="urn:adsk.eagle:package:23555/3" value="2k26"/>
+<part name="R32" library="resistor" deviceset="R-US_" device="R0603" package3d_urn="urn:adsk.eagle:package:23555/3" value="100R"/>
+<part name="R3" library="resistor" deviceset="R-US_" device="R0603" package3d_urn="urn:adsk.eagle:package:23555/3" value="100R"/>
 </parts>
 <sheets>
@@
 <attribute name="VALUE" x="-126.238" y="285.75" size="1.778" layer="96" rot="R90"/>
 </instance>
+<instance part="R32" gate="G$1" x="-177.8" y="96.52" smashed="yes" rot="R90">
+<attribute name="NAME" x="-179.2986" y="92.71" size="1.778" layer="95" rot="R90"/>
+<attribute name="VALUE" x="-174.498" y="92.71" size="1.778" layer="96" rot="R90"/>
+</instance>
+<instance part="R3" gate="G$1" x="-81.28" y="96.52" smashed="yes" rot="R90">
+<attribute name="NAME" x="-82.7786" y="92.71" size="1.778" layer="95" rot="R90"/>
+<attribute name="VALUE" x="-77.978" y="92.71" size="1.778" layer="96" rot="R90"/>
+</instance>
 </instances>
 <busses>
@@
 <net name="B2-ROZE" class="0">
 <segment>
-<pinref part="R14" gate="G$1" pin="1"/>
-<wire x1="-96.52" y1="88.9" x2="-81.28" y2="88.9" width="0.1524" layer="91"/>
-<pinref part="U$13" gate="G$1" pin="G"/>
-<wire x1="-81.28" y1="88.9" x2="-81.28" y2="86.36" width="0.1524" layer="91"/>
-<wire x1="-81.28" y1="88.9" x2="-81.28" y2="106.68" width="0.1524" layer="91"/>
-<junction x="-81.28" y="88.9"/>
-<label x="-81.28" y="96.52" size="1.778" layer="95" rot="R90"/>
-</segment>
-<segment>
 <wire x1="149.86" y1="177.8" x2="149.86" y2="198.12" width="0.1524" layer="91"/>
 <label x="149.86" y="185.42" size="1.778" layer="95" rot="R90"/>
 <pinref part="BKU" gate="A" pin="3"/>
+</segment>
+<segment>
+<pinref part="R3" gate="G$1" pin="2"/>
+<wire x1="-81.28" y1="101.6" x2="-81.28" y2="111.76" width="0.1524" layer="91"/>
+<label x="-81.28" y="104.14" size="1.778" layer="95" rot="R90"/>
 </segment>
 </net>
@@
 <net name="B2-KHEAT" class="0">
 <segment>
-<pinref part="R8" gate="G$1" pin="1"/>
-<wire x1="-193.04" y1="88.9" x2="-177.8" y2="88.9" width="0.1524" layer="91"/>
-<pinref part="U$8" gate="G$1" pin="G"/>
-<wire x1="-177.8" y1="88.9" x2="-177.8" y2="86.36" width="0.1524" layer="91"/>
-<wire x1="-177.8" y1="88.9" x2="-177.8" y2="106.68" width="0.1524" layer="91"/>
-<junction x="-177.8" y="88.9"/>
-<label x="-177.8" y="96.52" size="1.778" layer="95" rot="R90"/>
-</segment>
-<segment>
 <wire x1="144.78" y1="177.8" x2="144.78" y2="198.12" width="0.1524" layer="91"/>
 <label x="144.78" y="185.42" size="1.778" layer="95" rot="R90"/>
 <pinref part="BKU" gate="A" pin="1"/>
+</segment>
+<segment>
+<pinref part="R32" gate="G$1" pin="2"/>
+<wire x1="-177.8" y1="101.6" x2="-177.8" y2="111.76" width="0.1524" layer="91"/>
+<label x="-177.8" y="104.14" size="1.778" layer="95" rot="R90"/>
 </segment>
 </net>
@@
 </segment>
 </net>
+<net name="N$19" class="0">
+<segment>
+<pinref part="R8" gate="G$1" pin="1"/>
+<wire x1="-193.04" y1="88.9" x2="-177.8" y2="88.9" width="0.1524" layer="91"/>
+<pinref part="R32" gate="G$1" pin="1"/>
+<wire x1="-177.8" y1="88.9" x2="-177.8" y2="91.44" width="0.1524" layer="91"/>
+<pinref part="U$8" gate="G$1" pin="G"/>
+<wire x1="-177.8" y1="86.36" x2="-177.8" y2="88.9" width="0.1524" layer="91"/>
+<junction x="-177.8" y="88.9"/>
+</segment>
+</net>
+<net name="N$20" class="0">
+<segment>
+<pinref part="R14" gate="G$1" pin="1"/>
+<wire x1="-96.52" y1="88.9" x2="-81.28" y2="88.9" width="0.1524" layer="91"/>
+<pinref part="R3" gate="G$1" pin="1"/>
+<wire x1="-81.28" y1="88.9" x2="-81.28" y2="91.44" width="0.1524" layer="91"/>
+<pinref part="U$13" gate="G$1" pin="G"/>
+<wire x1="-81.28" y1="86.36" x2="-81.28" y2="88.9" width="0.1524" layer="91"/>
+<junction x="-81.28" y="88.9"/>
+</segment>
+</net>

Commit message: Две линии i2c на платах БСК заменены на одну
Connections:
- net SCL-INA renamed SCL-TM
- net SDA-INA renamed SDA-TM
Changed lines of the file:
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@@
 </segment>
 </net>
-<net name="SCL-INA" class="0">
+<net name="SCL-TM" class="0">
 <segment>
 <wire x1="-273.05" y1="220.98" x2="-273.05" y2="231.14" width="0.1524" layer="91"/>
@@
 </segment>
 </net>
-<net name="SDA-INA" class="0">
+<net name="SDA-TM" class="0">
 <segment>
 <wire x1="-270.51" y1="220.98" x2="-270.51" y2="228.6" width="0.1524" layer="91"/>
