File: schematics/board/BSK3.sch (EAGLE design)
At the start: 28 parts

Commit message: Сделаны платы CROSSnew, SPIDERnew, BSK2
Parts:
- removed DS18B20Z: DS18B20Z, CanCubeSat:DS18B20Z
- removed FS8205A: FS8205A+, CanCubeSat:FS8205A+
- removed L293DD: L293DD, CanCubeSat:L293DD
- removed LAP4: LAP4-BOTTOM, led:LAP4-BOTTOM
- removed LED1, LED2, LED3, LED4: (no value), led:LEDCHIPLED_0603
- removed R1, R2, R3, R81: 2k, resistor:R-US_R0603
- removed R10, R11: 100R, resistor:R-US_R0603
- removed R19: 1M, resistor:R-US_R0603
- removed R20: 510k, resistor:R-US_R0603
- removed U$6, U$7: EM_HEAT, CanCubeSat:EM_HEAT
- added DS18B20Z1: DS18B20Z, CanCubeSat:DS18B20Z
- added LAP1: LAP4-BOTTOM, led:LAP4-BOTTOM
- added LED6, LED7: (no value), led:LEDCHIPLED_0603
- added R12, R6: 2M, resistor:R-US_R0603
- added R13: 1k5, resistor:R-US_R0603
- added R14, R5, R8, R9: 1M, resistor:R-US_R0603
- added R4, R7: 2k, resistor:R-US_R0603
- added R94, R95: 2k26, resistor:R-US_R0603
- added U$13, U$8: SI2302CDS, CanCubeSat:SI2302CDS
- added U$14: EM_HEAT, CanCubeSat:EM_HEAT
- added U$26: FS8205A+, CanCubeSat:FS8205A+
- added U$5: MOCD217M, CanCubeSat:MOCD217M
Connections:
- removed net HEAT: DS18B20Z.HEAT, FS8205A.HEAT, L293DD.HEAT
- removed net N$1: L293DD.OUT1, LED1.C, LED2.A, U$6.5V
- removed net N$2: L293DD.OUT2, R1.1, R81.1, U$6.GND
- removed net N$3: L293DD.OUT4, LED3.A, U$7.5V
- removed net N$4: LED2.C, R81.2
- removed net N$5: LED1.A, R1.2
- removed net N$6: LED3.C, R2.1
- removed net N$7: LAP4.A, LED4.A, R3.2
- removed net N$8: FS8205A.G1, R10.2
- removed net N$9: FS8205A.G2, R11.2
- new net 1: R7.2, U$14.GND, U$8.D
- new net 2: R13.2, U$13.D
- new net B3-KHEAT: R8.1, U$8.G
- new net B3-KVCC: R94.2, R95.2, U$5.AN1, U$5.AN2
- new net B3-ROZE: R14.1, U$13.G
- new net N$10: R5.1, R6.2, U$26.G2
- new net N$27: R12.1, R9.1, U$26.G1
- new net N$28: LAP1.A, R4.2
- new net N$29: LED7.C, R13.1
- new net N$30: DS18B20Z1.HEAT, U$26.HEAT
- new net N$31: LED6.C, R7.1
- new net OC1: R9.2, U$5.COL2
- new net OD1: R5.2, U$5.COL1
- net 1W: now also DS18B20Z1.DQ; no longer DS18B20Z.DQ
- net 5V: now also DS18B20Z1.VDD, LED6.A, R4.1, U$14.5V; no longer DS18B20Z.VDD, L293DD.EN1, L293DD.EN2, L293DD.VS, L293DD.VSS, R3.1
- net B3_KEM+: no longer L293DD.IN1
- net B3_KEM-: no longer L293DD.IN2
- net B3_KHEAT: no longer L293DD.IN4
- net B3_KVCC: no longer R10.1, R11.1, R19.1, R20.1
- net BUS+: now also LED7.A, R12.2, R6.1; no longer R19.2
- net BUS-: now also LAP1.C, U$26.S2, U$5.EM1; no longer FS8205A.S1, LAP4.C, LED4.C, R20.2
- net GND: now also DS18B20Z1.GND, R14.2, R8.2, R94.1, R95.1, U$13.S, U$26.S1, U$5.CAT1, U$5.CAT2, U$5.EM2, U$8.S; no longer DS18B20Z.GND, FS8205A.S2, L293DD.GND, R2.2, U$7.GND
Other:
- note removed: "EM"

Commit message: Плата АB+DC-DC
Parts:
- removed BSK1: (no value), pinheadCS:PINHD-1X12
- removed LAP1: LAP4-BOTTOM, led:LAP4-BOTTOM
- added BKU: (no value), pinheadCS:PINHD-1X16
- added C41: 0,1µ, rcl:C-USC0603
- added CMD: KCONNECTQUAD, CanCubeSat:KCONNECTQUAD
- added R1, R2: 2k26, resistor:R-US_R0603
- added R75: R01, rcl:R-US_R2512
- added R76, R77: 10R, resistor:R-US_R0603
- added U$15, U$16, U$6, U$7: GRAFITGRAFIT3_1, CanCubeSat:GRAFITGRAFIT3_1
- added U$57: INA219AID, CanCubeSat:INA219AID
- added YELLOW: LAP4-BOTTOM, led:LAP4-BOTTOM
- BSK5: device pinheadCS:PINHD-1X8 -> pinheadCS:PINHD-1X12
- R12, R6: value 2M -> 100k
- R5, R9: value 1M -> 100R
- R94, R95: value 2k26 -> 200k
Connections:
- net BUS+1 renamed SP+1
- net BUS+2 renamed SP+2
- net BUS+3 renamed SP+3
- net BUS-1 renamed SP-1
- net BUS-2 renamed SP-2
- net BUS-3 renamed SP-3
- removed net B3_KEM+: BSK1.5
- removed net B3_KEM-: BSK1.4
- removed net B3_KHEAT: BSK1.6
- removed net B3_KVCC: BSK1.7
- removed net B5_KEM+: BSK1.2, BSK5.3
- removed net B5_KEM-: BSK1.1, BSK5.2
- removed net B5_KHEAT: BSK1.11, BSK5.4
- removed net B5_KVCC: BSK1.12, BSK5.5
- removed net BUS-: LAP1.C, U$2.P$1, U$26.S2, U$5.EM1
- removed net N$30: DS18B20Z1.HEAT, U$26.HEAT
- new net 3V3: BKU.8, BSK5.4, U$57.VS
- new net B3-CMD: BKU.4, CMD.P$1
- new net B5-CMD: BKU.13, BSK5.9
- new net B5-KHEAT: BKU.10, BSK5.6
- new net B5-KVCC: BKU.11, BSK5.7
- new net B5-ROZE: BKU.12, BSK5.8
- new net N$150: C41.1, R76.2, U$57.IN+
- new net N$151: C41.2, R77.2, U$57.IN-
- new net N$2: R1.1, R94.2, U$5.AN1
- new net N$3: R2.1, R95.2, U$5.AN2
- new net SCL-INA: BKU.15, BSK5.11, U$57.A0, U$57.SCL
- new net SDA-INA: BKU.16, BSK5.12, U$57.SDA
- new net SINS-KVCC: BKU.14, BSK5.10
- new net SP+: R75.1, R77.1, U$3.P$1
- new net SP-: U$2.P$1, U$26.S2, U$5.EM1, YELLOW.C
- net 1W: now also BKU.5, BSK5.1; no longer BSK1.8, BSK5.6
- net 2: now also U$15.P$1, U$16.P$1, U$6.P$1, U$7.P$1
- net 5V: now also BKU.7, BSK5.3; no longer BSK1.9, BSK5.7
- net B3-KHEAT: now also BKU.1
- net B3-KVCC: now also BKU.2, R1.2, R2.2; no longer R94.2, R95.2, U$5.AN1, U$5.AN2
- net B3-ROZE: now also BKU.3
- net BUS+: now also BKU.6, BSK5.2, R75.2, R76.1, U$15.P$2, U$16.P$2, U$6.P$2, U$7.P$2; no longer BSK1.10, BSK5.8, U$3.P$1
- net GND: now also BKU.9, BSK5.5, DS18B20Z1.HEAT, U$26.HEAT, U$57.A1, U$57.GND; no longer BSK1.3, BSK5.1
- net N$28: now also YELLOW.A; no longer LAP1.A
Other:
- moved on the sheet: LED6, LED7, R12, R13, R14, R4, R5, R6, R7, R8, R9, R94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

Commit message: Внесены правки в платы БСК
Parts:
- added R3, R32: 100R, resistor:R-US_R0603
- BKU: device pinheadCS:PINHD-1X16 -> pinheadCS:PINHD-1X14
- BSK5: device pinheadCS:PINHD-1X12 -> pinheadCS:PINHD-1X8
Connections:
- removed net B5-CMD: BKU.13, BSK5.9
- removed net B5-KVCC: BKU.11, BSK5.7
- removed net B5-ROZE: BKU.12, BSK5.8
- new net N$20: R32.1, R8.1, U$8.G
- new net N$21: R14.1, R3.1, U$13.G
- net 3V3: no longer BSK5.4
- net B3-KHEAT: now also R32.2; no longer R8.1, U$8.G
- net B3-ROZE: now also R3.2; no longer R14.1, U$13.G
- net B5-KHEAT: now also BSK5.5; no longer BSK5.6
- net GND: now also BKU.14, BSK5.4; no longer BSK5.5
- net SCL-INA: now also BKU.12, BSK5.7; no longer BKU.15, BSK5.11
- net SDA-INA: now also BKU.13, BSK5.8; no longer BKU.16, BSK5.12
- net SINS-KVCC: now also BKU.11, BSK5.6; no longer BKU.14, BSK5.10

Commit message: Две линии i2c на платах БСК заменены на одну
Parts:
- BSK5: device pinheadCS:PINHD-1X8 -> pinheadCS:PINHD-1X6
Connections:
- removed net SCL-INA: BKU.12, BSK5.7, U$57.A0, U$57.SCL
- removed net SDA-INA: BKU.13, BSK5.8, U$57.SDA
- new net SCL-TM: BKU.12, U$57.A0, U$57.SCL
- new net SDA-TM: BKU.13, U$57.SDA
Changed lines of the file:
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@@
 <part name="U$20" library="CanCubeSat" deviceset="KCONNECT" device=""/>
 <part name="U$21" library="CanCubeSat" deviceset="KCONNECT" device=""/>
-<part name="BSK5" library="pinheadCS" deviceset="PINHD-1X8" device=""/>
+<part name="BSK5" library="pinheadCS" deviceset="PINHD-1X6" device=""/>
 <part name="DS18B20Z1" library="CanCubeSat" deviceset="DS18B20Z" device=""/>
 <part name="R94" library="resistor" library_urn="urn:adsk.eagle:library:348" deviceset="R-US_" device="R0603" package3d_urn="urn:adsk.eagle:package:23555/3" value="200k"/>
@@
 <attribute name="NAME" x="64.262" y="89.662" size="1.27" layer="95"/>
 </instance>
-<instance part="BSK5" gate="A" x="162.56" y="119.38" smashed="yes" rot="MR270">
-<attribute name="NAME" x="175.133" y="124.968" size="1.778" layer="95" rot="MR270"/>
-<attribute name="VALUE" x="175.26" y="125.73" size="1.778" layer="96" rot="MR270"/>
+<instance part="BSK5" gate="A" x="160.02" y="119.38" smashed="yes" rot="MR270">
+<attribute name="NAME" x="170.053" y="124.968" size="1.778" layer="95" rot="MR270"/>
+<attribute name="VALUE" x="172.72" y="125.73" size="1.778" layer="96" rot="MR270"/>
 </instance>
 <instance part="DS18B20Z1" gate="G$1" x="-91.44" y="167.64" smashed="yes"/>
@@
 </segment>
 </net>
-<net name="SCL-INA" class="0">
+<net name="SCL-TM" class="0">
 <segment>
 <wire x1="-273.05" y1="208.28" x2="-273.05" y2="218.44" width="0.1524" layer="91"/>
@@
 </segment>
 <segment>
-<wire x1="167.64" y1="121.92" x2="167.64" y2="137.16" width="0.1524" layer="91"/>
-<label x="167.64" y="127" size="1.778" layer="95" rot="R90"/>
-<pinref part="BSK5" gate="A" pin="7"/>
-</segment>
-<segment>
 <wire x1="180.34" y1="88.9" x2="180.34" y2="104.14" width="0.1524" layer="91"/>
 <label x="180.34" y="93.98" size="1.778" layer="95" rot="R90"/>
@@
 </segment>
 </net>
-<net name="SDA-INA" class="0">
+<net name="SDA-TM" class="0">
 <segment>
 <wire x1="-270.51" y1="208.28" x2="-270.51" y2="215.9" width="0.1524" layer="91"/>
@@
 </segment>
 <segment>
-<wire x1="170.18" y1="121.92" x2="170.18" y2="137.16" width="0.1524" layer="91"/>
-<label x="170.18" y="127" size="1.778" layer="95" rot="R90"/>
-<pinref part="BSK5" gate="A" pin="8"/>
-</segment>
-<segment>
