File: schematics/board/PLnew.brd (EAGLE design)
At the start: 89 x 89 mm, 39 parts, among them IC2 STM32F103C8T, Q5 8MHz

Commit message: плата БСК5
Parts:
- removed C005R: 32,768KHz, CanCubeSat:C005R
- removed C44, C45: 27pF, rcl:C0603
- removed C46, C47: 10pF, rcl:C0603
- removed Q5: 8MHz, 9C-8.000MEEJ-T:XTAL_9C-8.000MEEJ-T
- removed R78: 1M, resistor:R0603
- added C1, C5: 10nF, rcl:C0603
- added C4: 1nF, rcl:C0603
- added U$18: Q32.768, CanCubeSat:Q32.768
- added U$21: Q24, CanCubeSat:Q24
Connections:
- removed net N$133: C44.1, IC2.6, Q5.1, R78.1
- removed net N$145: C45.1, IC2.5, Q5.2, R78.2
- removed net N$148: C005R.P$2, C47.1, IC2.4
- removed net N$152: C005R.P$1, C46.1, IC2.3
- new net 3V3: C1.2, C5.2, U$18.P$4, U$21.P$4
- new net N$2: IC2.3, U$18.P$3
- new net N$43: C4.2, U$21.P$3
- new net N$44: C4.1, IC2.5
- net GND: now also C1.1, C5.1, U$18.P$2, U$21.P$2; no longer C44.2, C45.2, C46.2, C47.2
Routing:
- net N$145: track 25.7 -> 0.00 mm
- net N$133: track 22.9 -> 0.00 mm
- net N$148: track 7.91 -> 0.00 mm
- net N$152: track 7.49 -> 0.00 mm

Commit message: Две линии i2c на платах БСК заменены на одну
Parts:
- removed BSK4: (no value), pinheadCS:1X08
- removed C1, C5: 10nF, rcl:C0603
- removed C15, C48, C53, C54, C55: 100nF, rcl:C0603
- removed C16: 10µ, rcl:C1206
- removed C4: 1nF, rcl:C0603
- removed IC2: STM32F103C8T, CanCubeSat:LQFP48
- removed ME-O2: ME-O2, CanCubeSat:ME-O2
- removed PB5, PWR: (no value), led:CHIPLED_0603
- removed R101, R102: 5k1, resistor:R0603
- removed R64, R79: 10k, resistor:R0603
- removed R81, R82: 2k, resistor:R0603
- removed U$18: Q32.768, CanCubeSat:Q32.768
- removed U$21: Q24, CanCubeSat:Q24
- removed USB-C: USB-C, CanCubeSat:USB-C
- added BSK1: (no value), pinheadCS:2X04
- added C10: 10nF, rcl:C0603
- added C13, C9: 2,2µ, rcl:C0603
- added C18, C2, C20, C3, C6: 100nF, rcl:C0603
- added C19: 10µ, rcl:C1206
- added C8: 1nF, rcl:C0603
- added LED2, LED3: (no value), led:CHIPLED_0603
- added R10, R11, R12: 10k, resistor:R0603
- added R13, R20, R24, R30: 0.05A, rcl:R1210
- added R14, R21, R22, R28: 1M, resistor:R0603
- added R15, R16: 2k, resistor:R0603
- added R17, R18: 5k1, resistor:R0603
- added R19, R23, R29, R31: 100R, resistor:R0603
- added U$1: MS5611, CanCubeSat:MS5611
- added U$19, U$3, U$4, U$5, U$7: SI2302CDS, CanCubeSat:SOT23-3
- added U$2: Q24, CanCubeSat:Q24
- added U$6: USB-C, CanCubeSat:USB-C
- added U1: STM32F405RGT6, STM32F405RGT6:QFP50P1200X1200X160-64N
- R25: value 5k1 -> 1M
- R26: value 5k1 -> 100R
- R27: value 10k -> 0.05A; device resistor:R0603 -> rcl:R1210
- moved R26 226.4 mm to (1.50, -193.5), turned to 0 degrees
- moved R25 224.3 mm to (7.50, -193.5), turned to 0 degrees
- moved R27 218.6 mm to (3.00, -187.0), turned to 0 degrees
Connections:
- removed net BUS+: BSK4.4
- removed net I2CINT: BSK4.6, IC2.43
- removed net N$159: PWR.C, R82.2
- removed net N$161: IC2.41, R81.1
- removed net N$43: C4.2, U$21.P$3
- removed net N$44: C4.1, IC2.5
- removed net RX-C: IC2.31, USB-C.RX0
- removed net SCLTM: BSK4.8, IC2.45, R25.2
- removed net SDATM: BSK4.7, IC2.46, R26.2
- removed net SENS_O2: IC2.13, ME-O2.P$1
- removed net TX-C: IC2.30, USB-C.TX0
- removed net VDD: BSK4.2, C15.1, C16.1, C48.1, C53.1, C54.1, C55.1, IC2.1, IC2.24, IC2.36, IC2.48, IC2.9, ME-O2.P$7, PB5.A, PWR.A, R101.1, R102.1, R25.1, R26.1, R27.1, R64.1, R7.2, R79.1, R8.2, R9.2, USB-C.3V3/BUS0, USB-C.3V3/BUS1
- new net 4OXV: R26.1, U1.9
- new net BIPER: U1.21
- new net BME280: R19.1, U1.35
- new net CO: U1.16
- new net COMPR: U1.57
- new net CTRL-CO-1: U1.27
- new net CTRL-CO-2: U1.26
- new net CTRL-NH3-1: U1.45
- new net CTRL-NH3-2: U1.44
- new net CTRL-NO2-1: U1.23
- new net CTRL-NO2-2: U1.22
- new net GND-40XV: U$5.3
- new net GND-4OXV: R27.2
- new net GND-BME280: R20.2, U$3.3
- new net GND-MICS: R24.2, U$4.3
- new net GND-MS-EXT: R13.2, U$19.3
- new net GND-MS-INT: R30.2, U$7.3
- new net MICRO-CK: U1.34
- new net MICRO-SD: U1.62
- new net MICRO-WS: U1.36
- new net MICS: R23.1, U1.8
- new net MS5611-EXT: R31.1, U1.41
- new net MS5611-INT: R29.1, U1.33
- new net N$10: BSK1.8
- new net N$11: R22.1, R31.2, U$19.1
- new net N$12: R28.1, R29.2, U$7.1
- new net N$13: R30.1
- new net N$29: C13.2, U1.47
- new net N$3: BME280.P$2, R20.1
- new net N$36: C9.2, U1.31
- new net N$37: LED2.C, R15.2
- new net N$38: R15.1, U1.53
- new net N$4: C8.2, U$2.P$3
- new net N$40: LED3.C, R16.2
- new net N$5: C8.1, U1.5
- new net N$6: R21.1, R23.2, U$4.1
- new net N$7: R24.1
- new net N$8: R25.1, R26.2, U$5.1
- new net N$9: R27.1
- new net NH3: U1.15
- new net NO2: U1.14
- new net RX-O2: U1.43
- new net RX-S: U$6.RX0, U1.51
- new net SCL-TM: BSK1.5, U1.29
- new net SDA-TM: BSK1.6, U1.30
- new net SOUND: U1.10
- new net TX-O2: U1.42
- new net TX-S: U$6.TX0, U1.52
- new net VALVE: U1.61
- net 3V3: now also BSK1.1, C10.2, C18.2, C19.2, C2.2, C20.2, C3.2, C6.2, LED2.A, LED3.A, R10.2, R11.2, R12.2, R17.1, R18.1, R7.2, R8.2, R9.2, U$2.P$4, U$6.3V3/BUS0, U$6.3V3/BUS1, U1.1, U1.13, U1.19, U1.32, U1.48, U1.64; no longer C1.2, C5.2, U$18.P$4, U$21.P$4
- net 5V: now also BSK1.2, U$1.P$1, U$1.P$7; no longer BSK4.3
- net GND: now also BSK1.3, BSK1.4, C10.1, C13.1, C18.1, C19.1, C2.1, C20.1, C3.1, C6.1, C9.1, R14.2, R16.1, R21.2, R22.2, R25.2, R28.2, U$19.2, U$2.P$2, U$3.2, U$4.2, U$5.2, U$6.GND0, U$6.GND1, U$7.2, U1.12, U1.18, U1.28, U1.60, U1.63; no longer BME280.P$2, BSK4.1, C1.1, C15.2, C16.2, C48.2, C5.1, C53.2, C54.2, C55.2, IC2.20, IC2.23, IC2.35, IC2.44, IC2.47, IC2.8, ME-O2.P$4, R82.1, U$18.P$2, U$21.P$2, USB-C.GND0, USB-C.GND1
- net N$1: now also R13.1, U$1.P$3, U$1.P$6; no longer PB5.C, R81.2
- net N$2: now also R14.1, R19.2, U$3.1; no longer IC2.3, U$18.P$3
- net NRST: now also R10.1, U$6.NRST/EN, U1.7; no longer IC2.7, R79.2, USB-C.NRST/EN
- net SCL: now also R17.2, U$1.P$5, U1.58; no longer IC2.21, R101.2
- net SDA: now also R18.2, U$1.P$4, U1.59; no longer IC2.22, R102.2
- net SENS_CO: no longer IC2.12
- net SENS_CTL_CO_1: no longer IC2.19
- net SENS_CTL_CO_2: no longer IC2.18
- net SENS_CTL_NH3_1: no longer IC2.17
- net SENS_CTL_NH3_2: no longer IC2.16
- net SENS_CTL_NO2_1: no longer IC2.15
- net SENS_CTL_NO2_2: no longer IC2.14
- net SENS_NH3: no longer IC2.11
- net SENS_NO2: no longer IC2.10
- net SWC: now also R12.1, U$6.SWC/TXD, U1.49; no longer IC2.37, R27.2, USB-C.SWC/TXD
- net SWD: now also R11.1, U$6.SWD/RXD, U1.46; no longer IC2.34, R64.2, USB-C.SWD/RXD
- net TIME: now also BSK1.7, U1.50; no longer BSK4.5, IC2.42
Routing:
- net VDD: track 267.5 -> 0.00 mm, vias 13 -> 0
- net 3V3: track 0.00 -> 100.2 mm, vias 0 -> 9
- net NRST: track 47.8 -> 0.00 mm, vias 2 -> 0
- net GND: track 40.0 -> 0.00 mm, vias 3 -> 0
- net TX-C: track 34.0 -> 0.00 mm, vias 2 -> 0
- net SCLTM: track 31.8 -> 0.00 mm, vias 4 -> 0
- net SDATM: track 31.7 -> 0.00 mm
- net SENS_O2: track 30.6 -> 0.00 mm, vias 4 -> 0
- net RX-C: track 29.7 -> 0.00 mm, vias 2 -> 0
- net SWD: track 29.4 -> 0.00 mm, vias 2 -> 0
- net SWC: track 27.7 -> 0.00 mm, vias 2 -> 0
- net TIME: track 27.0 -> 0.00 mm
- net I2CINT: track 24.5 -> 0.00 mm
- net N$161: track 15.2 -> 0.00 mm
- net SENS_CTL_CO_1: track 22.5 -> 8.16 mm
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
Commit message: Добавлена схема дозиметра, исправлены платы СБ
Parts:
- removed MICS-6814: MICS-6814, CanCubeSat:MICS-6814
- added C1: 100nF, rcl:C0603
- added C4, C5: 22nF, rcl:C1210
- added C7: 100pF, rcl:C0603
- added D1, D2, D3, D4, D5: DIODE-MBR, CanCubeSat:SOD123
- added R32: 1M, resistor:R0603
- added R33: 100R, resistor:R0603
- added R34: 0.05A, rcl:R1210
- added R35: 100k, resistor:R0603
- added R36: 3k3, resistor:R0603
- added RT1, RT2: DS1820, CanCubeSat:TO92/TO226
- added U$10, U$11, U$12, U$13: BA159, CanCubeSat:BA159
- added U$14: ECAP, CanCubeSat:ECAP1MK
- added U$15: DOSIM, CanCubeSat:DOSIM
- added U$8: SI2302CDS, CanCubeSat:SOT23-3
- added U$9: 100µ, CanCubeSat:ECAP100-CMD
- added U2: LMC555CMX/NOPB, LMC555CMX_NOPB:SOIC127P599X175-8N
- added VR1: 3362H-1-502LF, CanCubeSat:TRIM_3362H-1-502LF
- R1: value 10k -> 0.5A; device resistor:R0603 -> rcl:R1210
- R2: value 10k -> 1k
- R3: value 10k -> 4k7
- R4: value 10k -> 22k
- R5, R6, R7, R8, R9: value 10k -> 1M
- moved R9 480.4 mm to (-23.5, -423.0), turned to 0 degrees
- moved R8 474.7 mm to (-23.5, -418.0), turned to 0 degrees
- moved R7 469.1 mm to (-23.5, -413.0), turned to 0 degrees
- moved R6 468.1 mm to (-23.5, -408.0), turned to 0 degrees
- moved R5 463.9 mm to (-23.5, -403.0), turned to 0 degrees
- moved R4 459.7 mm to (-23.5, -398.0), turned to 0 degrees
- moved R3 338.4 mm to (-15.0, -273.5), turned to 0 degrees
- moved R2 322.7 mm to (-6.50, -258.5), turned to 0 degrees
- moved R1 310.3 mm to (3.00, -247.0), turned to 0 degrees
- moved R24 60.0 mm to (3.00, -239.5)
Connections:
- removed net BIPER: U1.21
- removed net MICRO-CK: U1.34
- removed net MICRO-SD: U1.62
- removed net MICRO-WS: U1.36
- removed net SENS_CO: MICS-6814.P$5, R3.1
- removed net SENS_CTL_CO_1: R3.2, R6.1
- removed net SENS_CTL_CO_2: R6.2, R7.1
- removed net SENS_CTL_NH3_1: R2.2, R5.1
- removed net SENS_CTL_NH3_2: R5.2, R8.1
- removed net SENS_CTL_NO2_1: R1.2, R4.1
- removed net SENS_CTL_NO2_2: R4.2, R9.1
- removed net SENS_NH3: MICS-6814.P$4, R2.1
- removed net SENS_NO2: MICS-6814.P$3, R1.1
- removed net SOUND: U1.10
- new net DOS-G: C1.1, C5.2, D1.A, R34.1, R35.2, RT1.1, RT2.1, U$10.P$1, U$14.P$2, U$9.P$1, U2.1
- new net DOSE: C7.2, R36.2, RT2.3, U1.34
- new net DOSIM: R33.1, U1.10
- new net GND-DOSIM: R34.2, U$8.3
- new net GND-OUT: BSK1.3, BSK1.4, R1.2
- new net N$14: R32.1, R33.2, U$8.1
- new net N$15: C1.2, R2.1, U2.2, U2.6
- new net N$16: R2.2, VR1.2, VR1.3
- new net N$17: R3.2, U2.3, VR1.1
- new net N$18: R3.1, RT1.2
- new net N$19: C4.1, RT1.3, U$10.P$2, U$11.P$1
- new net N$20: C5.1, U$11.P$2, U$12.P$1
- new net N$21: C4.2, U$12.P$2, U$13.P$1
- new net N$22: R4.2, R5.2, U$13.P$2, U$14.P$1
- new net N$23: D1.C, D2.A
- new net N$24: D2.C, D3.A
- new net N$25: D3.C, D4.A
- new net N$26: D4.C, D5.A
- new net N$27: D5.C, R4.1
- new net N$28: R5.1, R6.1
- new net N$30: R6.2, R7.2
- new net N$31: R7.1, R8.1
- new net N$32: R8.2, R9.2
- new net N$33: R9.1, U$15.P$1
- new net N$34: C7.1, R35.1, RT2.2, U$15.P$2
- net 3V3: no longer R7.2, R8.2, R9.2
- net 5V: now also R36.1, U$9.P$2, U2.4, U2.8; no longer MICS-6814.P$1
- net GND: now also R1.1, R32.2, U$8.2; no longer BSK1.3, BSK1.4, MICS-6814.P$2
Routing:
- net 5V: track 119.3 -> 13.5 mm
- net 3V3: track 100.2 -> 0.00 mm, vias 9 -> 0
- net SENS_NH3: track 35.9 -> 0.00 mm, vias 1 -> 0
- net SENS_CO: track 35.9 -> 0.00 mm, vias 1 -> 0
- net SENS_NO2: track 33.1 -> 0.00 mm, vias 2 -> 0
- net SENS_CTL_NO2_1: track 25.8 -> 0.00 mm
- net SENS_CTL_NH3_1: track 22.1 -> 0.00 mm
- net SENS_CTL_NO2_2: track 21.9 -> 0.00 mm
- net SENS_CTL_NH3_2: track 18.1 -> 0.00 mm
- net SENS_CTL_CO_1: track 8.16 -> 0.00 mm
- net SENS_CTL_CO_2: track 7.66 -> 0.00 mm
