File: schematics/board/PLnew.sch (EAGLE design)
At the start: 39 parts, among them IC2 STM32F103C8T, Q5 8MHz

Commit message: плата БСК5
Parts:
- removed C005R: 32,768KHz, CanCubeSat:C005R
- removed C44, C45: 27pF, rcl:C-EUC0603
- removed C46, C47: 10pF, rcl:C-EUC0603
- removed Q5: 8MHz, 9C-8.000MEEJ-T:9C-8.000MEEJ-T
- removed R78: 1M, resistor:R-US_R0603
- added C1, C5: 10nF, rcl:C-EUC0603
- added C4: 1nF, rcl:C-EUC0603
- added U$18: Q32.768, CanCubeSat:Q32.768
- added U$21: Q24, CanCubeSat:Q24
Connections:
- removed net N$133: C44.1, IC2.OSC_OUT, Q5.1, R78.1
- removed net N$145: C45.1, IC2.OSC_IN, Q5.2, R78.2
- removed net N$148: C005R.2, C47.1, IC2.PC15
- removed net N$152: C005R.1, C46.1, IC2.PC14
- new net 3V3: C1.2, C5.2, U$18.VCC, U$21.VCC
- new net N$2: IC2.PC14, U$18.OUTPUT
- new net N$43: C4.2, U$21.OUTPUT
- new net N$44: C4.1, IC2.OSC_IN
- net GND: now also C1.1, C5.1, U$18.GND, U$21.GND; no longer C44.2, C45.2, C46.2, C47.2

Commit message: Две линии i2c на платах БСК заменены на одну
Parts:
- removed BSK4: (no value), pinheadCS:PINHD-1X8
- removed C1, C5: 10nF, rcl:C-EUC0603
- removed C15, C48, C53, C54, C55: 100nF, rcl:C-EUC0603
- removed C16: 10µ, rcl:C-USC1206
- removed C4: 1nF, rcl:C-EUC0603
- removed IC2: STM32F103C8T, CanCubeSat:STM32F103C8T
- removed ME-O2: ME-O2, CanCubeSat:ME-O2
- removed PB5, PWR: (no value), led:LEDCHIPLED_0603
- removed R101, R102: 5k1, resistor:R-US_R0603
- removed R64, R79: 10k, resistor:R-US_R0603
- removed R81, R82: 2k, resistor:R-US_R0603
- removed U$18: Q32.768, CanCubeSat:Q32.768
- removed U$21: Q24, CanCubeSat:Q24
- removed USB-C: USB-C, CanCubeSat:USB-C
- added BSK1: (no value), pinheadCS:PINHD-2X4
- added C10: 10nF, rcl:C-EUC0603
- added C13, C9: 2,2µ, rcl:C-USC0603
- added C18, C2, C20, C3, C6: 100nF, rcl:C-EUC0603
- added C19: 10µ, rcl:C-USC1206
- added C8: 1nF, rcl:C-EUC0603
- added LED2, LED3: (no value), led:LEDCHIPLED_0603
- added R10, R11, R12: 10k, resistor:R-US_R0603
- added R13, R20, R24, R30: 0.05A, rcl:R-EU_R1210
- added R14, R21, R22, R28: 1M, resistor:R-US_R0603
- added R15, R16: 2k, resistor:R-US_R0603
- added R17, R18: 5k1, resistor:R-US_R0603
- added R19, R23, R29, R31: 100R, resistor:R-US_R0603
- added U$1: MS5611, CanCubeSat:MS5611
- added U$19, U$3, U$4, U$5, U$7: SI2302CDS, CanCubeSat:SI2302CDS
- added U$2: Q24, CanCubeSat:Q24
- added U$6: USB-C, CanCubeSat:USB-C
- added U1: STM32F405RGT6, STM32F405RGT6:STM32F405RGT6
- R25: value 5k1 -> 1M
- R26: value 5k1 -> 100R
- R27: value 10k -> 0.05A; device resistor:R-US_R0603 -> rcl:R-EU_R1210
Connections:
- removed net BUS+: BSK4.4
- removed net I2CINT: BSK4.6, IC2.PB7
- removed net N$159: PWR.C, R82.2
- removed net N$161: IC2.PB5, R81.1
- removed net N$43: C4.2, U$21.OUTPUT
- removed net N$44: C4.1, IC2.OSC_IN
- removed net RX-C: IC2.PA10, USB-C.RX0
- removed net SCLTM: BSK4.8, IC2.PB8, R25.2
- removed net SDATM: BSK4.7, IC2.PB9, R26.2
- removed net SENS_O2: IC2.PA3, ME-O2.SIG
- removed net TX-C: IC2.PA9, USB-C.TX0
- removed net VDD: BSK4.2, C15.1, C16.1, C48.1, C53.1, C54.1, C55.1, IC2.VBAT, IC2.VDDA, ME-O2.3V3, PB5.A, PWR.A, R101.1, R102.1, R25.1, R26.1, R27.1, R64.1, R7.2, R79.1, R8.2, R9.2, USB-C.3V3/BUS
- new net 4OXV: R26.1, U1.PC1
- new net BIPER: U1.PA5/SPI1_SCK
- new net BME280: R19.1, U1.PB14
- new net CO: U1.PA2/USART2_TX
- new net COMPR: U1.PB5
- new net CTRL-CO-1: U1.PB1
- new net CTRL-CO-2: U1.PB0
- new net CTRL-NH3-1: U1.PA12
- new net CTRL-NH3-2: U1.PA11
- new net CTRL-NO2-1: U1.PA7/SPI1_MOSI
- new net CTRL-NO2-2: U1.PA6/SPI1_MISO
- new net GND-40XV: U$5.D
- new net GND-4OXV: R27.2
- new net GND-BME280: R20.2, U$3.D
- new net GND-MICS: R24.2, U$4.D
- new net GND-MS-EXT: R13.2, U$19.D
- new net GND-MS-INT: R30.2, U$7.D
- new net MICRO-CK: U1.PB13
- new net MICRO-SD: U1.PB9
- new net MICRO-WS: U1.PB15
- new net MICS: R23.1, U1.PC0
- new net MS5611-EXT: R31.1, U1.PA8
- new net MS5611-INT: R29.1, U1.PB12
- new net N$10: BSK1.8
- new net N$11: R22.1, R31.2, U$19.G
- new net N$12: R28.1, R29.2, U$7.G
- new net N$13: R30.1
- new net N$29: C13.2, U1.VCAP_2
- new net N$3: BME280.GND, R20.1
- new net N$36: C9.2, U1.VCAP_1
- new net N$37: LED2.C, R15.2
- new net N$38: R15.1, U1.PC12
- new net N$4: C8.2, U$2.OUTPUT
- new net N$40: LED3.C, R16.2
- new net N$5: C8.1, U1.PH0/OSC_IN
- new net N$6: R21.1, R23.2, U$4.G
- new net N$7: R24.1
- new net N$8: R25.1, R26.2, U$5.G
- new net N$9: R27.1
- new net NH3: U1.PA1/USART2_RTS
- new net NO2: U1.PA0/WKUP
- new net RX-O2: U1.PA10
- new net RX-S: U$6.RX0, U1.PC10
- new net SCL-TM: BSK1.5, U1.PB10
- new net SDA-TM: BSK1.6, U1.PB11
- new net SOUND: U1.PC2/SPI2_MISO
- new net TX-O2: U1.PA9
- new net TX-S: U$6.TX0, U1.PC11
- new net VALVE: U1.PB8
- net 3V3: now also BSK1.1, C10.2, C18.2, C19.2, C2.2, C20.2, C3.2, C6.2, LED2.A, LED3.A, R10.2, R11.2, R12.2, R17.1, R18.1, R7.2, R8.2, R9.2, U$2.VCC, U$6.3V3/BUS, U1.VBAT, U1.VDD, U1.VDDA; no longer C1.2, C5.2, U$18.VCC, U$21.VCC
- net 5V: now also BSK1.2, U$1.PS, U$1.VCC; no longer BSK4.3
- net GND: now also BSK1.3, BSK1.4, C10.1, C13.1, C18.1, C19.1, C2.1, C20.1, C3.1, C6.1, C9.1, R14.2, R16.1, R21.2, R22.2, R25.2, R28.2, U$19.S, U$2.GND, U$3.S, U$4.S, U$5.S, U$6.GND, U$7.S, U1.BOOT0, U1.PB2/BOOT1, U1.VSS, U1.VSSA; no longer BME280.GND, BSK4.1, C1.1, C15.2, C16.2, C48.2, C5.1, C53.2, C54.2, C55.2, IC2.BOOT0, IC2.PB2, IC2.VSSA, ME-O2.GND, R82.1, U$18.GND, U$21.GND, USB-C.GND
- net N$1: now also R13.1, U$1.CSB, U$1.GND; no longer PB5.C, R81.2
- net N$2: now also R14.1, R19.2, U$3.G; no longer IC2.PC14, U$18.OUTPUT
- net NRST: now also R10.1, U$6.NRST/EN, U1.NRST; no longer IC2.NRST, R79.2, USB-C.NRST/EN
- net SCL: now also R17.2, U$1.SCL, U1.PB6; no longer IC2.PB10, R101.2
- net SDA: now also R18.2, U$1.SDA, U1.PB7; no longer IC2.PB11, R102.2
- net SENS_CO: no longer IC2.PA2
- net SENS_CTL_CO_1: no longer IC2.PB1
- net SENS_CTL_CO_2: no longer IC2.PB0
- net SENS_CTL_NH3_1: no longer IC2.PA7
- net SENS_CTL_NH3_2: no longer IC2.PA6
- net SENS_CTL_NO2_1: no longer IC2.PA5
- net SENS_CTL_NO2_2: no longer IC2.PA4
- net SENS_NH3: no longer IC2.PA1
- net SENS_NO2: no longer IC2.PA0-WKUP
- net SWC: now also R12.1, U$6.SWC/TXD, U1.PA14/JTCK-SWCLK; no longer IC2.PA14, R27.2, USB-C.SWC/TXD
- net SWD: now also R11.1, U$6.SWD/RXD, U1.PA13/JMS-SWDIO; no longer IC2.PA13, R64.2, USB-C.SWD/RXD
- net TIME: now also BSK1.7, U1.PA15; no longer BSK4.5, IC2.PB6
Other:
- moved on the sheet: BME280, MICS-6814, R1, R2, R25, R26, R3, R4, R5, R6, R7, R8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

Commit message: Добавлена схема дозиметра, исправлены платы СБ
Parts:
- removed MICS-6814: MICS-6814, CanCubeSat:MICS-6814
- added C1: 100nF, rcl:C-EUC0603
- added C4, C5: 22nF, rcl:C-EUC1210
- added C7: 100pF, rcl:C-EUC0603
- added D1, D2, D3, D4, D5: DIODE-MBR, CanCubeSat:DIODE-MBR
- added R32: 1M, resistor:R-US_R0603
- added R33: 100R, resistor:R-US_R0603
- added R34: 0.05A, rcl:R-EU_R1210
- added R35: 100k, resistor:R-US_R0603
- added R36: 3k3, resistor:R-US_R0603
- added RT1, RT2: DS1820, CanCubeSat:DS1820
- added U$10, U$11, U$12, U$13: BA159, CanCubeSat:BA159
- added U$14: ECAP, CanCubeSat:ECAP
- added U$15: DOSIM, CanCubeSat:DOSIM
- added U$8: SI2302CDS, CanCubeSat:SI2302CDS
- added U$9: 100µ, CanCubeSat:ECAPECAP100
- added U2: LMC555CMX/NOPB, LMC555CMX_NOPB:LMC555CMX/NOPB
- added VR1: 3362H-1-502LF, CanCubeSat:3362H-1-502LF
- R1: value 10k -> 0.5A; device resistor:R-US_R0603 -> rcl:R-EU_R1210
- R2: value 10k -> 1k
- R3: value 10k -> 4k7
- R4: value 10k -> 22k
- R5, R6, R7, R8, R9: value 10k -> 1M
Connections:
- removed net BIPER: U1.PA5/SPI1_SCK
- removed net MICRO-CK: U1.PB13
- removed net MICRO-SD: U1.PB9
- removed net MICRO-WS: U1.PB15
- removed net SENS_CO: MICS-6814.CO, R3.1
- removed net SENS_CTL_CO_1: R3.2, R6.1
- removed net SENS_CTL_CO_2: R6.2, R7.1
- removed net SENS_CTL_NH3_1: R2.2, R5.1
- removed net SENS_CTL_NH3_2: R5.2, R8.1
- removed net SENS_CTL_NO2_1: R1.2, R4.1
- removed net SENS_CTL_NO2_2: R4.2, R9.1
- removed net SENS_NH3: MICS-6814.NH3, R2.1
- removed net SENS_NO2: MICS-6814.NO2, R1.1
- removed net SOUND: U1.PC2/SPI2_MISO
- new net DOS-G: C1.1, C5.2, D1.A, R34.1, R35.2, RT1.GND, RT2.GND, U$10.A, U$14.2, U$9.1, U2.GND
- new net DOSE: C7.2, R36.2, RT2.VDD, U1.PB13
- new net DOSIM: R33.1, U1.PC2/SPI2_MISO
- new net GND-DOSIM: R34.2, U$8.D
- new net GND-OUT: BSK1.3, BSK1.4, R1.2
- new net N$14: R32.1, R33.2, U$8.G
- new net N$15: C1.2, R2.1, U2.!TRIGGER!, U2.THRESHOLD
- new net N$16: R2.2, VR1.CW, VR1.WIPER
- new net N$17: R3.2, U2.OUTPUT, VR1.CCW
- new net N$18: R3.1, RT1.DQ
- new net N$19: C4.1, RT1.VDD, U$10.C, U$11.A
- new net N$20: C5.1, U$11.C, U$12.A
- new net N$21: C4.2, U$12.C, U$13.A
- new net N$22: R4.2, R5.2, U$13.C, U$14.1
- new net N$23: D1.C, D2.A
- new net N$24: D2.C, D3.A
- new net N$25: D3.C, D4.A
- new net N$26: D4.C, D5.A
- new net N$27: D5.C, R4.1
- new net N$28: R5.1, R6.1
- new net N$30: R6.2, R7.2
- new net N$31: R7.1, R8.1
- new net N$32: R8.2, R9.2
- new net N$33: R9.1, U$15.+
- new net N$34: C7.1, R35.1, RT2.DQ, U$15.-
- net 3V3: no longer R7.2, R8.2, R9.2
- net 5V: now also R36.1, U$9.2, U2.!RESET!, U2.V+; no longer MICS-6814.5V
- net GND: now also R1.1, R32.2, U$8.S; no longer BSK1.3, BSK1.4, MICS-6814.GND
Other:
- moved on the sheet: R2, R3, R4, R5, R6, R7, R8, R9
