File: schematics/board/PL.sch (EAGLE design)
At the start: 39 parts, among them IC2 STM32F103C8T, Q5 8MHz

Commit message: Папка с платами
Connections:
- net 5V: now also BSK4.3; no longer BSK4.8
- net BUS+: now also BSK4.4; no longer BSK4.7
- net I2CINT: now also BSK4.6; no longer BSK4.3
- net SCLTM: now also BSK4.8; no longer BSK4.5
- net SDATM: now also BSK4.7; no longer BSK4.4
- net TIME: now also BSK4.5; no longer BSK4.2
- net VDD: now also BSK4.2; no longer BSK4.6
Changed lines of the file:
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@@
 <layer number="54" name="bGND_GNDA" color="1" fill="9" visible="no" active="no"/>
 <layer number="56" name="wert" color="7" fill="1" visible="no" active="no"/>
+<layer number="57" name="tCAD" color="7" fill="1" visible="no" active="no"/>
+<layer number="59" name="tCarbon" color="7" fill="1" visible="no" active="no"/>
+<layer number="60" name="bCarbon" color="7" fill="1" visible="no" active="no"/>
 <layer number="88" name="SimResults" color="9" fill="1" visible="yes" active="yes"/>
 <layer number="89" name="SimProbes" color="9" fill="1" visible="yes" active="yes"/>
@@
 <layer number="112" name="tSilk" color="7" fill="1" visible="no" active="no"/>
 <layer number="113" name="IDFDebug" color="7" fill="1" visible="no" active="yes"/>
+<layer number="114" name="Badge_Outline" color="7" fill="1" visible="no" active="no"/>
+<layer number="115" name="ReferenceISLANDS" color="7" fill="1" visible="no" active="no"/>
 <layer number="116" name="Patch_BOT" color="9" fill="4" visible="no" active="no"/>
 <layer number="118" name="Rect_Pads" color="7" fill="1" visible="no" active="no"/>
@@
 <layer number="127" name="_tValues" color="7" fill="1" visible="no" active="no"/>
 <layer number="128" name="_bValues" color="7" fill="1" visible="no" active="no"/>
+<layer number="129" name="Mask" color="7" fill="1" visible="no" active="no"/>
 <layer number="131" name="tAdjust" color="7" fill="1" visible="no" active="no"/>
 <layer number="132" name="bAdjust" color="7" fill="1" visible="no" active="no"/>
 <layer number="144" name="DrillLegend" color="7" fill="1" visible="no" active="no"/>
+<layer number="150" name="Notes" color="7" fill="1" visible="no" active="no"/>
 <layer number="151" name="HeatSink" color="14" fill="1" visible="no" active="no"/>
 <layer number="152" name="_bDocu" color="7" fill="1" visible="no" active="no"/>
+<layer number="153" name="FabDoc1" color="7" fill="1" visible="no" active="no"/>
+<layer number="154" name="FabDoc2" color="7" fill="1" visible="no" active="no"/>
+<layer number="155" name="FabDoc3" color="7" fill="1" visible="no" active="no"/>
 <layer number="199" name="Contour" color="7" fill="1" visible="no" active="no"/>
 <layer number="200" name="200bmp" color="1" fill="10" visible="no" active="no"/>
@@
 <layer number="227" name="227bmp" color="7" fill="1" visible="no" active="yes"/>
 <layer number="228" name="228bmp" color="7" fill="1" visible="no" active="yes"/>
+<layer number="229" name="229bmp" color="7" fill="1" visible="no" active="no"/>
 <layer number="230" name="230bmp" color="7" fill="1" visible="no" active="yes"/>
+<layer number="231" name="231bmp" color="7" fill="1" visible="no" active="no"/>
+<layer number="232" name="Eagle3D_PG2" color="7" fill="1" visible="no" active="no"/>
+<layer number="233" name="Eagle3D_PG3" color="7" fill="1" visible="no" active="no"/>
 <layer number="248" name="Housing" color="7" fill="1" visible="no" active="no"/>
 <layer number="249" name="Edge" color="7" fill="1" visible="no" active="no"/>
@@
 <layer number="251" name="SMDround" color="7" fill="1" visible="no" active="yes"/>
 <layer number="254" name="OrgLBR" color="13" fill="1" visible="no" active="no"/>
+<layer number="255" name="routoute" color="7" fill="1" visible="no" active="no"/>
 </layers>
 <schematic xreflabel="%F%N/%S.%C%R" xrefpart="/%S.%C%R">
@@
 </segment>
 <segment>
-<wire x1="-17.78" y1="160.02" x2="-17.78" y2="172.72" width="0.1524" layer="91"/>
-<pinref part="BSK4" gate="A" pin="6"/>
-<label x="-17.78" y="165.1" size="1.778" layer="95" rot="R90"/>
-</segment>
-<segment>
 <wire x1="60.96" y1="147.32" x2="50.8" y2="147.32" width="0.1524" layer="91"/>
 <label x="50.8" y="147.32" size="1.778" layer="95"/>
@@
 <label x="-12.7" y="35.56" size="1.778" layer="95"/>
 </segment>
+<segment>
+<wire x1="-7.62" y1="160.02" x2="-7.62" y2="172.72" width="0.1524" layer="91"/>
+<pinref part="BSK4" gate="A" pin="2"/>
+<label x="-7.62" y="165.1" size="1.778" layer="95" rot="R90"/>
+</segment>
 </net>
 <net name="N$133" class="0">
@@
 <net name="SDATM" class="0">
 <segment>
-<wire x1="-12.7" y1="160.02" x2="-12.7" y2="172.72" width="0.1524" layer="91"/>
-<pinref part="BSK4" gate="A" pin="4"/>
-<label x="-12.7" y="165.1" size="1.778" layer="95" rot="R90"/>
-</segment>
-<segment>
 <wire x1="152.4" y1="88.9" x2="152.4" y2="66.04" width="0.1524" layer="91"/>
 <label x="152.4" y="81.28" size="1.778" layer="95" rot="R90"/>
@@
 <pinref part="R26" gate="G$1" pin="2"/>
 </segment>
+<segment>
+<wire x1="-20.32" y1="160.02" x2="-20.32" y2="172.72" width="0.1524" layer="91"/>
+<pinref part="BSK4" gate="A" pin="7"/>
+<label x="-20.32" y="165.1" size="1.778" layer="95" rot="R90"/>
+</segment>
 </net>
 <net name="SCLTM" class="0">
-<segment>
-<wire x1="-15.24" y1="160.02" x2="-15.24" y2="172.72" width="0.1524" layer="91"/>
-<pinref part="BSK4" gate="A" pin="5"/>
-<label x="-15.24" y="165.1" size="1.778" layer="95" rot="R90"/>
-</segment>
 <segment>
 <wire x1="149.86" y1="88.9" x2="149.86" y2="66.04" width="0.1524" layer="91"/>
@@
 <pinref part="R25" gate="G$1" pin="2"/>
 </segment>
-</net>
-<net name="5V" class="0">
 <segment>
 <wire x1="-22.86" y1="160.02" x2="-22.86" y2="172.72" width="0.1524" layer="91"/>
@@
 <label x="-22.86" y="165.1" size="1.778" layer="95" rot="R90"/>
 </segment>
+</net>
+<net name="5V" class="0">
 <segment>
 <pinref part="MICS-6814" gate="G$1" pin="5V"/>
@@
 <label x="15.24" y="-68.58" size="1.778" layer="95"/>
 </segment>
+<segment>
+<wire x1="-10.16" y1="160.02" x2="-10.16" y2="172.72" width="0.1524" layer="91"/>
+<pinref part="BSK4" gate="A" pin="3"/>
+<label x="-10.16" y="165.1" size="1.778" layer="95" rot="R90"/>
+</segment>
 </net>
 <net name="TIME" class="0">
-<segment>
-<wire x1="-7.62" y1="160.02" x2="-7.62" y2="172.72" width="0.1524" layer="91"/>
-<pinref part="BSK4" gate="A" pin="2"/>
-<label x="-7.62" y="165.1" size="1.778" layer="95" rot="R90"/>
-</segment>
 <segment>
 <wire x1="144.78" y1="88.9" x2="144.78" y2="81.28" width="0.1524" layer="91"/>
@@
 <pinref part="IC2" gate="MCU" pin="PB6"/>
 </segment>
+<segment>
+<wire x1="-15.24" y1="160.02" x2="-15.24" y2="172.72" width="0.1524" layer="91"/>
+<pinref part="BSK4" gate="A" pin="5"/>
+<label x="-15.24" y="165.1" size="1.778" layer="95" rot="R90"/>
+</segment>
 </net>
 <net name="I2CINT" class="0">
-<segment>
-<wire x1="-10.16" y1="160.02" x2="-10.16" y2="172.72" width="0.1524" layer="91"/>
-<pinref part="BSK4" gate="A" pin="3"/>
-<label x="-10.16" y="165.1" size="1.778" layer="95" rot="R90"/>
-</segment>
 <segment>
 <wire x1="147.32" y1="88.9" x2="147.32" y2="81.28" width="0.1524" layer="91"/>
@@
 <pinref part="IC2" gate="MCU" pin="PB7"/>
 </segment>
+<segment>
+<wire x1="-17.78" y1="160.02" x2="-17.78" y2="172.72" width="0.1524" layer="91"/>
+<pinref part="BSK4" gate="A" pin="6"/>
+<label x="-17.78" y="165.1" size="1.778" layer="95" rot="R90"/>
+</segment>
 </net>
 <net name="BUS+" class="0">
 <segment>
-<wire x1="-20.32" y1="160.02" x2="-20.32" y2="172.72" width="0.1524" layer="91"/>
-<pinref part="BSK4" gate="A" pin="7"/>
-<label x="-20.32" y="165.1" size="1.778" layer="95" rot="R90"/>
-</segment>
-</net>
+<wire x1="-12.7" y1="160.02" x2="-12.7" y2="172.72" width="0.1524" layer="91"/>
+<pinref part="BSK4" gate="A" pin="4"/>
+<label x="-12.7" y="165.1" size="1.778" layer="95" rot="R90"/>
+</segment>
+</net>

Commit message: Обновлен список плат, работа над платой ПН
Parts:
- removed BSK4: (no value), pinheadCS:PINHD-1X8
- removed C005R: 32,768KHz, CanCubeSat:C005R
- removed C15, C48, C53, C54, C55: 100nF, rcl:C-EUC0603
- removed C16: 10µ, rcl:C-USC1206
- removed C44, C45: 27pF, rcl:C-EUC0603
- removed C46, C47: 10pF, rcl:C-EUC0603
- removed IC2: STM32F103C8T, CanCubeSat:STM32F103C8T
- removed ME-O2: ME-O2, CanCubeSat:ME-O2
- removed MICS-6814: MICS-6814, CanCubeSat:MICS-6814
- removed PB5, PWR: (no value), led:LEDCHIPLED_0603
- removed Q5: 8MHz, 9C-8.000MEEJ-T:9C-8.000MEEJ-T
- removed R101, R102: 5k1, resistor:R-US_R0603
- removed R64, R79: 10k, resistor:R-US_R0603
- removed R78: 1M, resistor:R-US_R0603
- removed R81, R82: 2k, resistor:R-US_R0603
- removed USB-C: USB-C, CanCubeSat:USB-C
- added 2N6517, BC546: DS1820, CanCubeSat:DS1820
- added BSK1: (no value), pinheadCS:PINHD-2X5
- added C1, C18, C2, C20, C3, C6: 100nF, rcl:C-EUC0603
- added C10: 10nF, rcl:C-EUC0603
- added C13, C9: 2,2µ, rcl:C-USC0603
- added C19: 10µ, rcl:C-USC1206
- added C4, C5: 22nF, rcl:C-EUC1210
- added C7: 100pF, rcl:C-EUC0603
- added C8: 1nF, rcl:C-EUC0603
- added COMPR, HEAT, TEMP, VALVE1, VALVE2: (no value), pinheadCS:PINHD-1X2
- added D1, D2, D3, D4, D5: DIODE-MBR, CanCubeSat:DIODE-MBR
- added LED2, LED3: (no value), led:LEDCHIPLED_0603
- added R10, R11, R12, R37, R38, R39, R40, R41, R42, R43, R44, R45: 10k, resistor:R-US_R0603
- added R13, R20, R24, R30, R34, R48: 0.05A, rcl:R-EU_R1210
- added R14, R21, R22, R28, R32, R46, R49, R53, R55: 1M, resistor:R-US_R0603
- added R15, R16: 2k, resistor:R-US_R0603
- added R17, R18: 5k1, resistor:R-US_R0603
- added R19, R23, R29, R31, R33, R47, R50, R54, R56: 100R, resistor:R-US_R0603
- added R35: 100k, resistor:R-US_R0603
- added R36: 3k3, resistor:R-US_R0603
- added R51: 124k, resistor:R-US_R0603
- added R52: 22k, resistor:R-US_R0603
- added U$1: MS5611, CanCubeSat:MS5611
- added U$10, U$11, U$12, U$13: BA159, CanCubeSat:BA159
- added U$14: ECAP, CanCubeSat:ECAP
- added U$15: DOSIM, CanCubeSat:DOSIM
- added U$16, U$21: FFC-CONNECT68611, CanCubeSat:FFC-CONNECT68611
- added U$17: 33mH, CanCubeSat:RCH114NPRCH114NP
- added U$18, U$19, U$20, U$22, U$23, U$3, U$4, U$5, U$7, U$8: SI2302CDS, CanCubeSat:SI2302CDS
- added U$2: Q24, CanCubeSat:Q24
- added U$9: 100µ, CanCubeSat:ECAPECAP100
- added U1: STM32F405RGT6, STM32F405RGT6:STM32F405RGT6
- added U2: LMC555CMX/NOPB, LMC555CMX_NOPB:LMC555CMX/NOPB
- added VR1: 3362H-1-502LF, CanCubeSat:3362H-1-502LF
- R1: value 10k -> 0.5A; device resistor:R-US_R0603 -> rcl:R-EU_R1210
- R2: value 10k -> 1k
- R25: value 5k1 -> 1M
- R26: value 5k1 -> 100R
- R27: value 10k -> 0.05A; device resistor:R-US_R0603 -> rcl:R-EU_R1210
- R3: value 10k -> 4k7
- R4: value 10k -> 22k
- R5, R6, R7, R8, R9: value 10k -> 1M
Connections:
- removed net I2CINT: BSK4.6, IC2.PB7
- removed net N$133: C44.1, IC2.OSC_OUT, Q5.1, R78.1
- removed net N$145: C45.1, IC2.OSC_IN, Q5.2, R78.2
- removed net N$148: C005R.2, C47.1, IC2.PC15
- removed net N$152: C005R.1, C46.1, IC2.PC14
- removed net N$159: PWR.C, R82.2
- removed net N$161: IC2.PB5, R81.1
- removed net RX-C: IC2.PA10, USB-C.RX0
- removed net SCLTM: BSK4.8, IC2.PB8, R25.2
- removed net SDATM: BSK4.7, IC2.PB9, R26.2
- removed net SENS_CO: IC2.PA2, MICS-6814.CO, R3.1
- removed net SENS_CTL_CO_1: IC2.PB1, R3.2, R6.1
- removed net SENS_CTL_CO_2: IC2.PB0, R6.2, R7.1
- removed net SENS_CTL_NH3_1: IC2.PA7, R2.2, R5.1
- removed net SENS_CTL_NH3_2: IC2.PA6, R5.2, R8.1
- removed net SENS_CTL_NO2_1: IC2.PA5, R1.2, R4.1
- removed net SENS_CTL_NO2_2: IC2.PA4, R4.2, R9.1
- removed net SENS_NH3: IC2.PA1, MICS-6814.NH3, R2.1
- removed net SENS_NO2: IC2.PA0-WKUP, MICS-6814.NO2, R1.1
- removed net SENS_O2: IC2.PA3, ME-O2.SIG
- removed net TX-C: IC2.PA9, USB-C.TX0
- removed net VDD: BSK4.2, C15.1, C16.1, C48.1, C53.1, C54.1, C55.1, IC2.VBAT, IC2.VDDA, ME-O2.3V3, PB5.A, PWR.A, R101.1, R102.1, R25.1, R26.1, R27.1, R64.1, R7.2, R79.1, R8.2, R9.2, USB-C.3V3/BUS
- new net 3V3: BSK1.3, C10.2, C18.2, C19.2, C2.2, C20.2, C3.2, C6.2, LED2.A, LED3.A, R10.2, R11.2, R12.2, R17.1, R18.1, R43.2, R44.2, R45.2, R52.2, U$2.VCC, U$21.1, U$21.2, U1.VBAT, U1.VDD, U1.VDDA
- new net 4OXV: R26.1, U1.PC1
- new net BME280-EXT: R19.1, U1.PB14
- new net BME280-INT: R47.1, U1.PB13
- new net CO: R39.1, U$16.7, U1.PA2/USART2_TX
- new net COMPR: R54.1, U1.PB5
- new net CTRL-CO-1: R39.2, R42.1, U1.PB1
- new net CTRL-CO-2: R42.2, R43.1, U1.PB0
- new net CTRL-NH3-1: R38.2, R41.1, U1.PA12
- new net CTRL-NH3-2: R41.2, R44.1, U1.PA11
- new net CTRL-NO2-1: R37.2, R40.1, U1.PA7/SPI1_MOSI
- new net CTRL-NO2-2: R40.2, R45.1, U1.PA6/SPI1_MISO
- new net DOS-G: 2N6517.GND, BC546.GND, C1.1, C5.2, D1.A, R34.1, R35.2, U$10.A, U$14.2, U$9.1, U2.GND
- new net DOSE: BC546.VDD, C7.2, R36.2
- new net DOSIM: R33.1, U1.PC2/SPI2_MISO
- new net G-4OXV: R27.1, U$16.2
- new net G-BME: R48.1, U$16.14
- new net G-MICS: R24.1, U$16.6
- new net G-MS: R30.1, U$16.11
- new net GND-40XV: U$5.D
- new net GND-4OXV: R27.2
- new net GND-BME-EXT: R20.2, U$3.D
- new net GND-BME-INT: R48.2, U$18.D
- new net GND-COMPR: COMPR.2, U$22.D
- new net GND-DOSIM: R34.2, U$8.D
- new net GND-HEAT: HEAT.2, U$23.D
- new net GND-MICS: R24.2, U$4.D
- new net GND-MS-EXT: R13.2, U$19.D
- new net GND-MS-INT: R30.2, U$7.D
- new net GND-OUT: BSK1.5, BSK1.6, R1.2
- new net GND-VALVE: U$20.D, VALVE1.2, VALVE2.2
- new net HEAT: R56.1, U1.PC3/SPI2_MOSI
- new net MICS: R23.1, U1.PC0
- new net MS5611-EXT: R31.1, U1.PA8
- new net MS5611-INT: R29.1, U1.PB12
- new net N$10: R46.1, R47.2, U$18.G
- new net N$11: R22.1, R31.2, U$19.G
- new net N$12: R28.1, R29.2, U$7.G
- new net N$14: R32.1, R33.2, U$8.G
- new net N$15: C1.2, R2.1, U2.!TRIGGER!, U2.THRESHOLD
- new net N$16: R2.2, VR1.CW, VR1.WIPER
- new net N$17: R3.2, U2.OUTPUT, VR1.CCW
- new net N$18: 2N6517.DQ, R3.1
- new net N$19: 2N6517.VDD, C4.1, U$10.C, U$11.A, U$17.2
- new net N$2: R14.1, R19.2, U$3.G
- new net N$20: C5.1, U$11.C, U$12.A
- new net N$21: C4.2, U$12.C, U$13.A
- new net N$22: R4.2, R5.2, U$13.C, U$14.1
- new net N$23: D1.C, D2.A
- new net N$24: D2.C, D3.A
- new net N$25: D3.C, D4.A
- new net N$26: D4.C, D5.A
- new net N$27: D5.C, R4.1
- new net N$28: R5.1, R6.1
- new net N$29: C13.2, U1.VCAP_2
- new net N$3: BME280.GND, R20.1
- new net N$30: R6.2, R7.2
- new net N$31: R7.1, R8.1
- new net N$32: R8.2, R9.2
- new net N$33: R9.1, U$15.+
- new net N$34: BC546.DQ, C7.1, R35.1, U$15.-
- new net N$36: C9.2, U1.VCAP_1
- new net N$37: LED2.C, R15.2
- new net N$38: R15.1, U1.PC12
- new net N$4: C8.2, U$2.OUTPUT
- new net N$40: LED3.C, R16.2
- new net N$47: R53.1, R54.2, U$22.G
- new net N$48: R55.1, R56.2, U$23.G
- new net N$5: C8.1, U1.PH0/OSC_IN
- new net N$6: R21.1, R23.2, U$4.G
- new net N$7: R49.1, R50.2, U$20.G
- new net N$8: R25.1, R26.2, U$5.G
- new net NH3: R38.1, U$16.8, U1.PA1/USART2_RTS
- new net NO2: R37.1, U$16.9, U1.PA0/WKUP
- new net RX-O2: U$16.4, U1.PA10
- new net RX-S: U$21.5, U1.PC10
- new net SCL-TM: BSK1.7, U1.PB10
- new net SDA-TM: BSK1.8, U1.PB11
- new net TEMP: R51.2, R52.1, TEMP.1, U1.PA4/USART2_CK
- new net TX-O2: U$16.3, U1.PA9
- new net TX-S: U$21.7, U1.PC11
- new net VALVE: R50.1, U1.PB8
- net 5V: now also BSK1.4, HEAT.1, R36.1, U$1.PS, U$1.VCC, U$16.1, U$16.10, U$16.15, U$16.5, U$17.1, U$9.2, U2.!RESET!, U2.V+, VALVE1.1, VALVE2.1; no longer BSK4.3, MICS-6814.5V
- net BUS+: now also BSK1.2, COMPR.1; no longer BSK4.4
- net GND: now also C10.1, C13.1, C18.1, C19.1, C2.1, C20.1, C3.1, C6.1, C9.1, R1.1, R14.2, R16.1, R21.2, R22.2, R25.2, R28.2, R32.2, R46.2, R49.2, R51.1, R53.2, R55.2, TEMP.2, U$18.S, U$19.S, U$2.GND, U$20.S, U$21.10, U$21.4, U$21.6, U$21.8, U$22.S, U$23.S, U$3.S, U$4.S, U$5.S, U$7.S, U$8.S, U1.BOOT0, U1.PB2/BOOT1, U1.VSS, U1.VSSA; no longer BME280.GND, BSK4.1, C15.2, C16.2, C44.2, C45.2, C46.2, C47.2, C48.2, C53.2, C54.2, C55.2, IC2.BOOT0, IC2.PB2, IC2.VSSA, ME-O2.GND, MICS-6814.GND, R82.1, USB-C.GND
- net N$1: now also R13.1, U$1.CSB, U$1.GND; no longer PB5.C, R81.2
- net NRST: now also R10.1, U$21.3, U1.NRST; no longer IC2.NRST, R79.2, USB-C.NRST/EN
- net SCL: now also R17.2, U$1.SCL, U$16.12, U1.PB6; no longer IC2.PB10, R101.2
- net SDA: now also R18.2, U$1.SDA, U$16.13, U1.PB7; no longer IC2.PB11, R102.2
- net SWC: now also R12.1, U$21.11, U1.PA14/JTCK-SWCLK; no longer IC2.PA14, R27.2, USB-C.SWC/TXD
- net SWD: now also R11.1, U$21.9, U1.PA13/JMS-SWDIO; no longer IC2.PA13, R64.2, USB-C.SWD/RXD
- net TIME: now also BSK1.9, U1.PA15; no longer BSK4.5, IC2.PB6
Other:
- moved on the sheet: BME280, R2, R25, R26, R3, R4, R5, R6, R7, R8, R9

Commit message: Схема БКУ
Connections:
- net GND: no longer U$21.10, U$21.4, U$21.6, U$21.8
- net GND-OUT: now also U$21.10, U$21.4, U$21.6, U$21.8
Other:
- moved on the sheet: R1
Changed lines of the file:
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@@
 <attribute name="VALUE" x="54.61" y="1.778" size="1.778" layer="96"/>
 </instance>
-<instance part="R1" gate="G$1" x="246.38" y="-48.26" smashed="yes">
-<attribute name="NAME" x="242.57" y="-46.7614" size="1.778" layer="95"/>
-<attribute name="VALUE" x="242.57" y="-51.562" size="1.778" layer="96"/>
+<instance part="R1" gate="G$1" x="238.76" y="-15.24" smashed="yes">
+<attribute name="NAME" x="234.95" y="-13.7414" size="1.778" layer="95"/>
+<attribute name="VALUE" x="234.95" y="-18.542" size="1.778" layer="96"/>
 </instance>
 <instance part="U2" gate="G$1" x="-307.34" y="-472.44" smashed="yes">
@@
 <segment>
 <pinref part="R1" gate="G$1" pin="1"/>
-<wire x1="241.3" y1="-48.26" x2="228.6" y2="-48.26" width="0.1524" layer="91"/>
-<label x="228.6" y="-48.26" size="1.778" layer="95"/>
+<wire x1="233.68" y1="-15.24" x2="220.98" y2="-15.24" width="0.1524" layer="91"/>
+<label x="220.98" y="-15.24" size="1.778" layer="95"/>
 </segment>
 <segment>
@@
 <junction x="246.38" y="-368.3"/>
 <label x="231.14" y="-368.3" size="1.778" layer="95"/>
-</segment>
-<segment>
-<wire x1="360.68" y1="147.32" x2="360.68" y2="127" width="0.1524" layer="91"/>
-<label x="360.68" y="127" size="1.778" layer="95" rot="R90"/>
-<pinref part="U$21" gate="G$1" pin="8"/>
-</segment>
-<segment>
-<pinref part="U$21" gate="G$1" pin="4"/>
-<wire x1="350.52" y1="147.32" x2="350.52" y2="127" width="0.1524" layer="91"/>
-<label x="350.52" y="127" size="1.778" layer="95" rot="R90"/>
-</segment>
-<segment>
-<pinref part="U$21" gate="G$1" pin="6"/>
-<wire x1="355.6" y1="147.32" x2="355.6" y2="127" width="0.1524" layer="91"/>
-<label x="355.6" y="127" size="1.778" layer="95" rot="R90"/>
-</segment>
-<segment>
-<wire x1="365.76" y1="147.32" x2="365.76" y2="127" width="0.1524" layer="91"/>
-<label x="365.76" y="127" size="1.778" layer="95" rot="R90"/>
-<pinref part="U$21" gate="G$1" pin="10"/>
 </segment>
 </net>
@@
 <net name="GND-OUT" class="0">
 <segment>
-<wire x1="269.24" y1="-48.26" x2="251.46" y2="-48.26" width="0.1524" layer="91"/>
+<wire x1="261.62" y1="-15.24" x2="243.84" y2="-15.24" width="0.1524" layer="91"/>
 <pinref part="R1" gate="G$1" pin="2"/>
-<label x="259.08" y="-48.26" size="1.778" layer="95"/>
+<label x="251.46" y="-15.24" size="1.778" layer="95"/>
 </segment>
 <segment>
@@
 <pinref part="BSK1" gate="A" pin="5"/>
 </segment>
-</net>
+<segment>
+<wire x1="365.76" y1="147.32" x2="365.76" y2="127" width="0.1524" layer="91"/>
+<label x="365.76" y="127" size="1.778" layer="95" rot="R90"/>
+<pinref part="U$21" gate="G$1" pin="10"/>
+</segment>
+<segment>
+<wire x1="360.68" y1="147.32" x2="360.68" y2="127" width="0.1524" layer="91"/>
+<label x="360.68" y="127" size="1.778" layer="95" rot="R90"/>
+<pinref part="U$21" gate="G$1" pin="8"/>
+</segment>
+<segment>
+<pinref part="U$21" gate="G$1" pin="6"/>
+<wire x1="355.6" y1="147.32" x2="355.6" y2="127" width="0.1524" layer="91"/>
+<label x="355.6" y="127" size="1.778" layer="95" rot="R90"/>
+</segment>
+<segment>
+<pinref part="U$21" gate="G$1" pin="4"/>
+<wire x1="350.52" y1="147.32" x2="350.52" y2="127" width="0.1524" layer="91"/>
+<label x="350.52" y="127" size="1.778" layer="95" rot="R90"/>
+</segment>
+</net>

Commit message: Плата ПН почти разведена. Осталось добавить конденсаторы на компрессор и клапаны и запитать AVCC МК через стабилизатор напряжения
Parts:
- BME280: value BME280 -> BME280BME280-PINS-ONLY; device CanCubeSat:BME280 -> CanCubeSat:BME280BME280-PINS-ONLY
- U$1: value MS5611 -> MS5611MS5611-PIN-ONLY; device CanCubeSat:MS5611 -> CanCubeSat:MS5611MS5611-PIN-ONLY
Connections:
- removed net GND-40XV: U$5.D
- removed net RX-O2: U$16.4, U1.PA10
- removed net SCL: BME280.SCL, R17.2, U$1.SCL, U$16.12, U1.PB6
- removed net SDA: BME280.SDA, R18.2, U$1.SDA, U$16.13, U1.PB7
- removed net TX-O2: U$16.3, U1.PA9
- new net O2: U$16.3, U1.PA3/USART2_RX
- new net SENS-EXT-SCL: BME280.SCL, U$1.SCL, U1.PA8
- new net SENS-EXT-SDA: BME280.SDA, U$1.SDA, U1.PC9
- new net SENS-INT-SCL: R17.2, U$16.12, U1.PB6
- new net SENS-INT-SDA: R18.2, U$16.13, U1.PB7
- net 4OXV: now also U1.PA12; no longer U1.PC1
- net BME280-EXT: now also U1.PC0; no longer U1.PB14
- net BME280-INT: now also U1.PB1; no longer U1.PB13
- net CTRL-CO-1: now also U1.PB14; no longer U1.PB1
- net CTRL-CO-2: now also U1.PA9; no longer U1.PB0
- net CTRL-NH3-1: now also U1.PB12; no longer U1.PA12
- net CTRL-NH3-2: now also U1.PB13; no longer U1.PA11
- net DOSE: now also U1.PD2
- net GND-4OXV: now also U$5.D
- net GND-OUT: now also U$21.3, U$21.5, U$21.7, U$21.9; no longer U$21.10, U$21.4, U$21.6, U$21.8
- net MICS: now also U1.PA11; no longer U1.PC0
- net MS5611-EXT: now also U1.PC1; no longer U1.PA8
- net MS5611-INT: now also U1.PB0; no longer U1.PB12
- net NRST: now also U$21.11; no longer U$21.3
- net RX-S: now also U$21.4; no longer U$21.5
- net SWC: now also U$21.10; no longer U$21.11
- net SWD: now also U$21.8; no longer U$21.9
- net TX-S: now also U$21.6; no longer U$21.7

Commit message: Плата ПН готова к проверке
Parts:
- added C11, C12: 1uF, CanCubeSat:ECAP1UF
- added U$24, U$6: 220uF, CanCubeSat:ECAPECAP220
- added U$25: ADP150AUJZ-3.3-R7, CanCubeSat:ADP150AUJZ-3.3-R7
- U$14: value ECAP -> 1uF
- renumbered U$1 to MS5611
Connections:
- new net N$9: C11.1, C3.1, U$25.VOUT, U1.VDDA
- net 3V3: no longer C3.2, U1.VDDA
- net 5V: now also C12.1, U$24.1, U$25.EN, U$25.VIN
- net BUS+: now also U$6.1
- net GND: now also C11.2, C12.2, C3.2, U$25.GND; no longer C3.1
- net GND-COMPR: now also U$6.2
- net GND-VALVE: now also U$24.2
Other:
- moved on the sheet: C3

Commit message: Добавил красоты на плате ПН, поправил подтяжки некоторых транзисторов
Parts:
- added U$1, U$26: PCB "Payload", CanCubeSat:ITS-LOGOPCB-""
Connections:
- net 3V3: now also R14.2, R21.2, R22.2, R25.2, R28.2, R32.2, R46.2
- net GND: no longer R14.2, R21.2, R22.2, R25.2, R28.2, R32.2, R46.2
Other:
- note added: "Внешние интерфейсы"
- note added: "Дозиметр"
- note added: "Интерфейс внешнего BME280"
- note added: "Интерфейс внешнего MS5611"
- note added: "Интерфейс герметичного отсека"
- note added: "Интерфейс клапанов"
- note added: "Интерфейс компрессора"
- note added: "Интерфейс нагревателя ДНК"
- note added: "Интерфейс термометра ДНК"
- note added: "Коммутация 4OXV"
- note added: "Коммутация MICS-6814"
- note added: "Коммутация внешнего BME280"
- note added: "Коммутация внешнего MS5611"
- note added: "Коммутация внутреннего BME280"
- note added: "Коммутация внутреннего MS5611"
- note added: "Коммутация дозиметра"
- note added: "Коммутация клапанов"
- note added: "Коммутация компрессора"
- note added: "Коммутация нагревателя ДНК"
- note added: "Микроконтроллер"
- note added: "Плавкий предохранитель платы "Payload""
- moved on the sheet: 2N6517, BC546, BME280, BSK1, C1, C10, C11, C12, C13, C18, C19, C2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
