File: schematics/board/BSK3.brd (EAGLE design)
At the start: 82 x 100 mm, 28 parts

Commit message: Сделаны платы CROSSnew, SPIDERnew, BSK2
Parts:
- removed DS18B20Z: DS18B20Z, CanCubeSat:DS18B20Z
- removed FS8205A: FS8205A+, CanCubeSat:FS8205A+
- removed L293DD: L293DD, CanCubeSat:L293DD
- removed LAP4: LAP4-BOTTOM, led:P47F-BOTTOM
- removed LED1, LED2, LED3, LED4: (no value), led:CHIPLED_0603
- removed R1, R2, R3, R81: 2k, resistor:R0603
- removed R10, R11: 100R, resistor:R0603
- removed R19: 1M, resistor:R0603
- removed R20: 510k, resistor:R0603
- removed U$6, U$7: EM_HEAT, CanCubeSat:EM_HEAT
- added DS18B20Z1: DS18B20Z, CanCubeSat:DS18B20Z
- added LAP1: LAP4-BOTTOM, led:P47F-BOTTOM
- added LED6, LED7: (no value), led:CHIPLED_0603
- added R12, R6: 2M, resistor:R0603
- added R13: 1k5, resistor:R0603
- added R14, R5, R8, R9: 1M, resistor:R0603
- added R4, R7: 2k, resistor:R0603
- added R94, R95: 2k26, resistor:R0603
- added U$13, U$8: SI2302CDS, CanCubeSat:SOT23-3
- added U$14: EM_HEAT, CanCubeSat:EM_HEAT
- added U$26: FS8205A+, CanCubeSat:FS8205A+
- added U$5: MOCD217M, CanCubeSat:SOIC8
Connections:
- removed net HEAT: DS18B20Z.HEAT, FS8205A.HEAT, L293DD.HEAT
- removed net N$1: L293DD.3, LED1.C, LED2.A, U$6.1
- removed net N$2: L293DD.8, R1.1, R81.1, U$6.2
- removed net N$3: L293DD.18, LED3.A, U$7.1
- removed net N$4: LED2.C, R81.2
- removed net N$5: LED1.A, R1.2
- removed net N$6: LED3.C, R2.1
- removed net N$7: LAP4.A, LED4.A, R3.2
- removed net N$8: FS8205A.4, R10.2
- removed net N$9: FS8205A.5, R11.2
- new net 1: R7.2, U$14.2, U$8.3
- new net 2: R13.2, U$13.3
- new net B3-KHEAT: R8.1, U$8.1
- new net B3-KVCC: R94.2, R95.2, U$5.1, U$5.3
- new net B3-ROZE: R14.1, U$13.1
- new net N$10: R5.1, R6.2, U$26.5
- new net N$27: R12.1, R9.1, U$26.4
- new net N$28: LAP1.A, R4.2
- new net N$29: LED7.C, R13.1
- new net N$30: DS18B20Z1.HEAT, U$26.HEAT
- new net N$31: LED6.C, R7.1
- new net OC1: R9.2, U$5.6
- new net OD1: R5.2, U$5.8
- net 1W: now also DS18B20Z1.4; no longer DS18B20Z.4
- net 5V: now also DS18B20Z1.3, LED6.A, R4.1, U$14.1; no longer DS18B20Z.3, L293DD.1, L293DD.10, L293DD.11, L293DD.20, R3.1
- net B3_KEM+: no longer L293DD.2
- net B3_KEM-: no longer L293DD.9
- net B3_KHEAT: no longer L293DD.19
- net B3_KVCC: no longer R10.1, R11.1, R19.1, R20.1
- net BUS+: now also LED7.A, R12.2, R6.1; no longer R19.2
- net BUS-: now also LAP1.C, U$26.67, U$5.7; no longer FS8205A.23, LAP4.C, LED4.C, R20.2
- net GND: now also DS18B20Z1.5, R14.2, R8.2, R94.1, R95.1, U$13.2, U$26.23, U$5.2, U$5.4, U$5.5, U$8.2; no longer DS18B20Z.5, FS8205A.67, L293DD.14, L293DD.15, L293DD.16, L293DD.17, L293DD.4, L293DD.5, L293DD.6, L293DD.7, R2.2, U$7.2
Routing:
- net N$2: track 64.3 -> 0.00 mm, vias 2 -> 0
- net N$7: track 61.5 -> 0.00 mm, vias 4 -> 0
- net N$1: track 60.8 -> 0.00 mm, vias 2 -> 0
- net N$3: track 53.0 -> 0.00 mm, vias 2 -> 0
- net GND: track 206.4 -> 191.2 mm
- net 5V: track 173.4 -> 160.9 mm, vias 6 -> 4
- net B3_KVCC: track 20.6 -> 13.1 mm
- net BUS-: track 104.9 -> 100.4 mm
- net N$9: track 2.74 -> 0.00 mm
- net N$5: track 1.94 -> 0.00 mm
- net N$4: track 1.94 -> 0.00 mm
- net N$8: track 1.77 -> 0.00 mm
- net N$6: track 1.74 -> 0.00 mm
- net BUS+: track 150.9 -> 150.2 mm

Commit message: Плата АB+DC-DC
Parts:
- removed BSK1: (no value), pinheadCS:1X12
- removed LAP1: LAP4-BOTTOM, led:P47F-BOTTOM
- added BKU: (no value), pinheadCS:1X16
- added C41: 0,1µ, rcl:C0603
- added CMD: KCONNECTQUAD, CanCubeSat:KCONNECT_QUAD
- added R1, R2: 2k26, resistor:R0603
- added R75: R01, rcl:R2512
- added R76, R77: 10R, resistor:R0603
- added U$15, U$16, U$6, U$7: GRAFITGRAFIT3_1, CanCubeSat:GRAFIT3_1
- added U$57: INA219AID, CanCubeSat:SOT23-8
- added YELLOW: LAP4-BOTTOM, led:P47F-BOTTOM
- BSK5: device pinheadCS:1X08 -> pinheadCS:1X12
- DS18B20Z1: device CanCubeSat:DS18B20Z -> CanCubeSat:SOIC8+HEAT_S
- R12, R6: value 2M -> 100k
- R5, R9: value 1M -> 100R
- R94, R95: value 2k26 -> 200k
- moved R9 125.7 mm to (33.6, 88.6), turned to 90 degrees
- moved R12 120.3 mm to (31.2, 88.6), turned to 90 degrees
- moved R5 117.1 mm to (26.4, 88.6), turned to 90 degrees
- moved R6 117.0 mm to (28.8, 88.6), turned to 270 degrees
- moved R95 105.2 mm to (40.1, 80.5)
- moved R94 104.1 mm to (40.1, 78.1)
- moved R7 102.1 mm to (11.4, 69.2), turned to 270 degrees
- moved U$5 102.0 mm to (41.2, 86.4)
- moved U$26 102.0 mm to (30.0, 85.0), turned to 90 degrees
- moved R13 100.7 mm to (65.0, 53.7)
- moved LED7 99.6 mm to (65.0, 56.5), turned to 90 degrees
- moved LED6 93.1 mm to (8.80, 69.2)
- moved R14 93.0 mm to (65.0, 47.6)
- moved U$8 92.7 mm to (7.10, 60.5)
- moved U$13 91.0 mm to (65.0, 50.7)
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Connections:
- net BUS+1 renamed SP+1
- net BUS+2 renamed SP+2
- net BUS+3 renamed SP+3
- net BUS-1 renamed SP-1
- net BUS-2 renamed SP-2
- net BUS-3 renamed SP-3
- removed net B3_KEM+: BSK1.5
- removed net B3_KEM-: BSK1.4
- removed net B3_KHEAT: BSK1.6
- removed net B3_KVCC: BSK1.7
- removed net B5_KEM+: BSK1.2, BSK5.3
- removed net B5_KEM-: BSK1.1, BSK5.2
- removed net B5_KHEAT: BSK1.11, BSK5.4
- removed net B5_KVCC: BSK1.12, BSK5.5
- removed net BUS-: LAP1.C, U$2.1, U$2.2, U$2.3, U$2.4, U$2.P$1, U$2.P$2, U$26.67, U$5.7
- removed net N$30: DS18B20Z1.HEAT, U$26.HEAT
- new net 3V3: BKU.8, BSK5.4, U$57.4
- new net B3-CMD: BKU.4, CMD.1, CMD.2, CMD.3, CMD.4, CMD.P$1, CMD.P$2
- new net B5-CMD: BKU.13, BSK5.9
- new net B5-KHEAT: BKU.10, BSK5.6
- new net B5-KVCC: BKU.11, BSK5.7
- new net B5-ROZE: BKU.12, BSK5.8
- new net N$150: C41.1, R76.2, U$57.1
- new net N$151: C41.2, R77.2, U$57.2
- new net N$2: R1.1, R94.2, U$5.1
- new net N$3: R2.1, R95.2, U$5.3
- new net SCL-INA: BKU.15, BSK5.11, U$57.5, U$57.7
- new net SDA-INA: BKU.16, BSK5.12, U$57.6
- new net SINS-KVCC: BKU.14, BSK5.10
- new net SP+: R75.1, R77.1, U$3.1, U$3.2, U$3.3, U$3.4, U$3.P$1, U$3.P$2
- new net SP-: U$2.1, U$2.2, U$2.3, U$2.4, U$2.P$1, U$2.P$2, U$26.67, U$5.7, YELLOW.C
- net 1W: now also BKU.5, BSK5.1; no longer BSK1.8, BSK5.6
- net 2: now also U$15.P$1, U$16.P$1, U$6.P$1, U$7.P$1
- net 5V: now also BKU.7, BSK5.3; no longer BSK1.9, BSK5.7
- net B3-KHEAT: now also BKU.1
- net B3-KVCC: now also BKU.2, R1.2, R2.2; no longer R94.2, R95.2, U$5.1, U$5.3
- net B3-ROZE: now also BKU.3
- net BUS+: now also BKU.6, BSK5.2, R75.2, R76.1, U$15.P$2, U$16.P$2, U$6.P$2, U$7.P$2; no longer BSK1.10, BSK5.8, U$3.1, U$3.2, U$3.3, U$3.4, U$3.P$1, U$3.P$2
- net GND: now also BKU.9, BSK5.5, DS18B20Z1.HEAT, U$26.HEAT, U$57.3, U$57.8; no longer BSK1.3, BSK5.1
- net N$28: now also YELLOW.A; no longer LAP1.A
Routing:
- net 2: track 0.00 -> 140.1 mm, vias 0 -> 4
- net B5_KEM-: track 135.1 -> 0.00 mm
- net SP-: track 0.00 -> 125.8 mm, vias 0 -> 1
- net SCL-INA: track 0.00 -> 123.5 mm, vias 0 -> 4
- net 3V3: track 0.00 -> 122.7 mm, vias 0 -> 7
- net GND: track 191.2 -> 73.3 mm, vias 5 -> 1
- net SDA-INA: track 0.00 -> 116.7 mm, vias 0 -> 1
- net B5_KHEAT: track 116.6 -> 0.00 mm
- net B5_KVCC: track 115.4 -> 0.00 mm
- net B5-KHEAT: track 0.00 -> 113.3 mm, vias 0 -> 2
- net B5-ROZE: track 0.00 -> 111.8 mm, vias 0 -> 5
- net B5-CMD: track 0.00 -> 110.7 mm
- net SINS-KVCC: track 0.00 -> 107.6 mm
- net B5_KEM+: track 106.8 -> 0.00 mm
- net B3-ROZE: track 0.00 -> 105.8 mm, vias 0 -> 3
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- added copper zone on layer 1, net GND
- added copper zone on layer 1, net GND1
- added copper zone on layer 1, net GND2
- added copper zone on layer 1, net GND3
- added copper zone on layer 1, net GND4
- removed copper zone on layer 1, net HEAT
Other:
- outline, holes or cut-outs redrawn
- board text added: "to BKU"
- board text removed: "BUS"
- board text removed: "EM+"
- board text removed: "EM-"
- board text removed: "to BSK1"

Commit message: Внесены правки в платы БСК
Parts:
- added R3, R32: 100R, resistor:R0603
- BKU: device pinheadCS:1X16 -> pinheadCS:1X14
- BSK5: device pinheadCS:1X12 -> pinheadCS:1X08
- moved LED7 2.00 mm to (67.0, 56.5)
- moved R13 2.00 mm to (67.0, 53.7)
- moved R14 2.00 mm to (67.0, 47.6)
- moved U$13 2.00 mm to (67.0, 50.7)
Connections:
- removed net B5-CMD: BKU.13, BSK5.9
- removed net B5-KVCC: BKU.11, BSK5.7
- removed net B5-ROZE: BKU.12, BSK5.8
- new net N$20: R32.1, R8.1, U$8.1
- new net N$21: R14.1, R3.1, U$13.1
- net 3V3: no longer BSK5.4
- net B3-KHEAT: now also R32.2; no longer R8.1, U$8.1
- net B3-ROZE: now also R3.2; no longer R14.1, U$13.1
- net B5-KHEAT: now also BSK5.5; no longer BSK5.6
- net GND: now also BKU.14, BSK5.4; no longer BSK5.5
- net SCL-INA: now also BKU.12, BSK5.7; no longer BKU.15, BSK5.11
- net SDA-INA: now also BKU.13, BSK5.8; no longer BKU.16, BSK5.12
- net SINS-KVCC: now also BKU.11, BSK5.6; no longer BKU.14, BSK5.10
Routing:
- net B5-ROZE: track 111.8 -> 0.00 mm, vias 5 -> 0
- net B5-CMD: track 110.7 -> 0.00 mm
- net B5-KVCC: track 104.2 -> 0.00 mm, vias 4 -> 0
- net 3V3: track 122.7 -> 25.8 mm, vias 7 -> 3
- net GND: track 73.3 -> 66.5 mm
- net SINS-KVCC: track 107.6 -> 100.9 mm, vias 0 -> 2
- net BUS+: track 241.7 -> 247.2 mm
- net N$21: track 0.00 -> 4.30 mm
- net N$20: track 0.00 -> 4.24 mm
- net 5V: track 144.1 -> 147.2 mm
- net 1W: track 122.5 -> 125.6 mm
- net SCL-INA: track 123.5 -> 126.5 mm
- net B3-ROZE: track 105.8 -> 103.1 mm
- net 2: track 140.1 -> 142.1 mm
- net B3-KVCC: track 35.0 -> 34.1 mm
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
Commit message: Две линии i2c на платах БСК заменены на одну
Parts:
- BSK5: device pinheadCS:1X08 -> pinheadCS:1X06
Connections:
- removed net SCL-INA: BKU.12, BSK5.7, U$57.5, U$57.7
- removed net SDA-INA: BKU.13, BSK5.8, U$57.6
- new net SCL-TM: BKU.12, U$57.5, U$57.7
- new net SDA-TM: BKU.13, U$57.6
Routing:
- net SCL-INA: track 126.5 -> 0.00 mm, vias 4 -> 0
- net SDA-INA: track 117.4 -> 0.00 mm, vias 1 -> 0
- net SCL-TM: track 0.00 -> 13.9 mm, vias 0 -> 1
- net SDA-TM: track 0.00 -> 11.9 mm, vias 0 -> 1
- net B3-ROZE: track 103.1 -> 95.6 mm, vias 3 -> 1
- net BUS+: track 247.2 -> 248.3 mm
- net 5V: track 147.2 -> 148.3 mm
- net 1W: track 125.6 -> 126.7 mm
- net SINS-KVCC: track 100.9 -> 99.8 mm
- net B5-KHEAT: track 112.8 -> 113.8 mm
- net GND: track 66.5 -> 65.8 mm
Changed lines of the file:
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@@
 <attribute name="VALUE" x="53.384540625" y="67.390853125" size="1.27" layer="27" rot="R315"/>
 </element>
-<element name="BSK5" library="pinheadCS" package="1X08" value="" x="41" y="1.25" smashed="yes">
+<element name="BSK5" library="pinheadCS" package="1X06" value="" x="41" y="1.25" smashed="yes">
 <attribute name="VALUE" x="30.84" y="-1.925" size="1.27" layer="27"/>
 </element>
@@
 <wire x1="34.84" y1="76.7" x2="35.62" y2="76.7" width="0.3" layer="1"/>
 <wire x1="35.62" y1="76.7" x2="35.7" y2="76.695" width="0.3" layer="1"/>
-<wire x1="33.02" y1="78.52" x2="33.1" y2="78.6" width="0.3" layer="1"/>
-<wire x1="33.02" y1="78.78" x2="33.1" y2="78.6" width="0.3" layer="1"/>
 <wire x1="33.28" y1="85.28" x2="40.56" y2="85.28" width="0.3" layer="1"/>
 <wire x1="33" y1="85" x2="33.28" y2="85.28" width="0.3" layer="1"/>
@@
 <wire x1="44.81" y1="98.75" x2="44.81" y2="97.11" width="0.3" layer="16"/>
 <wire x1="56.16" y1="90.22" x2="56.125" y2="90" width="0.3" layer="1"/>
-<wire x1="35.88" y1="76.44" x2="35.7" y2="76.695" width="0.3" layer="1"/>
 <wire x1="68.04" y1="47.84" x2="68.04" y2="49.66" width="0.3" layer="1"/>
 <wire x1="68.04" y1="49.66" x2="67.95" y2="49.7" width="0.3" layer="1"/>
 <wire x1="68.04" y1="47.84" x2="67.85" y2="47.6" width="0.3" layer="1"/>
-<wire x1="67.78" y1="47.58" x2="67.85" y2="47.6" width="0.3" layer="1"/>
 <wire x1="8.06" y1="57.2" x2="7.95" y2="57.4" width="0.3" layer="1"/>
 <wire x1="34.84" y1="76.7" x2="35.7" y2="76.695" width="0.3" layer="1"/>
@@
 <wire x1="38.16" y1="97.18" x2="38.16" y2="84.66" width="0.5" layer="16"/>
 <wire x1="38.16" y1="84.66" x2="35.309828125" y2="81.809828125" width="0.5" layer="16"/>
-<wire x1="37.19" y1="1.25" x2="37.19" y2="19.42" width="0.5" layer="16"/>
-<wire x1="37.19" y1="19.42" x2="32.11" y2="24.5" width="0.5" layer="16"/>
+<wire x1="39.73" y1="1.25" x2="39.73" y2="16.88" width="0.5" layer="16"/>
+<wire x1="39.73" y1="16.88" x2="32.11" y2="24.5" width="0.5" layer="16"/>
 </signal>
 <signal name="1W">
@@
 <via x="33.8" y="74.62" extent="1-16" drill="0.35"/>
 <wire x1="32.5" y1="63.8" x2="33.8" y2="65.1" width="0.3" layer="16"/>
-<wire x1="32.11" y1="1.25" x2="32.11" y2="17.92" width="0.3" layer="16"/>
-<wire x1="32.11" y1="17.92" x2="24.53" y2="25.5" width="0.3" layer="16"/>
+<wire x1="34.65" y1="1.25" x2="34.65" y2="15.38" width="0.3" layer="16"/>
+<wire x1="34.65" y1="15.38" x2="24.53" y2="25.5" width="0.3" layer="16"/>
 </signal>
 <signal name="BUS+">
@@
 <wire x1="37.19" y1="98.75" x2="37.19" y2="94.7567875" width="1" layer="16"/>
 <wire x1="37.19" y1="94.7567875" x2="33.43" y2="90.9967875" width="1" layer="16"/>
-<wire x1="34.65" y1="1.25" x2="34.65" y2="17.195590625" width="1" layer="16"/>
-<wire x1="34.65" y1="17.195590625" x2="27.72734375" y2="24.118246875" width="1" layer="16"/>
+<wire x1="37.19" y1="1.25" x2="37.19" y2="14.655590625" width="1" layer="16"/>
+<wire x1="37.19" y1="14.655590625" x2="27.72734375" y2="24.118246875" width="1" layer="16"/>
 </signal>
 <signal name="SP+1">
@@
 <signal name="B3-ROZE">
 <contactref element="BKU" pad="3"/>
-<wire x1="42.12" y1="32.76" x2="42.12" y2="32.24" width="0.3" layer="16"/>
-<wire x1="33.54" y1="41.34" x2="42.12" y2="32.76" width="0.3" layer="16"/>
-<wire x1="33.54" y1="62.4" x2="33.54" y2="41.34" width="0.3" layer="16"/>
+<wire x1="33.54" y1="41.5" x2="33.54" y2="62.4" width="0.3" layer="16"/>
 <wire x1="36.36" y1="65.22" x2="33.54" y2="62.4" width="0.3" layer="16"/>
 <wire x1="36.36" y1="73.7" x2="36.36" y2="65.22" width="0.3" layer="16"/>
 <wire x1="28.74" y1="81.32" x2="36.36" y2="73.7" width="0.3" layer="16"/>
-<via x="42.12" y="32.24" extent="1-16" drill="0.35"/>
-<wire x1="42.12" y1="32.24" x2="43.94215" y2="34.06215" width="0.3" layer="1"/>
-<wire x1="43.94215" y1="34.06215" x2="43.94215" y2="34.14215" width="0.3" layer="1"/>
-<via x="43.94215" y="34.14215" extent="1-16" drill="0.35"/>
-<wire x1="43.94215" y1="34.14215" x2="57.08" y2="47.28" width="0.3" layer="16"/>
+<wire x1="57.08" y1="47.28" x2="50.5" y2="40.7" width="0.3" layer="16"/>
 <wire x1="57.08" y1="47.28" x2="60.165" y2="47.28" width="0.3" layer="16"/>
 <via x="60.165" y="47.28" extent="1-16" drill="0.35"/>
@@
 <wire x1="29.57" y1="98.75" x2="28.74" y2="97.92" width="0.3" layer="16"/>
 <wire x1="28.74" y1="97.92" x2="28.74" y2="81.32" width="0.3" layer="16"/>
+<wire x1="50.5" y1="40.7" x2="34.34" y2="40.7" width="0.3" layer="16"/>
+<wire x1="34.34" y1="40.7" x2="33.54" y2="41.5" width="0.3" layer="16"/>
 </signal>
 <signal name="B3-KVCC">
@@
 <wire x1="35.8" y1="44.7" x2="46.5" y2="44.7" width="1" layer="16"/>
 </signal>
-<signal name="SCL-INA">
+<signal name="SCL-TM">
 <contactref element="U$57" pad="5"/>
 <contactref element="U$57" pad="7"/>
 <wire x1="56.775" y1="90" x2="56.775" y2="89.405025" width="0.3" layer="1"/>
 <wire x1="56.775" y1="89.405025" x2="57.080025" y2="89.1" width="0.3" layer="1"/>
-<wire x1="57.769975" y1="89.1" x2="57.9149875" y2="89.2450125" width="0.3" layer="1"/>
-<wire x1="57.9149875" y1="89.2450125" x2="58.075" y2="89.405025" width="0.3" layer="1"/>
+<wire x1="57.769975" y1="89.1" x2="58.075" y2="89.405025" width="0.3" layer="1"/>
 <wire x1="58.075" y1="89.405025" x2="58.075" y2="90" width="0.3" layer="1"/>
 <wire x1="57.080025" y1="89.1" x2="57.769975" y2="89.1" width="0.3" layer="1"/>
-<wire x1="57.98" y1="89.18" x2="60" y2="89.18" width="0.3" layer="1"/>
-<wire x1="57.98" y1="89.18" x2="57.9149875" y2="89.2450125" width="0.3" layer="1"/>
 <via x="58.1" y="91.1" extent="1-16" drill="0.35"/>
 <wire x1="58.1" y1="91.1" x2="58.075" y2="91.075" width="0.3" layer="1"/>
 <wire x1="58.075" y1="90" x2="58.075" y2="91.075" width="0.3" layer="1"/>
-<wire x1="60" y1="89.18" x2="60.00215" y2="89.17785" width="0.3" layer="1"/>
-<via x="60.00215" y="89.17785" extent="1-16" drill="0.35"/>
-<wire x1="60.00215" y1="89.17785" x2="65.52215" y2="89.17785" width="0.3" layer="16"/>
-<wire x1="65.52215" y1="89.17785" x2="75.9" y2="78.8" width="0.3" layer="16"/>
-<wire x1="75.9" y1="78.8" x2="75.9" y2="56.3" width="0.3" layer="16"/>
-<wire x1="75.9" y1="56.3" x2="62.4" y2="42.8" width="0.3" layer="16"/>
-<via x="60.7" y="42.7" extent="1-16" drill="0.35"/>
-<wire x1="60.7" y1="42.7" x2="60.8" y2="42.8" width="0.3" layer="1"/>
-<wire x1="60.8" y1="42.8" x2="62.4" y2="42.8" width="0.3" layer="1"/>
-<via x="62.4" y="42.8" extent="1-16" drill="0.35"/>
-<contactref element="BSK5" pad="7"/>
 <contactref element="BKU" pad="12"/>
 <wire x1="52.43" y1="98.75" x2="58.1" y2="93.08" width="0.3" layer="16"/>
 <wire x1="58.1" y1="93.08" x2="58.1" y2="91.1" width="0.3" layer="16"/>
-<wire x1="47.35" y1="29.35" x2="47.35" y2="1.25" width="0.3" layer="16"/>
-<wire x1="60.7" y1="42.7" x2="47.35" y2="29.35" width="0.3" layer="16"/>
-</signal>
-<signal name="SDA-INA">
+</signal>
+<signal name="SDA-TM">
 <contactref element="U$57" pad="6"/>
-<wire x1="61.58" y1="61.66" x2="61.58" y2="38.44" width="0.3" layer="16"/>
-<wire x1="51.8" y1="71.44" x2="61.58" y2="61.66" width="0.3" layer="16"/>
-<wire x1="51.8" y1="88.5" x2="51.8" y2="71.44" width="0.3" layer="16"/>
 <wire x1="57.425" y1="90" x2="57.425" y2="90.6" width="0.3" layer="1"/>
 <wire x1="57.425" y1="90.6" x2="57.225" y2="90.8" width="0.3" layer="1"/>
@@
 <wire x1="57.7" y1="91.9" x2="57.225" y2="91.425" width="0.3" layer="1"/>
 <via x="58.9" y="91.9" extent="1-16" drill="0.35"/>
-<wire x1="58.9" y1="91.9" x2="58.9" y2="90.4" width="0.3" layer="16"/>
-<wire x1="58.9" y1="90.4" x2="57" y2="88.5" width="0.3" layer="16"/>
-<wire x1="51.8" y1="88.5" x2="57" y2="88.5" width="0.3" layer="16"/>
-<contactref element="BSK5" pad="8"/>
 <contactref element="BKU" pad="13"/>
 <wire x1="54.97" y1="98.75" x2="58.9" y2="94.82" width="0.3" layer="16"/>
 <wire x1="58.9" y1="94.82" x2="58.9" y2="91.9" width="0.3" layer="16"/>
-<wire x1="49.89" y1="26.75" x2="49.89" y2="1.25" width="0.3" layer="16"/>
-<wire x1="61.58" y1="38.44" x2="49.89" y2="26.75" width="0.3" layer="16"/>
 </signal>
 <signal name="3V3">
@@
 <wire x1="50.8" y1="41" x2="51.4" y2="40.4" width="0.3" layer="1"/>
 <via x="51.4" y="40.4" extent="1-16" drill="0.35"/>
-<wire x1="51.4" y1="40.4" x2="44.81" y2="33.81" width="0.3" layer="16"/>
-<wire x1="44.81" y1="33.81" x2="44.81" y2="1.25" width="0.3" layer="16"/>
 <wire x1="50.8" y1="97.84" x2="50.8" y2="42.3" width="0.3" layer="16"/>
+<wire x1="47.35" y1="1.25" x2="47.35" y2="36.35" width="0.3" layer="16"/>
+<wire x1="47.35" y1="36.35" x2="51.4" y2="40.4" width="0.3" layer="16"/>
 </signal>
 <signal name="B5-KHEAT">
 <contactref element="BKU" pad="10"/>
-<wire x1="42.3" y1="30.76" x2="42.3" y2="1.28" width="0.3" layer="16"/>
-<wire x1="33.02" y1="40.04" x2="42.3" y2="30.76" width="0.3" layer="16"/>
-<wire x1="33.02" y1="63.48" x2="33.02" y2="40.04" width="0.3" layer="16"/>
+<wire x1="33.02" y1="40.04" x2="33.02" y2="63.48" width="0.3" layer="16"/>
 <wire x1="35.52" y1="73.18" x2="35.52" y2="65.98" width="0.3" layer="16"/>
 <wire x1="35.52" y1="65.98" x2="33.02" y2="63.48" width="0.3" layer="16"/>
@@
 <via x="41.12" y="73.94" extent="1-16" drill="0.35"/>
 <contactref element="BSK5" pad="5"/>
-<wire x1="42.3" y1="1.28" x2="42.27" y2="1.25" width="0.3" layer="16"/>
+<wire x1="44.81" y1="1.25" x2="44.81" y2="28.25" width="0.3" layer="16"/>
+<wire x1="44.81" y1="28.25" x2="33.02" y2="40.04" width="0.3" layer="16"/>
 </signal>
 <signal name="N$11">

Commit message: Обновлен список плат, работа над платой ПН
Changed lines of the file:
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@@
 <wire x1="82" y1="8.5" x2="75" y2="8.5" width="0.1524" layer="20"/>
 <wire x1="7" y1="8.5" x2="0" y2="8.5" width="0.1524" layer="20"/>
-<hole x="11" y="4" drill="6"/>
-<hole x="71" y="4" drill="6"/>
-<hole x="71" y="96" drill="6"/>
-<hole x="11" y="96" drill="6"/>
+<hole x="11" y="4" drill="4.5"/>
+<hole x="71" y="4" drill="4.5"/>
+<hole x="71" y="96" drill="4.5"/>
+<hole x="11" y="96" drill="4.5"/>
 <text x="10.5" y="72.4" size="1.4224" layer="26" rot="MR45">BUS+</text>
 <text x="74.5" y="75.3" size="1.4224" layer="26" rot="MR315">BUS+</text>

Commit message: Схема БКУ
Changed lines of the file:
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@@
 <wire x1="18.328" y1="37.462" x2="6.328" y2="37.462" width="0.1" layer="21"/>
 <rectangle x1="6.328" y1="37.462" x2="18.328" y2="54.462" layer="29"/>
+<hole x="11" y="33" drill="5"/>
 </plain>
 <attributes>
