File: schematics/board/BSK5.brd (EAGLE design)
At the start: 94 x 94 mm, 88 parts, among them U1 STM32F405RGT6, X1 JST-6, X11 JST-6

Commit message: Добавлены подписи Концерна к платам
Parts:
- added U$26: PCB "BSK5", CanCubeSat:ITS-LOGO
Other:
- board text removed: "BSK5 "Концерн ИТС""
Changed lines of the file:
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@@
 <drawing>
 <settings>
-<setting alwaysvectorfont="no"/>
+<setting alwaysvectorfont="yes"/>
 <setting verticaltext="up"/>
 </settings>
@@
 <wire x1="25.262" y1="13.572" x2="25.262" y2="25.572" width="0.1" layer="21"/>
 <rectangle x1="27.762" y1="11.072" x2="39.762" y2="28.072" layer="29" rot="R270"/>
-<text x="46.8" y="81.4" size="2" layer="26" rot="MR180" align="bottom-center">BSK5
-"Концерн ИТС"</text>
 <text x="38" y="89.5" size="2" layer="26" rot="MR0" align="bottom-right">to BSK3</text>
 <wire x1="0" y1="72.5" x2="0" y2="66.5" width="0.15" layer="20"/>
@@
 <attribute name="NAME" x="88.735" y="27.965" size="1.27" layer="25" rot="R180"/>
 <attribute name="VALUE" x="88.735" y="30.505" size="1.27" layer="27" rot="R180"/>
+</element>
+<element name="U$26" library="CanCubeSat" package="ITS-LOGO" value="PCB &quot;BSK5&quot;" x="7" y="28.3" smashed="yes" rot="MR90">
+<attribute name="VALUE" x="5.5" y="28.3" size="1" layer="22" font="vector" ratio="15" rot="MR90"/>
 </element>
 </elements>
@@
 </drawing>
 <compatibility>
-<note version="6.3" minversion="6.2.2" severity="warning">
-Since Version 6.2.2 text objects can contain more than one line,
-which will not be processed correctly with this version.
-</note>
 <note version="8.2" severity="warning">
 Since Version 8.2, EAGLE supports online libraries. The ids

Commit message: Начато исправление разъемов
Connections:
- net RX-S: now also U1.52; no longer U1.51
- net TX-S: now also U1.51; no longer U1.52
Routing:
- net TX-S: track 40.6 -> 41.6 mm
- net RX-S: track 41.5 -> 40.8 mm
Changed lines of the file:
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@@
 <wire x1="58.55" y1="19.8" x2="58.75" y2="19.6" width="0.4" layer="1"/>
 <wire x1="58.85" y1="64.4" x2="59.05" y2="64.2" width="0.4" layer="1"/>
-<wire x1="52.05" y1="64.6" x2="52.25" y2="64.4" width="0.4" layer="1"/>
 <wire x1="45.25" y1="64.6" x2="45.45" y2="64.4" width="0.4" layer="1"/>
 <wire x1="38.45" y1="64.6" x2="38.65" y2="64.4" width="0.4" layer="1"/>
@@
 </signal>
 <signal name="RX-S">
-<contactref element="U1" pad="51"/>
 <wire x1="11.25" y1="55.5" x2="10.75" y2="55.5" width="0.3" layer="16"/>
 <wire x1="16.75" y1="50" x2="11.25" y2="55.5" width="0.3" layer="16"/>
 <wire x1="33.75" y1="50" x2="16.75" y2="50" width="0.3" layer="16"/>
 <wire x1="35.55" y1="48.2" x2="33.75" y2="50" width="0.3" layer="16"/>
-<wire x1="36.45" y1="48.2" x2="35.55" y2="48.2" width="0.3" layer="16"/>
-<wire x1="37.25" y1="49" x2="36.45" y2="48.2" width="0.3" layer="16"/>
-<wire x1="36.75" y1="49.5" x2="37.25" y2="49" width="0.3" layer="1"/>
-<wire x1="36.75" y1="50.47" x2="36.75" y2="49.5" width="0.3" layer="1"/>
+<wire x1="35.55" y1="48.2" x2="36.2" y2="48.2" width="0.3" layer="16"/>
 <via x="10.75" y="55.5" extent="1-16" drill="0.35"/>
-<via x="37.25" y="49" extent="1-16" drill="0.35"/>
 <contactref element="U$12" pad="P$4"/>
 <wire x1="10.75" y1="55.5" x2="10.75" y2="56.45" width="0.3" layer="1"/>
@@
 <via x="3.7" y="57" extent="1-16" drill="0.35"/>
 <wire x1="3.7" y1="57" x2="5.05" y2="57" width="0.3" layer="16"/>
+<contactref element="U1" pad="52"/>
+<via x="36.2" y="48.2" extent="1-16" drill="0.35"/>
+<wire x1="36.2" y1="49.570525" x2="36.2" y2="48.2" width="0.3" layer="1"/>
+<wire x1="36.25" y1="50.47" x2="36.25" y2="49.620525" width="0.3" layer="1"/>
+<wire x1="36.25" y1="49.620525" x2="36.2" y2="49.570525" width="0.3" layer="1"/>
 </signal>
 <signal name="TX-S">
-<contactref element="U1" pad="52"/>
 <wire x1="9.15" y1="60.55" x2="8.75" y2="60.55" width="0.3" layer="16"/>
 <wire x1="19.2" y1="50.5" x2="9.15" y2="60.55" width="0.3" layer="16"/>
 <wire x1="34.5" y1="50.5" x2="19.2" y2="50.5" width="0.3" layer="16"/>
-<wire x1="36" y1="49" x2="34.5" y2="50.5" width="0.3" layer="16"/>
-<wire x1="36.25" y1="49.25" x2="36" y2="49" width="0.3" layer="1"/>
-<wire x1="36.25" y1="50.47" x2="36.25" y2="49.25" width="0.3" layer="1"/>
+<wire x1="34.5" y1="50.5" x2="36" y2="49" width="0.3" layer="16"/>
 <via x="8.75" y="60.55" extent="1-16" drill="0.35"/>
-<via x="36" y="49" extent="1-16" drill="0.35"/>
 <contactref element="U$12" pad="P$6"/>
 <wire x1="8.75" y1="60.55" x2="7.2" y2="59" width="0.3" layer="1"/>
@@
 <via x="3.7" y="59" extent="1-16" drill="0.35"/>
 <wire x1="3.7" y1="59" x2="5.05" y2="59" width="0.3" layer="16"/>
+<contactref element="U1" pad="51"/>
+<wire x1="36" y1="49" x2="37" y2="49" width="0.3" layer="16"/>
+<via x="37" y="49" extent="1-16" drill="0.35"/>
+<wire x1="37" y1="49" x2="36.75" y2="49.25" width="0.3" layer="1"/>
+<wire x1="36.75" y1="49.25" x2="36.75" y2="50.47" width="0.3" layer="1"/>
 </signal>
 <signal name="SWC">
