File: schematics/board/SPin.brd (EAGLE design)
At the start: 71.4 x 71.4 mm, 15 parts

Commit message: Добавлены герберы плат BSK1-4, PL, SP и SPIDER
Connections:
- net 2: now also U$6.P$4
- net BUS+: now also U$6.P$5
Changed lines of the file:
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@@
 <drawing>
 <settings>
-<setting alwaysvectorfont="no"/>
+<setting alwaysvectorfont="yes"/>
 <setting verticaltext="up"/>
 </settings>
@@
 <layer number="25" name="tNames" color="7" fill="1" visible="yes" active="yes"/>
 <layer number="26" name="bNames" color="7" fill="1" visible="yes" active="yes"/>
-<layer number="27" name="tValues" color="7" fill="1" visible="no" active="yes"/>
-<layer number="28" name="bValues" color="7" fill="1" visible="no" active="yes"/>
+<layer number="27" name="tValues" color="7" fill="1" visible="yes" active="yes"/>
+<layer number="28" name="bValues" color="7" fill="1" visible="yes" active="yes"/>
 <layer number="29" name="tStop" color="7" fill="3" visible="no" active="yes"/>
 <layer number="30" name="bStop" color="7" fill="6" visible="no" active="yes"/>
@@
 <board>
 <plain>
-<text x="32.6" y="24.9" size="1.778" layer="26" rot="MR0">BUS-</text>
-<text x="45.1" y="24.8" size="1.778" layer="26" rot="MR0">BUS+</text>
-<text x="10.7" y="6.7" size="1.5" layer="26" rot="MR0">BUS+</text>
-<text x="65.7" y="6.7" size="1.5" layer="26" rot="MR0">BUS+</text>
-<text x="65.7" y="63.7" size="1.5" layer="26" rot="MR0">BUS+</text>
-<text x="10.7" y="63.7" size="1.5" layer="26" rot="MR0">BUS+</text>
-<text x="18.7" y="54.7" size="1.5" layer="26" rot="MR0">BUS-</text>
-<text x="57.7" y="54.7" size="1.5" layer="26" rot="MR0">BUS-</text>
-<text x="57.7" y="15.7" size="1.5" layer="26" rot="MR0">BUS-</text>
-<text x="18.7" y="15.7" size="1.5" layer="26" rot="MR0">BUS-</text>
+<text x="32.6" y="24.9" size="1.2" layer="26" ratio="20" rot="MR0">BUS-</text>
+<text x="45.1" y="24.8" size="1.2" layer="26" ratio="20" rot="MR0">BUS+</text>
+<text x="10.7" y="6.7" size="1.2" layer="26" ratio="20" rot="MR0">BUS+</text>
+<text x="65.7" y="6.7" size="1.2" layer="26" ratio="20" rot="MR0">BUS+</text>
+<text x="65.7" y="63.7" size="1.2" layer="26" ratio="20" rot="MR0">BUS+</text>
+<text x="10.7" y="63.7" size="1.2" layer="26" ratio="20" rot="MR0">BUS+</text>
+<text x="18.7" y="54.7" size="1.2" layer="26" ratio="20" rot="MR0">BUS-</text>
+<text x="57.7" y="54.7" size="1.2" layer="26" ratio="20" rot="MR0">BUS-</text>
+<text x="57.7" y="15.7" size="1.2" layer="26" ratio="20" rot="MR0">BUS-</text>
+<text x="18.7" y="15.7" size="1.2" layer="26" ratio="20" rot="MR0">BUS-</text>
 <wire x1="0" y1="7.071" x2="25.095" y2="32.166" width="0.1" layer="20"/>
 <wire x1="7.071" y1="0" x2="29.308534375" y2="22.237534375" width="0.1" layer="20"/>
@@
 </autorouter>
 <elements>
-<element name="U$1" library="CanCubeSat" package="KCONNECT-3" value="KCONNECT3" x="7.771" y="63.633" smashed="yes" rot="MR135">
-<attribute name="VALUE" x="0.7105375" y="65.68714375" size="1.27" layer="28" rot="MR135"/>
-</element>
-<element name="U$2" library="CanCubeSat" package="KCONNECT-3" value="KCONNECT3" x="16.256" y="55.147" smashed="yes" rot="MR315">
-<attribute name="VALUE" x="23.3164625" y="53.09285625" size="1.27" layer="28" rot="MR315"/>
-</element>
-<element name="U$3" library="CanCubeSat" package="KCONNECT-4" value="KCONNECT4" x="63.633" y="63.633" smashed="yes" rot="MR45">
-<attribute name="VALUE" x="61.578853125" y="56.5725375" size="1.27" layer="28" rot="MR45"/>
-</element>
-<element name="U$4" library="CanCubeSat" package="KCONNECT-4" value="KCONNECT4" x="55.147" y="55.147" smashed="yes" rot="MR225">
-<attribute name="VALUE" x="57.201146875" y="62.2074625" size="1.27" layer="28" rot="MR225"/>
-</element>
-<element name="U$18" library="CanCubeSat" package="KCONNECT-4" value="KCONNECT4" x="7.771" y="7.771" smashed="yes" rot="MR225">
-<attribute name="VALUE" x="9.82514375" y="14.831459375" size="1.27" layer="28" rot="MR225"/>
-</element>
-<element name="U$19" library="CanCubeSat" package="KCONNECT-1" value="KCONNECT1" x="16.256" y="16.256" smashed="yes" rot="MR225">
-<attribute name="VALUE" x="18.31014375" y="23.316459375" size="1.27" layer="28" rot="MR225"/>
-</element>
-<element name="U$20" library="CanCubeSat" package="KCONNECT-3" value="KCONNECT3" x="63.633" y="7.771" smashed="yes" rot="MR315">
-<attribute name="VALUE" x="70.693459375" y="5.716853125" size="1.27" layer="28" rot="MR315"/>
-</element>
-<element name="U$21" library="CanCubeSat" package="KCONNECT-3" value="KCONNECT3" x="55.147" y="16.256" smashed="yes" rot="MR135">
-<attribute name="VALUE" x="48.086540625" y="18.310146875" size="1.27" layer="28" rot="MR135"/>
-</element>
+<element name="U$1" library="CanCubeSat" package="KCONNECT-3" value="KCONNECT3" x="7.771" y="63.633" smashed="yes" rot="MR135"/>
+<element name="U$2" library="CanCubeSat" package="KCONNECT-3" value="KCONNECT3" x="16.256" y="55.147" smashed="yes" rot="MR315"/>
+<element name="U$3" library="CanCubeSat" package="KCONNECT-4" value="KCONNECT4" x="63.633" y="63.633" smashed="yes" rot="MR45"/>
+<element name="U$4" library="CanCubeSat" package="KCONNECT-4" value="KCONNECT4" x="55.147" y="55.147" smashed="yes" rot="MR225"/>
+<element name="U$18" library="CanCubeSat" package="KCONNECT-4" value="KCONNECT4" x="7.771" y="7.771" smashed="yes" rot="MR225"/>
+<element name="U$19" library="CanCubeSat" package="KCONNECT-1" value="KCONNECT1" x="16.256" y="16.256" smashed="yes" rot="MR225"/>
+<element name="U$20" library="CanCubeSat" package="KCONNECT-3" value="KCONNECT3" x="63.633" y="7.771" smashed="yes" rot="MR315"/>
+<element name="U$21" library="CanCubeSat" package="KCONNECT-3" value="KCONNECT3" x="55.147" y="16.256" smashed="yes" rot="MR135"/>
 <element name="JP1" library="pinhead" library_urn="urn:adsk.eagle:library:325" package="1X02" package3d_urn="urn:adsk.eagle:package:22435/2" value="" x="35.6" y="25.7" smashed="yes" rot="MR180">
 <attribute name="POPULARITY" value="98" x="35.6" y="25.7" size="1.778" layer="28" rot="MR180" display="off"/>
@@
 <element name="U$13" library="CanCubeSat" package="SOT23-3" value="SI2302CDS" x="28.7" y="63.7" smashed="yes"/>
 <element name="R13" library="resistor" package="R0603" package3d_urn="urn:adsk.eagle:package:23555/3" value="1k5" x="25.2" y="64.2" smashed="yes">
-<attribute name="VALUE" x="24.565" y="62.295" size="1.27" layer="27"/>
+<attribute name="VALUE" x="19.065" y="64.295" size="0.8" layer="27" ratio="15"/>
 </element>
 <element name="LED7" library="led" library_urn="urn:adsk.eagle:library:259" package="CHIPLED_0603" package3d_urn="urn:adsk.eagle:package:15822/2" value="" x="22.2" y="62.95" smashed="yes">
@@
 </element>
 <element name="R14" library="resistor" package="R0603" package3d_urn="urn:adsk.eagle:package:23555/3" value="1M" x="25.2" y="61.45" smashed="yes">
-<attribute name="VALUE" x="24.565" y="59.545" size="1.27" layer="27"/>
+<attribute name="VALUE" x="27.565" y="60.545" size="0.8" layer="27" ratio="15"/>
 </element>
 <element name="U$6" library="CanCubeSat" package="GRAFIT4_2" value="GRAFITGRAFIT4_2" x="35.7" y="62.7" smashed="yes" rot="R90"/>
-<element name="U$5" library="CanCubeSat" package="KCONNECT-_QUAD" value="KCONNECTQUAD-" x="35.702" y="35.702" smashed="yes">
-<attribute name="VALUE" x="32.162" y="29.257" size="1.27" layer="27"/>
-</element>
+<element name="U$5" library="CanCubeSat" package="KCONNECT-_QUAD" value="KCONNECTQUAD-" x="35.702" y="35.702" smashed="yes"/>
 </elements>
 <signals>
@@
 <contactref element="U$18" pad="3"/>
 <polygon width="0.5" layer="1" isolate="0.5" thermals="no">
-<vertex x="84.2" y="-1.8"/>
-<vertex x="84.2" y="85.1"/>
-<vertex x="-2.7" y="85.1"/>
-<vertex x="-2.7" y="-1.8"/>
+<vertex x="71.7" y="0.2"/>
+<vertex x="71.7" y="71.1"/>
+<vertex x="0.3" y="71.1"/>
+<vertex x="0.3" y="0.2"/>
 </polygon>
 <contactref element="JP1" pad="2"/>
@@
 <vertex x="40.7" y="64.7"/>
 </polygon>
+<contactref element="U$6" pad="P$5"/>
+<wire x1="39.1" y1="62.7" x2="39.2" y2="62.7" width="0" layer="19" extent="1-16"/>
 </signal>
 <signal name="BUS-">
@@
 <contactref element="U$19" pad="4"/>
 <polygon width="0.5" layer="16" isolate="0.5" thermals="no">
-<vertex x="-14.1" y="-8.2"/>
-<vertex x="89.7" y="-8.2"/>
-<vertex x="89.7" y="91.3"/>
-<vertex x="-14.1" y="91.3"/>
+<vertex x="0.4" y="0.3"/>
+<vertex x="71.7" y="0.3"/>
+<vertex x="71.7" y="71.3"/>
+<vertex x="0.4" y="71.3"/>
 </polygon>
 <polygon width="0.1" layer="16" pour="cutout">
@@
 <wire x1="32.3" y1="62.7" x2="30.3" y2="64.7" width="0.5" layer="1"/>
 <wire x1="30.3" y1="64.7" x2="28.7" y2="64.7" width="0.5" layer="1"/>
+<contactref element="U$6" pad="P$4"/>
+<wire x1="32.3" y1="62.7" x2="32.2" y2="62.7" width="0" layer="19" extent="1-16"/>
 </signal>
 </signals>
@@
 <mfgpreviewcolor name="substratecolor" color="0xFF786E46"/>
 </mfgpreviewcolors>
+<errors>
+</errors>
 </board>
 </drawing>
