File: schematics/board/SPin.sch (EAGLE design)
At the start: 45 parts

Commit message: Платы СБ
Parts:
- removed D1, D10, D11, D12, D13, D14, D15, D16, D17, D2, D3, D4, D5, D6, D7, D8, D9: MBR0520LT, diode:MBR0520LT
- removed PWR: (no value), led:LEDCHIPLED_0603
- removed R1_2K7: 2k7, rcl:R-US_R0603
- removed S1: (no value), CanCubeSat:255SB
- removed SOL1, SOL10, SOL11, SOL13, SOL14, SOL15, SOL2, SOL3, SOL5, SOL6, SOL7, SOL9: SOLAR_0, CanCubeSat:SOLAR_0
- removed SOL12, SOL16, SOL4, SOL8: SOLAR_1, CanCubeSat:SOLAR_1
- added LED7: (no value), led:LEDCHIPLED_0603
- added R13: 1k5, resistor:R-US_R0603
- added R14: 1M, resistor:R-US_R0603
- added U$13: SI2302CDS, CanCubeSat:SI2302CDS
- added U$5: KCONNECTQUAD-, CanCubeSat:KCONNECTQUAD-
- added U$6: GRAFITGRAFIT3_1, CanCubeSat:GRAFITGRAFIT3_1
Connections:
- removed net N$1: D16.A, D17.C, SOL1.OUT, SOL2.IN
- removed net N$10: D10.A, D11.C, SOL7.OUT, SOL8.IN
- removed net N$11: D10.C, D9.A, SOL8.OUT, SOL9.IN
- removed net N$12: D8.A, D9.C, SOL10.IN, SOL9.OUT
- removed net N$13: D7.A, D8.C, SOL10.OUT, SOL11.IN
- removed net N$14: D6.A, D7.C, SOL11.OUT, SOL12.IN
- removed net N$15: D5.A, D6.C, SOL12.OUT, SOL13.IN
- removed net N$16: D4.A, D5.C, SOL13.OUT, SOL14.IN
- removed net N$17: D3.A, D4.C, SOL14.OUT, SOL15.IN
- removed net N$18: D2.A, D3.C, SOL15.OUT, SOL16.IN
- removed net N$24: D13.A, D14.C, SOL4.OUT, SOL5.IN
- removed net N$3: D15.A, D16.C, SOL2.OUT, SOL3.IN
- removed net N$4: D1.A, D2.C, SOL16.OUT
- removed net N$5: PWR.A, R1_2K7.2
- removed net N$6: D14.A, D15.C, SOL3.OUT, SOL4.IN
- removed net N$7: D17.A, S1.S, SOL1.IN
- removed net N$8: D12.A, D13.C, SOL5.OUT, SOL6.IN
- removed net N$9: D11.A, D12.C, SOL6.OUT, SOL7.IN
- new net 2: R13.2, U$13.D, U$6.P$1
- new net GND: R14.2, U$13.S
- new net N$29: LED7.C, R13.1
- new net ROZE: R14.1, U$13.G, U$5.P$1
- net BUS+: now also LED7.A, U$6.P$2; no longer R1_2K7.1, S1.P
- net BUS-: no longer D1.C, PWR.C

Commit message: Плата СП изменена для возможности подключения 2 вариантов ФЭПов
Parts:
- U$6: value GRAFITGRAFIT3_1 -> GRAFITGRAFIT4_2; device CanCubeSat:GRAFITGRAFIT3_1 -> CanCubeSat:GRAFITGRAFIT4_2
Changed lines of the file:
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@@
 <part name="LED7" library="led" library_urn="urn:adsk.eagle:library:259" deviceset="LED" device="CHIPLED_0603" package3d_urn="urn:adsk.eagle:package:15822/2"/>
 <part name="R14" library="resistor" deviceset="R-US_" device="R0603" package3d_urn="urn:adsk.eagle:package:23555/3" value="1M"/>
-<part name="U$6" library="CanCubeSat" deviceset="GRAFIT" device="GRAFIT3_1"/>
+<part name="U$6" library="CanCubeSat" deviceset="GRAFIT" device="GRAFIT4_2" value="GRAFITGRAFIT4_2"/>
 <part name="U$5" library="CanCubeSat" deviceset="KCONNECT" device="QUAD-"/>
 </parts>

Commit message: Добавлены герберы плат BSK1-4, PL, SP и SPIDER
Changed lines of the file:
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@@
 <drawing>
 <settings>
-<setting alwaysvectorfont="no"/>
+<setting alwaysvectorfont="yes"/>
 <setting verticaltext="up"/>
 </settings>
