File: schematics/board/BSK1+BSK3.brd (EAGLE design)
At the start: 166 x 184 mm, 246 parts, among them Q24 Q24, U1 STM32F405RGT6, U2 LMC555

Commit message: Обновлены герберы плат BSK1-4, PL, SP и SPIDER
Parts:
- removed 2N6517, BC546: DS1820, CanCubeSat:TO92/TO226
- removed BME280: BME280BME280-PINS-ONLY, CanCubeSat:BME280-PINS-ONLY
- removed BSK2: (no value), pinheadCS:2X05
- removed C10: 10nF, rcl:C0603
- removed C11: 100pF, rcl:C0603
- removed C12, C14: 1uF, CanCubeSat:ECAP-SMD-D4
- removed C13, C9: 2,2µ, rcl:C0603
- removed C18, C2, C20, C3, C4, C6: 100nF, rcl:C0603
- removed C19: 10µ, rcl:C1206
- removed C5, C7: 22nF, rcl:C1210
- removed C8: 1nF, rcl:C0603
- removed COMPR, HEAT, TEMP, VALVE1, VALVE2: (no value), pinheadCS:1X02
- removed D1, D2, D3, D4, D5: DIODE-MBR, CanCubeSat:SOD123
- removed LED-B3, LED-G: (no value), led:CHIPLED_0603
- removed MS5611: MS5611MS5611-PIN-ONLY, CanCubeSat:MS5611-PINS-ONLY
- removed Q24: Q24, CanCubeSat:Q24
- removed R100, R103, R105, R107, R58, R60, R63, R65, R68, R71, R82, R83, R84, R85, R86: 1M, resistor:R0603
- removed R101, R104, R106, R108, R59, R61, R64, R66, R69, R72: 100R, resistor:R0603
- removed R102, R57, R62, R67, R70, R73, R74: 0.05A, rcl:R1210
- removed R109: 124k, resistor:R0603
- removed R110, R81: 22k, resistor:R0603
- removed R111, R112, R55, R56: 5k1, resistor:R0603
- removed R50, R52, R53, R89, R90, R91, R92, R93, R96, R97, R98, R99: 10k, resistor:R0603
- removed R51, R54: 2k, resistor:R0603
- removed R78: 0.5A, rcl:R1210
- removed R79: 1k, resistor:R0603
- removed R80: 4k7, resistor:R0603
- removed R87: 100k, resistor:R0603
- removed R88: 3k3, resistor:R0603
- removed SI2302-0, SI2302-10, SI2302-11, SI2302-12, SI2302-13, SI2302-14, SI2302-15, SI2302-16, SI2302-17, SI2302-9: SI2302CDS, CanCubeSat:SOT23-3
- removed STAB: ADP150AUJZ-3.3-R7, CanCubeSat:SOT23-5
- removed U$34: 100µ, CanCubeSat:ECAP100-CMD
- removed U$35, U$36, U$37, U$38: BA159, CanCubeSat:BA159
- removed U$39: 1uF, CanCubeSat:ECAP1MK
- removed U$40: DOSIM, CanCubeSat:DOSIM
- removed U$41, U$43: FFC-CONNECT68611, CanCubeSat:68611
- removed U$42: 33mH, CanCubeSat:RCH114NP
- removed U$44, U$45: 220uF, CanCubeSat:ECAP220-CMD
- removed U$46, U$47: PCB "Payload", CanCubeSat:ITS-LOGO
- removed U1: STM32F405RGT6, STM32F405RGT6:QFP50P1200X1200X160-64N
- removed U2: LMC555, LMC555CMX_NOPB:SOIC127P599X175-8N
- removed VR1: 3362H-1-502LF, CanCubeSat:TRIM_3362H-1-502LF
Connections:
- removed net 3V2: BSK2.3, C10.2, C18.2, C19.2, C2.2, C20.2, C6.2, LED-B3.A, LED-G.A, Q24.P$4, R100.2, R110.2, R111.1, R112.1, R50.2, R52.2, R53.2, R55.1, R56.1, R58.2, R60.2, R63.2, R65.2, R68.2, R71.2, R97.2, R98.2, R99.2, U$43.P$1, U$43.P$2, U1.1, U1.19, U1.32, U1.48, U1.64
- removed net 4OXV: R66.1, U1.45
- removed net 5V2: BME280.P$1, BSK2.4, C14.P+, HEAT.1, MS5611.P$1, MS5611.P$7, R88.1, STAB.P$1, STAB.P$3, U$34.P$2, U$41.P$1, U$41.P$10, U$41.P$15, U$41.P$5, U$42.P$1, U$45.P$1, U2.4, U2.8, VALVE1.1, VALVE2.1
- removed net BME280-EXT: R61.1, U1.8
- removed net BME280-INT: R101.1, U1.27
- removed net BUS+2: BSK2.10, COMPR.1, U$44.P$1
- removed net CO: R91.1, U$41.P$7, U1.16
- removed net COMPR: R106.1, U1.57
- removed net CTRL-CO-1: R91.2, R96.1, U1.35
- removed net CTRL-CO-2: R96.2, R97.1, U1.42
- removed net CTRL-NH3-1: R90.2, R93.1, U1.33
- removed net CTRL-NH3-2: R93.2, R98.1, U1.34
- removed net CTRL-NO2-1: R89.2, R92.1, U1.23
- removed net CTRL-NO2-2: R92.2, R99.1, U1.22
- removed net DOS-G: 2N6517.1, BC546.1, C4.1, C7.2, D1.A, R73.1, R87.2, U$34.P$1, U$35.P$1, U$39.P$2, U2.1
- removed net DOSE: BC546.3, C11.2, R88.2, U1.54
- removed net DOSIM: R72.1, U1.10
- removed net G-4OXV: R67.1, U$41.P$2
- removed net G-BME: R102.1, U$41.P$14
- removed net G-MICS: R74.1, U$41.P$6
- removed net G-MS: R70.1, U$41.P$11
- removed net GND-4OXV: R67.2, SI2302-12.3
- removed net GND-BME-EXT: R62.2, SI2302-10.3
- removed net GND-BME-INT: R102.2, SI2302-15.3
- removed net GND-COMPR: COMPR.2, SI2302-16.3, U$44.P$2
- removed net GND-DOSIM: R73.2, SI2302-14.3
- removed net GND-HEAT: HEAT.2, SI2302-17.3
- removed net GND-MICS: R74.2, SI2302-11.3
- removed net GND-MS-EXT: R57.2, SI2302-9.3
- removed net GND-MS-INT: R70.2, SI2302-13.3
- removed net GND-OUT: BSK2.5, BSK2.6, R78.2, U$43.P$3, U$43.P$5, U$43.P$7, U$43.P$9
- removed net GND-VALVE: SI2302-0.3, U$45.P$2, VALVE1.2, VALVE2.2
- removed net GND9: C10.1, C12.P-, C13.1, C14.P-, C18.1, C19.1, C2.1, C20.1, C3.2, C6.1, C9.1, Q24.P$2, R103.2, R105.2, R107.2, R109.1, R54.1, R78.1, SI2302-0.2, SI2302-10.2, SI2302-11.2, SI2302-12.2, SI2302-13.2, SI2302-14.2, SI2302-15.2, SI2302-16.2, SI2302-17.2, SI2302-9.2, STAB.P$2, TEMP.2, U1.12, U1.18, U1.28, U1.60, U1.63
- removed net HEAT: R108.1, U1.11
- removed net MICS: R64.1, U1.44
- removed net MS5611-EXT: R59.1, U1.9
- removed net MS5611-INT: R69.1, U1.26
- removed net N$100: R105.1, R106.2, SI2302-16.1
- removed net N$101: R107.1, R108.2, SI2302-17.1
- removed net N$102: C12.P+, C3.1, STAB.P$5, U1.13
- removed net N$103: LED-G.C, R54.2
- removed net N$65: R51.1, U1.53
- removed net N$66: C13.2, U1.47
- removed net N$67: C9.2, U1.31
- removed net N$68: C8.1, U1.5
- removed net N$69: LED-B3.C, R51.2
- removed net N$70: C8.2, Q24.P$3
- removed net N$71: R58.1, R59.2, SI2302-9.1
- removed net N$72: MS5611.P$3, MS5611.P$6, R57.1
- removed net N$73: R60.1, R61.2, SI2302-10.1
- removed net N$74: BME280.P$2, R62.1
- removed net N$75: R63.1, R64.2, SI2302-11.1
- removed net N$76: R65.1, R66.2, SI2302-12.1
- removed net N$77: R68.1, R69.2, SI2302-13.1
- removed net N$78: R71.1, R72.2, SI2302-14.1
- removed net N$79: C4.2, R79.1, U2.2, U2.6
- removed net N$80: R79.2, VR1.2, VR1.3
- removed net N$81: R80.2, U2.3, VR1.1
- removed net N$82: 2N6517.2, R80.1
- removed net N$83: 2N6517.3, C5.1, U$35.P$2, U$36.P$1, U$42.P$2
- removed net N$84: C7.1, U$36.P$2, U$37.P$1
- removed net N$85: C5.2, U$37.P$2, U$38.P$1
- removed net N$86: R81.2, R82.2, U$38.P$2, U$39.P$1
- removed net N$87: D1.C, D2.A
- removed net N$88: D2.C, D3.A
- removed net N$89: D3.C, D4.A
- removed net N$90: D4.C, D5.A
- removed net N$91: D5.C, R81.1
- removed net N$92: R82.1, R83.1
- removed net N$93: R83.2, R84.2
- removed net N$94: R84.1, R85.1
- removed net N$95: R85.2, R86.2
- removed net N$96: R86.1, U$40.P$1
- removed net N$97: BC546.2, C11.1, R87.1, U$40.P$2
- removed net N$98: R100.1, R101.2, SI2302-15.1
- removed net N$99: R103.1, R104.2, SI2302-0.1
- removed net NH3: R90.1, U$41.P$8, U1.15
- removed net NO2: R89.1, U$41.P$9, U1.14
- removed net NRST: R50.1, U$43.P$11, U1.7
- removed net O2: U$41.P$3, U1.17
- removed net RX-S: U$43.P$4, U1.52
- removed net SCL-TM2: BSK2.7, U1.29
- removed net SDA-TM2: BSK2.8, U1.30
- removed net SENS-EXT-SCL: BME280.P$3, MS5611.P$5, R112.2, U1.41
- removed net SENS-EXT-SDA: BME280.P$4, MS5611.P$4, R111.2, U1.40
- removed net SENS-INT-SCL: R55.2, U$41.P$12, U1.58
- removed net SENS-INT-SDA: R56.2, U$41.P$13, U1.59
- removed net SWC: R53.1, U$43.P$10, U1.49
- removed net SWD: R52.1, U$43.P$8, U1.46
- removed net TEMP: R109.2, R110.1, TEMP.1, U1.20
- removed net TIME1: BSK2.9, U1.50
- removed net TX-S: U$43.P$6, U1.51
- removed net VALVE: R104.1, U1.61
Routing:
- net GND9: track 340.6 -> 0.00 mm, vias 16 -> 0
- net 5V2: track 290.7 -> 0.00 mm, vias 3 -> 0
- net 3V2: track 270.7 -> 0.00 mm, vias 21 -> 0
- net GND-OUT: track 265.5 -> 0.00 mm, vias 2 -> 0
- net BUS+2: track 141.3 -> 0.00 mm
- net DOS-G: track 99.6 -> 0.00 mm, vias 13 -> 0
- net DOSE: track 98.7 -> 0.00 mm, vias 2 -> 0
- net TIME1: track 69.1 -> 0.00 mm, vias 3 -> 0
- net SENS-EXT-SDA: track 65.5 -> 0.00 mm, vias 1 -> 0
- net O2: track 64.9 -> 0.00 mm, vias 2 -> 0
- net SENS-INT-SDA: track 62.8 -> 0.00 mm
- net SENS-INT-SCL: track 61.1 -> 0.00 mm
- net SENS-EXT-SCL: track 59.5 -> 0.00 mm, vias 1 -> 0
- net CO: track 56.5 -> 0.00 mm, vias 2 -> 0
- net NO2: track 55.5 -> 0.00 mm, vias 2 -> 0
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- removed copper zone on layer 1, net DOS-G
- removed copper zone on layer 16, net DOS-G
- removed copper zone on layer 1, net GND9
- removed copper zone on layer 16, net GND9
Other:
- board size 166 x 184 mm -> 166 x 100 mm
- board text removed: "PC12"
- board text removed: "PWR"
- board text removed: "for firmware"
- board text removed: "to BSK1"
- board text removed: "to Sealed housing"
