File: schematics/board/ARK.sch (EAGLE design)
At the start: 213 parts, among them IC2 STM32F103C8T, Q5 8MHz

Commit message: Обновлен список плат, работа над платой ПН
Parts:
- removed AB1, AB2, AB3: (no value), pinheadCS:PINHD-1X8
- removed C1, C10, C11, C12, C17, C18, C19, C2, C20, C21, C22, C23, C24, C25, C26, C27, C28, C3, C32, C4, C5, C6, C7, C8, C9: 0,1µ, rcl:C-USC0603
- removed C42: 1µ, rcl:C-USC0603
- removed C43: 10µ, rcl:C-USC1206
- removed LED4, LED5, LED6, LED7: (no value), led:LEDCHIPLED_0603
- removed R1, R17, R33, R41, R49, R80, R83, R84, R85, R86, R9: 2k, resistor:R-US_R0603
- removed R10, R11, R18, R19, R2, R3, R34, R35, R42, R43, R50, R51: 330R, resistor:R-US_R0603
- removed R12, R13, R14, R15, R20, R21, R22, R23, R36, R37, R38, R39, R4, R44, R45, R46, R47, R5, R52, R53, R54, R55, R6, R7, R88, R89, R90, R91, R92, R93, R94, R95, R96, R97, R98, R99: 100R, resistor:R-US_R0603
- removed R16, R24, R40, R48, R56, R8: R05, rcl:R-US_R2512
- removed R63: 1M, resistor:R-US_R0603
- removed U$1, U$15, U$24, U$25, U$26, U$8: FS8205A-, CanCubeSat:FS8205A-
- removed U$10, U$17, U$3, U$31, U$38, U$45: HY2120, CanCubeSat:HY2120
- removed U$11, U$12, U$18, U$19, U$32, U$33, U$39, U$4, U$40, U$46, U$47, U$5: HY2213, CanCubeSat:HY2213
- removed U$13, U$14, U$20, U$21, U$34, U$35, U$41, U$42, U$48, U$49, U$6, U$7: SI2302CDS, CanCubeSat:SI2302CDS
- removed U$60: AD5272, CanCubeSat:AD5272
- added LED1, LED2: (no value), led:LEDCHIPLED_0603
- added R31, R32, R57: 2k, resistor:R-US_R0603
- added U$2: INVERTER, CanCubeSat:INVERTER
- R70: value 14k3 -> 24k3
- R72: value 91k -> 232k
Connections:
- removed net B-1: AB1.6, C1.2, C2.2, C4.2, R8.2, R86.1, U$3.VSS, U$5.VSS, U$7.D
- removed net B-2: AB1.1, C25.2, C26.2, C28.2, R100.1, R56.2, U$45.VSS, U$47.VSS, U$49.D
- removed net B-3: AB2.6, C5.2, C6.2, C8.2, R16.2, R84.1, U$10.VSS, U$12.VSS, U$14.D
- removed net B-4: AB2.1, C21.2, C22.2, C24.2, R48.2, R85.1, U$38.VSS, U$40.VSS, U$42.D
- removed net B-5: AB3.6, C10.2, C12.2, C9.2, R24.2, R83.1, U$17.VSS, U$19.VSS, U$21.D
- removed net B-6: AB3.1, C17.2, C18.2, C20.2, R40.2, R80.1, U$31.VSS, U$33.VSS, U$35.D
- removed net DPC_RST: IC2.PB14, U$60.RESET
- removed net N$1: C1.1, R2.1, U$3.VDD
- removed net N$10: R5.1, U$7.S
- removed net N$100: U$46.OUT, U$48.G
- removed net N$101: R52.1, U$48.S
- removed net N$102: U$47.OUT, U$49.G
- removed net N$103: R53.1, U$49.S
- removed net N$104: R49.2, R56.1, U$1.S2
- removed net N$107: C26.1, R51.1, U$45.VC
- removed net N$108: C28.1, R55.1, U$47.VDD
- removed net N$110: AB1.2, C27.2, R51.2, R53.2, R55.2, U$46.VSS, U$48.D
- removed net N$13: R1.2, R8.1, U$26.S2
- removed net N$15: C2.1, R3.1, U$3.VC
- removed net N$154: C42.1, U$60.CAP
- removed net N$16: C5.1, R10.1, U$10.VDD
- removed net N$18: R9.1, U$10.CS
- removed net N$19: C7.1, R14.1, U$11.VDD
- removed net N$2: C4.1, R7.1, U$5.VDD
- removed net N$20: U$11.OUT, U$13.G
- removed net N$21: R12.1, U$13.S
- removed net N$22: U$12.OUT, U$14.G
- removed net N$23: R13.1, U$14.S
- removed net N$24: R16.1, R9.2, U$25.S2
- removed net N$27: C6.1, R11.1, U$10.VC
- removed net N$28: C8.1, R15.1, U$12.VDD
- removed net N$3: R1.1, U$3.CS
- removed net N$30: AB2.7, C7.2, R11.2, R13.2, R15.2, U$11.VSS, U$13.D
- removed net N$33: C9.1, R18.1, U$17.VDD
- removed net N$34: R17.1, U$17.CS
- removed net N$35: C11.1, R22.1, U$18.VDD
- removed net N$36: U$18.OUT, U$20.G
- removed net N$37: R20.1, U$20.S
- removed net N$38: U$19.OUT, U$21.G
- removed net N$39: R21.1, U$21.S
- removed net N$4: C3.1, R6.1, U$4.VDD
- removed net N$40: R17.2, R24.1, U$24.S2
- removed net N$43: C10.1, R19.1, U$17.VC
- removed net N$44: C12.1, R23.1, U$19.VDD
- removed net N$45: C32.1, C39.1, C43.1, U$59.SVCC, U$59.VCC, U$60.VDD
- removed net N$46: AB3.7, C11.2, R19.2, R21.2, R23.2, U$18.VSS, U$20.D
- removed net N$53: R63.1, U$16.RUN
- removed net N$57: LED5.A, R84.2
- removed net N$58: LED6.A, R85.2
- removed net N$59: LED7.A, R86.2
- removed net N$6: U$4.OUT, U$6.G
- removed net N$65: C17.1, R34.1, U$31.VDD
- removed net N$66: R33.1, U$31.CS
- removed net N$67: C19.1, R38.1, U$32.VDD
- removed net N$68: U$32.OUT, U$34.G
- removed net N$69: R36.1, U$34.S
- removed net N$7: R4.1, U$6.S
- removed net N$70: U$33.OUT, U$35.G
- removed net N$71: R37.1, U$35.S
- removed net N$72: R33.2, R40.1, U$15.S2
- removed net N$75: C18.1, R35.1, U$31.VC
- removed net N$76: C20.1, R39.1, U$33.VDD
- removed net N$78: AB3.2, C19.2, R35.2, R37.2, R39.2, U$32.VSS, U$34.D
- removed net N$8: AB1.7, C3.2, R3.2, R5.2, R7.2, U$4.VSS, U$6.D
- removed net N$81: C21.1, R42.1, U$38.VDD
- removed net N$82: R41.1, U$38.CS
- removed net N$83: C23.1, R46.1, U$39.VDD
- removed net N$84: U$39.OUT, U$41.G
- removed net N$85: R44.1, U$41.S
- removed net N$86: U$40.OUT, U$42.G
- removed net N$87: R45.1, U$42.S
- removed net N$88: R41.2, R48.1, U$8.S2
- removed net N$9: U$5.OUT, U$7.G
- removed net N$91: C22.1, R43.1, U$38.VC
- removed net N$92: C24.1, R47.1, U$40.VDD
- removed net N$94: AB2.2, C23.2, R43.2, R45.2, R47.2, U$39.VSS, U$41.D
- removed net N$97: C25.1, R50.1, U$45.VDD
- removed net N$98: R49.1, U$45.CS
- removed net N$99: C27.1, R54.1, U$46.VDD
- removed net OC1: R95.2, U$26.G2, U$3.OC
- removed net OC2: R99.2, U$1.G2, U$45.OC
- removed net OC3: R93.2, U$10.OC, U$25.G2
- removed net OC4: R97.2, U$38.OC, U$8.G2
- removed net OC5: R91.2, U$17.OC, U$24.G2
- removed net OC6: R89.2, U$15.G2, U$31.OC
- removed net OD1: R94.2, U$26.G1, U$3.OD
- removed net OD2: R98.2, U$1.G1, U$45.OD
- removed net OD3: R92.2, U$10.OD, U$25.G1
- removed net OD4: R96.2, U$38.OD, U$8.G1
- removed net OD5: R90.2, U$17.OD, U$24.G1
- removed net OD6: R88.2, U$15.G1, U$31.OD
- new net A: C39.1, LED8.A, U$2.A, U$59.SVCC, U$59.VCC
- new net Y: U$16.RUN, U$2.Y
- net 1W: no longer AB1.5, AB2.5, AB3.5
- net BMS+: no longer AB1.8, AB2.8, AB3.8, LED3.C, LED4.C, LED5.C, LED6.C, LED7.C, LED8.C, R10.2, R12.2, R14.2, R18.2, R2.2, R20.2, R22.2, R34.2, R36.2, R38.2, R4.2, R42.2, R44.2, R46.2, R50.2, R52.2, R54.2, R6.2
- net BMS1: no longer R94.1, R95.1
- net BMS2: no longer R98.1, R99.1
- net BMS3: no longer R92.1, R93.1
- net BMS4: no longer R96.1, R97.1
- net BMS5: no longer R90.1, R91.1
- net BMS6: no longer R88.1, R89.1
- net GND: now also R100.1, R31.1, R32.1, R57.1, R70.2, U$2.GND; no longer AB1.4, AB2.4, AB3.4, C32.2, C42.2, C43.2, R70.1, U$1.S1, U$15.S1, U$24.S1, U$25.S1, U$26.S1, U$60.VSS, U$60.W, U$8.S1
- net INA_BMS+: no longer R63.2
- net N$25: now also R70.1; no longer U$60.A
- net N$26: now also LED1.C, R31.2; no longer R70.2, U$60.GND
- net N$47: now also LED1.A
- net N$54: now also LED2.C, R32.2; no longer LED3.A, R80.2
- net N$56: now also LED3.C, R57.2; no longer LED4.A, R83.2
- net N$60: now also LED8.C; no longer LED8.A
- net PGOOD1: now also LED2.A
- net PGOOD2: now also LED3.A
- net SCL: no longer U$60.SCL
- net SDA: no longer U$60.SDA
- net VDD: now also INA219#1.VS, U$2.VCC, U$57.VS; no longer AB1.3, AB2.3, AB3.3, INA219#1.VCC, U$57.VCC, U$60.ADDR
Other:
- note added: "Charge DC-DC"
- note added: "Discharge DC-DC"
- moved on the sheet: BSK4, C005R, C13, C14, C15, C16, C29, C30, C31, C33, C34, C35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

Commit message: Добавлены герберы плат BSK1-4, PL, SP и SPIDER
Parts:
- removed BSK4: (no value), pinheadCS:PINHD-1X8
- removed C005R: 32,768KHz, CanCubeSat:C005R
- removed C13, C14, C33, C34, C51: 0,1µ, rcl:C-USC0603
- removed C30, C36: 680p, rcl:C-USC0603
- removed C31, C39: 4.7µ, rcl:C-USC1206
- removed C35: 150µ, CanCubeSat:ECAPECAP150
- removed C37: 220µ, CanCubeSat:ECAPECAP220
- removed C38: 3,3n, rcl:C-USC0603
- removed LED1, LED2, LED3, LED8: (no value), led:LEDCHIPLED_0603
- removed MICRO: 629105136821, MicroUSB:629105136821
- removed Q5: 8MHz, 9C-8.000MEEJ-T:9C-8.000MEEJ-T
- removed R25, R26: 5k1, resistor:R-US_R0603
- removed R29: 150k, resistor:R-US_R0603
- removed R31: 2k, resistor:R-US_R0603
- removed R61: 91K, resistor:R-US_R0603
- removed R62, R72: 232k, resistor:R-US_R0603
- removed R70: 24k3, resistor:R-US_R0603
- removed R78: 1M, resistor:R-US_R0603
- removed R87: 680k, resistor:R-US_R0603
- removed S1: (no value), cansat-lib:UNICS-SWITCH
- removed U$16: LTC3119, CanCubeSat:LTC3119
- added C1: 1nF, rcl:C-EUC0603
- added C10, C56, C9: 0,1µ, rcl:C-USC0603
- added C2: 10nF, rcl:C-EUC0603
- added C3, C57: 10µ, rcl:C-USC1206
- added C4, C5, C6, C7, C8: 100nF, rcl:C-EUC0603
- added CAM1, CAM2, SWITCH: (no value), pinheadCS:PINHD-1X2
- added INVERT: INVERTER., CanCubeSat:INVERTER.
- added JP1: (no value), pinheadCS:PINHD-2X8
- added LD1117S33: LD1117S33, CanCubeSat:LD1117S33
- added LED_G1, LED_G2, LED_R1, LED_R2: (no value), led:LEDCHIPLED_0603
- added OPA: OPA333, CanCubeSat:OPA333
- added R1: 91K, resistor:R-US_R0603
- added R2: 3313J-1-205E, CanCubeSat:3313J-1-205E
- added R3: 14K3, resistor:R-US_R0603
- added R33: 2k, resistor:R-US_R0603
- added R4, R5, R6: 3314G-1-504E, CanCubeSat:3314G-1-504E
- added U$1: MF-R400, CanCubeSat:MF-R400
- added U$12: FFC-CONNECT68611, CanCubeSat:FFC-CONNECT68611
- 3,3µH1: value 3,3µ -> 3,3µH
- C44: value 27pF -> 680p; device rcl:C-EUC0603 -> rcl:C-USC0603
- C45: value 27pF -> 4.7µ; device rcl:C-EUC0603 -> rcl:C-USC1206
- C46: value 10pF -> 3,3n; device rcl:C-EUC0603 -> rcl:C-USC0603
- C47: value 10pF -> 150µ; device rcl:C-EUC0603 -> CanCubeSat:ECAPECAP150
- C48, C55: value 100nF -> 220µ; device rcl:C-EUC0603 -> CanCubeSat:ECAPECAP220
- C49: value 150µ -> 0,1µ; device CanCubeSat:ECAPECAP150 -> rcl:C-USC0603
- C50: value 220µ -> 0,1µ; device CanCubeSat:ECAPECAP220 -> rcl:C-USC0603
- C52: value 10µ -> 680p; device rcl:C-USC1206 -> rcl:C-USC0603
- C53: value 100nF -> 4.7µ; device rcl:C-EUC0603 -> rcl:C-USC1206
- C54: value 100nF -> 150µ; device rcl:C-EUC0603 -> CanCubeSat:ECAPECAP150
- R30: value 14K3 -> 150k
- U$2: value INVERTER -> Q24; device CanCubeSat:INVERTER -> CanCubeSat:Q24
- U$23: value USB-C -> LTC31191; device CanCubeSat:USB-C -> CanCubeSat:LTC31191
- U$59: value LTC3119 -> LTC31191; device CanCubeSat:LTC3119 -> CanCubeSat:LTC31191
Connections:
- removed net I2CINT: BSK4.3, IC2.PB7
- removed net N$11: 3,3µH1.2, C13.1, U$16.SW1
- removed net N$12: 3,3µH1.1, C14.1, U$16.SW2
- removed net N$133: C44.1, IC2.OSC_OUT, Q5.1, R78.1
- removed net N$145: C45.1, IC2.OSC_IN, Q5.2, R78.2
- removed net N$148: C005R.2, C47.1, IC2.PC15
- removed net N$152: C005R.1, C46.1, IC2.PC14
- removed net N$25: R70.1, R72.1, U$59.FB
- removed net N$26: LED1.C, R31.2
- removed net N$29: R28.2, U$16.RT
- removed net N$32: C13.2, U$16.BST1
- removed net N$41: R29.1, U$16.VC
- removed net N$42: C30.1, R29.2
- removed net N$47: AD5272#2.VDD, C31.1, C51.1, C52.1, LED1.A, U$16.MPPC, U$16.SVCC, U$16.VCC
- removed net N$5: AD5272#2.A, R61.1, U$16.FB
- removed net N$52: C14.2, U$16.BST2
- removed net N$54: LED2.C, R32.2
- removed net N$55: R62.2, R87.1, U$59.RUN
- removed net N$56: LED3.C, R57.2
- removed net N$60: LED8.C, R100.2
- removed net RX-C: IC2.PA10, U$23.RX0
- removed net TX-C: IC2.PA9, U$23.TX0
- removed net VDD: BSK4.6, C15.1, C16.1, C48.1, C53.1, C54.1, C55.1, IC2.VBAT, IC2.VDDA, INA219#1.VS, PB5.A, PWR.A, R101.1, R102.1, R25.1, R26.1, R27.1, R64.1, R79.1, U$2.VCC, U$23.3V3/BUS, U$57.A0, U$57.VS
- new net 1.65: R4.WIPER, R5.CW
- new net 302: OPA.IN-, R5.WIPER
- new net 3V3: C15.1, C16.1, C2.2, C5.1, C6.1, C7.1, C8.1, IC2.VBAT, IC2.VDDA, INA219#1.VS, JP1.9, PB5.A, PWR.A, R101.1, R102.1, R27.1, R64.1, R79.1, U$12.1, U$12.2, U$2.VCC, U$57.A0, U$57.VS
- new net 3V3-STAB: C3.1, INVERT.VCC, LD1117S33.VOUT, OPA.V+, R4.CCW
- new net GND-OUT: CAM1.2, CAM2.2, JP1.11, JP1.12, U$1.P$2, U$12.3, U$12.5, U$12.7, U$12.9
- new net N$1: C1.1, IC2.OSC_IN
- new net N$215: AD5272#2.VDD, C53.1, C56.1, C57.1, LED_G2.A, U$23.MPPC, U$23.SVCC, U$23.VCC
- new net N$234: C45.1, LED_G1.A, U$59.SVCC, U$59.VCC
- new net N$3: AD5272#2.A, R1.2, U$23.FB
- new net N$4: C1.2, U$2.OUTPUT
- new net N$77: 3,3µH1.2, C49.1, U$23.SW1
- new net N$78: 3,3µH1.1, C50.1, U$23.SW2
- new net N$79: R28.2, U$23.RT
- new net N$80: C49.2, U$23.BST1
- new net N$81: R30.1, U$23.VC
- new net N$82: C52.1, R30.2
- new net N$84: C50.2, U$23.BST2
- new net N$85: LED_R1.A, R32.2
- new net N$87: LED_R2.A, R57.2
- new net N$89: R6.WIPER, U$59.FB
- new net N$91: LED_G1.C, R100.2
- new net N$92: LED_G2.C, R33.2
- new net RUN: OPA.IN+, R2.WIPER
- new net RX-S: IC2.PA10, U$12.4
- new net TX-S: IC2.PA9, U$12.6
- net 1W: now also JP1.7
- net 5V: now also CAM1.1, CAM2.1, JP1.10; no longer BSK4.8, MICRO.1
- net A: now also INVERT.A, OPA.OUT, R32.1, R5.CCW, U$59.RUN; no longer C39.1, LED8.A, U$2.A, U$59.SVCC, U$59.VCC
- net BMS+: now also C4.1, JP1.8, LD1117S33.VIN
- net BMS1: now also IC2.PA6, JP1.1; no longer IC2.PA5
- net BMS2: now also IC2.PA5, JP1.2; no longer IC2.PA6
- net BMS3: now also IC2.PA4, JP1.3; no longer IC2.PA3
- net BMS4: now also IC2.PA3, JP1.4; no longer IC2.PA4
- net BMS5: now also IC2.PA2, JP1.5; no longer IC2.PA1
- net BMS6: now also IC2.PA1, JP1.6; no longer IC2.PA2
- net BUS+: now also SWITCH.2; no longer S1.P
- net BUSPLUS: now also JP1.16, SWITCH.1; no longer BSK4.7, S1.O
- net GND: now also C2.1, C3.2, C4.2, C5.2, C56.2, C57.2, C6.2, C7.2, C8.2, INVERT.GND, LD1117S33.GND, OPA.V-, R2.CW, R3.2, R33.1, R4.CW, R6.CW, U$1.P$1, U$23.PGND, U$23.PWM, U$23.SGND; no longer BSK4.1, C30.2, C31.2, C35.2, C36.2, C37.2, C38.2, C39.2, C49.2, C50.2, C51.2, MICRO.5, R30.2, R31.1, R32.1, R57.1, R62.1, R70.2, U$16.PGND, U$16.PWM, U$16.SGND, U$23.GND
- net INA_BMS+: now also C47.1, C55.1, R6.CCW, U$23.PVIN, U$23.VIN; no longer C35.1, C50.1, R72.2, U$16.PVIN, U$16.VIN
- net INA_BUS+: now also C48.1, C54.1, R1.1, R2.CCW, U$23.PVOUT; no longer C37.1, C49.1, R61.2, R87.2, U$16.PVOUT
- net N$129: now also C41.2; no longer C34.2
- net N$131: now also C40.1; no longer C33.1
- net N$132: now also C41.1; no longer C34.1
- net N$136: now also C44.1; no longer C36.1
- net N$139: now also C46.1; no longer C38.1
- net N$14: now also C9.2; no longer C40.2
- net N$144: now also C40.2; no longer C33.2
- net N$147: now also C9.1; no longer C40.1
- net N$150: now also C10.1; no longer C41.1
- net N$151: now also C10.2; no longer C41.2
- net N$48: now also R3.1; no longer R30.1
- net NRST: now also U$12.11; no longer U$23.NRST/EN
- net PGOOD1: now also IC2.PB1, LED_R1.C; no longer IC2.PB0, LED2.A
- net PGOOD2: now also IC2.PB0, LED_R2.C, U$23.PGOOD; no longer IC2.PB1, LED3.A, U$16.PGOOD
- net SCLTM: now also JP1.13; no longer BSK4.5, R25.2
- net SDATM: now also JP1.14; no longer BSK4.4, R26.2
- net SWC: now also U$12.10; no longer U$23.SWC/TXD
- net SWD: now also U$12.8; no longer U$23.SWD/RXD
- net TIME: now also JP1.15; no longer BSK4.2
- net Y: now also INVERT.Y, R57.1, U$23.RUN; no longer U$16.RUN, U$2.Y
Other:
- moved on the sheet: C15, C16, C29, C40, C41, C44, C45, C46, C47, C48, C49, C50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

Commit message: Исправления АРКа
Parts:
- removed C4: 100nF, rcl:C-EUC0603
- removed LD1117S33: LD1117S33, CanCubeSat:LD1117S33
- added R7: 680k, resistor:R-US_R0603
- added U$6: REF3033, CanCubeSat:REF3033
- C3: value 10µ -> 470nF; device rcl:C-USC1206 -> rcl:C-EUC0603
- R4: value 3314G-1-504E -> 120k; device CanCubeSat:3314G-1-504E -> resistor:R-US_R0603
- R5: value 3314G-1-504E -> 430k; device CanCubeSat:3314G-1-504E -> resistor:R-US_R0603
Connections:
- removed net 1.65: R4.WIPER, R5.CW
- removed net 302: OPA.IN-, R5.WIPER
- new net N$2: OPA.IN+, R4.2, R5.2, R7.2
- net 3V3: now also IC2.VDD; no longer IC2.VDDA
- net 3V3-STAB: now also IC2.VDDA, R4.1, U$6.OUT; no longer C3.1, LD1117S33.VOUT, R4.CCW
- net 5V: now also C3.2, U$6.IN
- net A: now also R7.1, U$23.RUN; no longer R5.CCW, U$59.RUN
- net BMS+: no longer C4.1, LD1117S33.VIN
- net GND: now also C3.1, R5.1, U$6.GND; no longer C3.2, C4.2, LD1117S33.GND, R4.CW
- net PGOOD1: now also LED_R2.C; no longer LED_R1.C
- net PGOOD2: now also LED_R1.C; no longer LED_R2.C
- net RUN: now also OPA.IN-; no longer OPA.IN+
- net Y: now also U$59.RUN; no longer U$23.RUN
Other:
- moved on the sheet: C15, C16, C3, C6, C7, C8, R2

Commit message: Плата АРК готова к проверке
Parts:
- removed CAM1, CAM2: (no value), pinheadCS:PINHD-1X2
- removed R2: 3313J-1-205E, CanCubeSat:3313J-1-205E
- removed R6: 3314G-1-504E, CanCubeSat:3314G-1-504E
- removed U$6: REF3033, CanCubeSat:REF3033
- added C11: 1uF, CanCubeSat:ECAP1UF
- added C4: 10uF, CanCubeSat:ECAP1UF
- added LD1117S33: LD1117S33, CanCubeSat:LD1117S33
- added REF3033: REF3033, CanCubeSat:REF3033
- added VR-FB: 3314G-1-504E, CanCubeSat:3314G-1-504E
- added VR-RUN: 3313J-1-205E, CanCubeSat:3313J-1-205E
Connections:
- removed net 5V: C3.2, CAM1.1, CAM2.1, JP1.10, U$6.IN
- new net 5V-OUT: JP1.10
- net 3V3: now also C4.1, LD1117S33.VOUT; no longer JP1.9
- net 3V3-STAB: now also REF3033.OUT; no longer U$6.OUT
- net BMS+: now also C11.1, C3.2, LD1117S33.VIN, REF3033.IN
- net GND: now also C11.2, C4.2, LD1117S33.GND, REF3033.GND, VR-FB.CW, VR-RUN.CW; no longer R2.CW, R6.CW, U$6.GND
- net GND-OUT: no longer CAM1.2, CAM2.2
- net INA_BMS+: now also VR-FB.CCW; no longer R6.CCW
- net INA_BUS+: now also VR-RUN.CCW; no longer R2.CCW
- net N$89: now also VR-FB.WIPER; no longer R6.WIPER
- net RUN: now also VR-RUN.WIPER; no longer R2.WIPER
Other:
- moved on the sheet: C10, C29, C3, C40, C41, C44, C45, C46, C47, C48, C49, C50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

Commit message: Украсил плату АРК
Parts:
- added U$3, U$4: PCB-"ARK", CanCubeSat:ITS-LOGOPCB-""
Connections:
- removed net 5V-OUT: JP1.10
- removed net BUSPLUS: JP1.16, SWITCH.1
- new net BMS+_OUT: JP1.8, SWITCH.1
- net BMS+: now also SWITCH.2; no longer JP1.8
- net BUS+: now also JP1.16; no longer SWITCH.2
Other:
- note added: "Датчики тока на шинах BUS+ и BMS+"
- note added: "Заряжающий АБ DC-DC"
- note added: "Интерфейс для прошивки"
- note added: "Интерфейс материнской платы"
- note added: "Источник опорного напряжения 3V3-STUB"
- note added: "Микроконтроллер STM32F103"
- note added: "Предохранитель и выключатель АРКа"
- note added: "Разряжающий АБ DC-DC"
- note added: "Стабилизатор напряжения 3V3"
- note added: "Управления работой DC-DC по уровню напряжения на шине BUS+"
- moved on the sheet: C1, C10, C11, C15, C16, C2, C29, C3, C4, C40, C41, C44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
