File: schematics/board/BKU.sch (EAGLE design)
At the start: 48 parts

Commit message: Сделаны платы CROSSnew, SPIDERnew, BSK2
Parts:
- removed BSK2A: (no value), pinheadCS:PINHD-1X8
- added BSK1: (no value), pinheadCS:PINHD-1X20
- BSK3: device pinheadCS:PINHD-1X12 -> pinheadCS:PINHD-1X14
- BSK4: device pinheadCS:PINHD-1X14 -> pinheadCS:PINHD-1X8
Connections:
- new net 3V3: BSK1.8, BSK3.8
- new net B1-CMD: BSK1.4
- new net B1-KHEAT: BSK1.1
- new net B1-KVCC: BSK1.2
- new net B1-ROZE: BSK1.3
- new net B2-CMD: BSK2.4
- new net B2-KHEAT: BSK2.1
- new net B2-KVCC: BSK2.2
- new net B2-ROZE: BSK2.3
- new net B3-CMD: BSK3.4
- new net B3-KHEAT: BSK3.1
- new net B3-KVCC: BSK3.2
- new net B3-ROZE: BSK3.3
- new net B4-CMD: BSK4.4
- new net B4-KHEAT: BSK4.1
- new net B4-KVCC: BSK4.2
- new net B4-ROZE: BSK4.3
- new net B5-CMD: BSK3.13
- new net B5-KHEAT: BSK3.10
- new net B5-KVCC: BSK3.11
- new net B5-ROZE: BSK3.12
- new net PL1-KVCC: BSK1.15
- new net PL2-KVCC: BSK1.16
- new net PL3-KVCC: BSK1.17
- new net PL4-KVCC: BSK1.18
- new net PL5-KVCC: BSK1.19
- new net PL6-KVCC: BSK1.20
- new net SCL: BSK1.10
- new net SDA: BSK1.12
- new net SINS-KVCC: BSK3.14
- net 1W: now also BSK1.5, BSK2.5, BSK3.5, BSK4.5; no longer BSK2.6, BSK2A.6, BSK3.8, BSK4.14
- net 5V: now also BSK1.7, BSK3.7, BSK4.7; no longer BSK2A.7, BSK3.9, BSK4.2
- net B2A_KEM+: no longer BSK2A.3
- net B2A_KEM-: no longer BSK2A.2
- net B2A_KHEAT: no longer BSK2A.4
- net B2A_KVCC: no longer BSK2A.5
- net B2_KEM+: no longer BSK2.3
- net B2_KEM-: no longer BSK2.2
- net B2_KHEAT: no longer BSK2.4
- net B2_KVCC: no longer BSK2.5
- net B3_KEM+: no longer BSK3.5
- net B3_KEM-: no longer BSK3.4
- net B3_KHEAT: no longer BSK3.6
- net B3_KVCC: no longer BSK3.7
- net B4_KEM+: no longer BSK4.11
- net B4_KEM-: no longer BSK4.10
- net B4_KHEAT: no longer BSK4.12
- net B4_KVCC: no longer BSK4.13
- net B5_KEM+: no longer BSK3.2
- net B5_KEM-: no longer BSK3.1
- net B5_KHEAT: no longer BSK3.11
- net B5_KVCC: no longer BSK3.12
- net BUS+: now also BSK1.6, BSK2.6, BSK3.6, BSK4.6; no longer BSK2.8, BSK2A.8, BSK3.10, BSK4.3
- net GND: now also BSK1.11, BSK1.9, BSK2.8, BSK3.9, BSK4.8; no longer BSK2.1, BSK2A.1, BSK3.3, BSK4.9
- net I2CINT: no longer BSK4.5
- net PL_KVCC: no longer BSK4.8
- net SCLTM: no longer BSK4.7
- net SDATM: no longer BSK4.6
- net TIME: now also BSK1.14; no longer BSK4.4
- net TIME-ES: now also BSK1.13
- net VDD: no longer BSK4.1
Other:
- moved on the sheet: BSK2

Commit message: Разведена БСК1
Parts:
- BSK2, BSK4: device pinheadCS:PINHD-1X8 -> pinheadCS:PINHD-1X10
- BSK3: device pinheadCS:PINHD-1X14 -> pinheadCS:PINHD-1X16
Connections:
- removed net SCL: BSK1.10
- removed net SCLTM: R10.2, U$13.IO16
- removed net SDA: BSK1.12
- removed net SDATM: R11.2, U$13.IO17
- new net SCL-INA: BSK2.9, BSK3.15, BSK4.9
- new net SCL-TM: BSK1.10, R10.2, U$13.IO16
- new net SDA-INA: BSK2.10, BSK3.16, BSK4.10
- new net SDA-TM: BSK1.12, R11.2, U$13.IO17
Changed lines of the file:
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@@
 <part name="R6" library="resistor" library_urn="urn:adsk.eagle:library:348" deviceset="R-US_" device="R0603" package3d_urn="urn:adsk.eagle:package:23555/3" value="5k1"/>
 <part name="U$6" library="CanCubeSat" deviceset="USB-C" device=""/>
-<part name="BSK3" library="pinheadCS" deviceset="PINHD-1X14" device=""/>
-<part name="BSK2" library="pinheadCS" deviceset="PINHD-1X8" device=""/>
-<part name="BSK4" library="pinheadCS" deviceset="PINHD-1X8" device=""/>
+<part name="BSK3" library="pinheadCS" deviceset="PINHD-1X16" device=""/>
+<part name="BSK2" library="pinheadCS" deviceset="PINHD-1X10" device=""/>
+<part name="BSK4" library="pinheadCS" deviceset="PINHD-1X10" device=""/>
 <part name="U$18" library="CanCubeSat" deviceset="74HC595" device=""/>
 <part name="U$19" library="CanCubeSat" deviceset="74HC595" device=""/>
@@
 </instance>
 <instance part="U$6" gate="G$1" x="353.06" y="119.38" smashed="yes"/>
-<instance part="BSK3" gate="A" x="226.06" y="157.48" smashed="yes" rot="MR270">
-<attribute name="NAME" x="247.015" y="156.21" size="1.778" layer="95" rot="MR90"/>
-<attribute name="VALUE" x="246.38" y="163.83" size="1.778" layer="96" rot="MR270"/>
+<instance part="BSK3" gate="A" x="228.6" y="157.48" smashed="yes" rot="MR270">
+<attribute name="NAME" x="252.095" y="156.21" size="1.778" layer="95" rot="MR90"/>
+<attribute name="VALUE" x="248.92" y="163.83" size="1.778" layer="96" rot="MR270"/>
 </instance>
 <instance part="BSK2" gate="A" x="223.52" y="190.5" smashed="yes" rot="MR270">
-<attribute name="NAME" x="234.315" y="189.23" size="1.778" layer="95" rot="MR90"/>
+<attribute name="NAME" x="239.395" y="189.23" size="1.778" layer="95" rot="MR90"/>
 <attribute name="VALUE" x="236.22" y="196.85" size="1.778" layer="96" rot="MR270"/>
 </instance>
 <instance part="BSK4" gate="A" x="223.52" y="121.92" smashed="yes" rot="MR270">
-<attribute name="NAME" x="234.315" y="120.65" size="1.778" layer="95" rot="MR90"/>
+<attribute name="NAME" x="239.395" y="120.65" size="1.778" layer="95" rot="MR90"/>
 <attribute name="VALUE" x="246.38" y="128.27" size="1.778" layer="96" rot="MR270"/>
 </instance>
@@
 </segment>
 </net>
-<net name="SCLTM" class="0">
+<net name="SCL-TM" class="0">
 <segment>
 <wire x1="43.18" y1="50.8" x2="33.02" y2="50.8" width="0.1524" layer="91"/>
@@
 <wire x1="25.4" y1="53.34" x2="25.4" y2="50.8" width="0.1524" layer="91"/>
 </segment>
-</net>
-<net name="SDATM" class="0">
+<segment>
+<pinref part="BSK1" gate="A" pin="10"/>
+<wire x1="236.22" y1="86.36" x2="236.22" y2="104.14" width="0.1524" layer="91"/>
+<label x="236.22" y="93.98" size="1.778" layer="95" rot="R90"/>
+</segment>
+</net>
+<net name="SDA-TM" class="0">
 <segment>
 <wire x1="43.18" y1="48.26" x2="33.02" y2="48.26" width="0.1524" layer="91"/>
@@
 <wire x1="25.4" y1="45.72" x2="25.4" y2="48.26" width="0.1524" layer="91"/>
 </segment>
+<segment>
+<pinref part="BSK1" gate="A" pin="12"/>
+<wire x1="241.3" y1="86.36" x2="241.3" y2="104.14" width="0.1524" layer="91"/>
+<label x="241.3" y="93.98" size="1.778" layer="95" rot="R90"/>
+</segment>
 </net>
 <net name="B1_KEM-" class="0">
@@
 </segment>
 </net>
-<net name="SCL" class="0">
-<segment>
-<pinref part="BSK1" gate="A" pin="10"/>
-<wire x1="236.22" y1="86.36" x2="236.22" y2="104.14" width="0.1524" layer="91"/>
-<label x="236.22" y="93.98" size="1.778" layer="95" rot="R90"/>
-</segment>
-</net>
-<net name="SDA" class="0">
-<segment>
-<pinref part="BSK1" gate="A" pin="12"/>
-<wire x1="241.3" y1="86.36" x2="241.3" y2="104.14" width="0.1524" layer="91"/>
-<label x="241.3" y="93.98" size="1.778" layer="95" rot="R90"/>
-</segment>
-</net>
 <net name="PL6-KVCC" class="0">
 <segment>
@@
 </segment>
 </net>
+<net name="SCL-INA" class="0">
+<segment>
+<pinref part="BSK2" gate="A" pin="9"/>
+<wire x1="233.68" y1="193.04" x2="233.68" y2="210.82" width="0.1524" layer="91"/>
+<label x="233.68" y="200.66" size="1.778" layer="95" rot="R90"/>
+</segment>
+<segment>
+<pinref part="BSK3" gate="A" pin="15"/>
+<wire x1="246.38" y1="160.02" x2="246.38" y2="177.8" width="0.1524" layer="91"/>
+<label x="246.38" y="167.64" size="1.778" layer="95" rot="R90"/>
+</segment>
+<segment>
+<pinref part="BSK4" gate="A" pin="9"/>
+<wire x1="233.68" y1="124.46" x2="233.68" y2="142.24" width="0.1524" layer="91"/>
+<label x="233.68" y="132.08" size="1.778" layer="95" rot="R90"/>
+</segment>
+</net>
+<net name="SDA-INA" class="0">
+<segment>
+<pinref part="BSK2" gate="A" pin="10"/>
+<wire x1="236.22" y1="193.04" x2="236.22" y2="210.82" width="0.1524" layer="91"/>
+<label x="236.22" y="200.66" size="1.778" layer="95" rot="R90"/>
+</segment>
+<segment>
+<pinref part="BSK3" gate="A" pin="16"/>
+<wire x1="248.92" y1="160.02" x2="248.92" y2="177.8" width="0.1524" layer="91"/>
+<label x="248.92" y="167.64" size="1.778" layer="95" rot="R90"/>
+</segment>
+<segment>
+<pinref part="BSK4" gate="A" pin="10"/>
+<wire x1="236.22" y1="124.46" x2="236.22" y2="142.24" width="0.1524" layer="91"/>
+<label x="236.22" y="132.08" size="1.778" layer="95" rot="R90"/>
+</segment>
+</net>

Commit message: Исправлена БСК1
Parts:
- BSK2, BSK4: device pinheadCS:PINHD-1X10 -> pinheadCS:PINHD-1X11
Connections:
- net 3V3: now also BSK2.8, BSK4.8
- net GND: now also BSK2.9, BSK4.9; no longer BSK2.8, BSK4.8
- net SCL-INA: now also BSK2.10, BSK4.10; no longer BSK2.9, BSK4.9
- net SDA-INA: now also BSK2.11, BSK4.11; no longer BSK2.10, BSK4.10
Changed lines of the file:
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@@
 <part name="U$6" library="CanCubeSat" deviceset="USB-C" device=""/>
 <part name="BSK3" library="pinheadCS" deviceset="PINHD-1X16" device=""/>
-<part name="BSK2" library="pinheadCS" deviceset="PINHD-1X10" device=""/>
-<part name="BSK4" library="pinheadCS" deviceset="PINHD-1X10" device=""/>
+<part name="BSK2" library="pinheadCS" deviceset="PINHD-1X11" device=""/>
+<part name="BSK4" library="pinheadCS" deviceset="PINHD-1X11" device=""/>
 <part name="U$18" library="CanCubeSat" deviceset="74HC595" device=""/>
 <part name="U$19" library="CanCubeSat" deviceset="74HC595" device=""/>
@@
 <attribute name="VALUE" x="248.92" y="163.83" size="1.778" layer="96" rot="MR270"/>
 </instance>
-<instance part="BSK2" gate="A" x="223.52" y="190.5" smashed="yes" rot="MR270">
-<attribute name="NAME" x="239.395" y="189.23" size="1.778" layer="95" rot="MR90"/>
-<attribute name="VALUE" x="236.22" y="196.85" size="1.778" layer="96" rot="MR270"/>
-</instance>
-<instance part="BSK4" gate="A" x="223.52" y="121.92" smashed="yes" rot="MR270">
-<attribute name="NAME" x="239.395" y="120.65" size="1.778" layer="95" rot="MR90"/>
-<attribute name="VALUE" x="246.38" y="128.27" size="1.778" layer="96" rot="MR270"/>
+<instance part="BSK2" gate="A" x="226.06" y="190.5" smashed="yes" rot="MR270">
+<attribute name="NAME" x="241.935" y="189.23" size="1.778" layer="95" rot="MR90"/>
+<attribute name="VALUE" x="238.76" y="196.85" size="1.778" layer="96" rot="MR270"/>
+</instance>
+<instance part="BSK4" gate="A" x="226.06" y="121.92" smashed="yes" rot="MR270">
+<attribute name="NAME" x="241.935" y="120.65" size="1.778" layer="95" rot="MR90"/>
+<attribute name="VALUE" x="248.92" y="128.27" size="1.778" layer="96" rot="MR270"/>
 </instance>
 <instance part="U$18" gate="G$1" x="119.38" y="266.7" smashed="yes"/>
@@
 </segment>
 <segment>
-<wire x1="231.14" y1="124.46" x2="231.14" y2="142.24" width="0.1524" layer="91"/>
-<label x="231.14" y="132.08" size="1.778" layer="95" rot="R90"/>
-<pinref part="BSK4" gate="A" pin="8"/>
-</segment>
-<segment>
 <pinref part="BSK3" gate="A" pin="9"/>
 <wire x1="231.14" y1="160.02" x2="231.14" y2="177.8" width="0.1524" layer="91"/>
@@
 </segment>
 <segment>
-<wire x1="231.14" y1="193.04" x2="231.14" y2="210.82" width="0.1524" layer="91"/>
-<label x="231.14" y="200.66" size="1.778" layer="95" rot="R90"/>
-<pinref part="BSK2" gate="A" pin="8"/>
+<wire x1="233.68" y1="193.04" x2="233.68" y2="210.82" width="0.1524" layer="91"/>
+<label x="233.68" y="200.66" size="1.778" layer="95" rot="R90"/>
+<pinref part="BSK2" gate="A" pin="9"/>
+</segment>
+<segment>
+<wire x1="233.68" y1="124.46" x2="233.68" y2="142.24" width="0.1524" layer="91"/>
+<label x="233.68" y="132.08" size="1.778" layer="95" rot="R90"/>
+<pinref part="BSK4" gate="A" pin="9"/>
 </segment>
 </net>
@@
 <label x="228.6" y="167.64" size="1.778" layer="95" rot="R90"/>
 </segment>
+<segment>
+<pinref part="BSK2" gate="A" pin="8"/>
+<wire x1="231.14" y1="193.04" x2="231.14" y2="210.82" width="0.1524" layer="91"/>
+<label x="231.14" y="200.66" size="1.778" layer="95" rot="R90"/>
+</segment>
+<segment>
+<pinref part="BSK4" gate="A" pin="8"/>
+<wire x1="231.14" y1="124.46" x2="231.14" y2="142.24" width="0.1524" layer="91"/>
+<label x="231.14" y="132.08" size="1.778" layer="95" rot="R90"/>
+</segment>
 </net>
 <net name="PL6-KVCC" class="0">
@@
 <net name="SCL-INA" class="0">
 <segment>
-<pinref part="BSK2" gate="A" pin="9"/>
-<wire x1="233.68" y1="193.04" x2="233.68" y2="210.82" width="0.1524" layer="91"/>
-<label x="233.68" y="200.66" size="1.778" layer="95" rot="R90"/>
-</segment>
-<segment>
 <pinref part="BSK3" gate="A" pin="15"/>
 <wire x1="246.38" y1="160.02" x2="246.38" y2="177.8" width="0.1524" layer="91"/>
@@
 </segment>
 <segment>
-<pinref part="BSK4" gate="A" pin="9"/>
-<wire x1="233.68" y1="124.46" x2="233.68" y2="142.24" width="0.1524" layer="91"/>
-<label x="233.68" y="132.08" size="1.778" layer="95" rot="R90"/>
-</segment>
-</net>
-<net name="SDA-INA" class="0">
-<segment>
-<pinref part="BSK2" gate="A" pin="10"/>
 <wire x1="236.22" y1="193.04" x2="236.22" y2="210.82" width="0.1524" layer="91"/>
 <label x="236.22" y="200.66" size="1.778" layer="95" rot="R90"/>
-</segment>
+<pinref part="BSK2" gate="A" pin="10"/>
+</segment>
+<segment>
+<wire x1="236.22" y1="124.46" x2="236.22" y2="142.24" width="0.1524" layer="91"/>
+<label x="236.22" y="132.08" size="1.778" layer="95" rot="R90"/>
+<pinref part="BSK4" gate="A" pin="10"/>
+</segment>
+</net>
+<net name="SDA-INA" class="0">
 <segment>
 <pinref part="BSK3" gate="A" pin="16"/>
@@
 </segment>
 <segment>
-<pinref part="BSK4" gate="A" pin="10"/>
-<wire x1="236.22" y1="124.46" x2="236.22" y2="142.24" width="0.1524" layer="91"/>
-<label x="236.22" y="132.08" size="1.778" layer="95" rot="R90"/>
-</segment>
-</net>
+<wire x1="238.76" y1="193.04" x2="238.76" y2="210.82" width="0.1524" layer="91"/>
+<label x="238.76" y="200.66" size="1.778" layer="95" rot="R90"/>
+<pinref part="BSK2" gate="A" pin="11"/>
+</segment>
+<segment>
+<wire x1="238.76" y1="124.46" x2="238.76" y2="142.24" width="0.1524" layer="91"/>
+<label x="238.76" y="132.08" size="1.778" layer="95" rot="R90"/>
+<pinref part="BSK4" gate="A" pin="11"/>
+</segment>
+</net>

Commit message: Схема БКУ
Parts:
- removed JP1: (no value), pinheadCS:PINHD-1X2
- removed JTAG: (no value), pinheadCS:PINHD-1X6
- removed LED-B#2, LED1: (no value), led:LEDCHIPLED_0603
- removed R27: 2k, resistor:R-US_R0603
- removed R29: 10k, resistor:R-US_R0603
- removed RADIO: RADIO, CanCubeSat:RADIO
- removed U$6: USB-C, CanCubeSat:USB-C
- removed U$7: EM_HEAT, CanCubeSat:EM_HEAT
- removed U$8: L293DD, CanCubeSat:L293DD
- added LED-B, LED-G, LED_B1: (no value), led:LEDCHIPLED_0603
- added R1: 5k1, resistor:R-US_R0603
- added R14, R16, R4: 1M, resistor:R-US_R0603
- added R15: 0.05A, rcl:R-EU_R1210
- added R17, R31, R32: 100R, resistor:R-US_R0603
- added R19, R33: 0.5A, rcl:R-EU_R1210
- added R3, R7: 2k, resistor:R-US_R0603
- added U$1: E22-400M30S, CanCubeSat:E22-400M30S
- added U$2: 74HC595, CanCubeSat:74HC595
- added U$21: FFC-CONNECT68611, CanCubeSat:FFC-CONNECT68611
- added U$23, U$3, U$4: SI2302CDS, CanCubeSat:SI2302CDS
- added U$24: EM_HEAT, CanCubeSat:EM_HEAT
- BSK3: device pinheadCS:PINHD-1X16 -> pinheadCS:PINHD-1X14
Connections:
- removed net AUX: RADIO.AUX, U$13.SVP
- removed net B1_KEM+: U$18.Q2, U$8.IN1
- removed net B1_KEM-: U$18.Q3, U$8.IN2
- removed net B1_KHEAT: U$18.Q1, U$8.IN4
- removed net B2A_KEM+: U$19.Q2
- removed net B2A_KEM-: U$19.Q3
- removed net B2A_KHEAT: U$19.Q1
- removed net B2A_KVCC: U$19.Q0
- removed net B2_KEM+: U$19.Q6
- removed net B2_KEM-: U$19.Q7
- removed net B2_KHEAT: U$19.Q5
- removed net B2_KVCC: U$19.Q4
- removed net B3_KEM+: U$20.Q6
- removed net B3_KEM-: U$20.Q7
- removed net B3_KHEAT: U$20.Q5
- removed net B3_KVCC: U$20.Q4
- removed net B4_KEM+: U$18.Q6
- removed net B4_KEM-: U$18.Q7
- removed net B4_KHEAT: U$18.Q5
- removed net B4_KVCC: U$18.Q4
- removed net B5-CMD: BSK3.13
- removed net B5-KVCC: BSK3.11
- removed net B5-ROZE: BSK3.12
- removed net B5_KEM+: U$20.Q2
- removed net B5_KEM-: U$20.Q3
- removed net B5_KHEAT: U$20.Q1
- removed net B5_KVCC: U$20.Q0
- removed net DS: U$13.IO25, U$18.DS
- removed net I2CINT: U$13.IO18
- removed net M1: R29.1, RADIO.M1, U$13.IO34, U$6.NC/M1
- removed net N$51: LED-B#2.C, R27.1
- removed net PL_KVCC: U$13.IO33
- removed net RX-ES: U$13.IO22
- removed net SCL-INA: BSK2.10, BSK3.15, BSK4.10
- removed net SDA-INA: BSK2.11, BSK3.16, BSK4.11
- removed net SHCP: U$13.IO27, U$18.SHCP, U$19.SHCP, U$20.SHCP
- removed net STCP: U$13.IO26, U$18.STCP, U$19.STCP, U$20.STCP
- removed net TX-ES: U$13.IO23
- removed net VDD: C12.2, C3.1, C33.1, C6.1, JTAG.2, LED1.A, R10.1, R11.1, R13.2, R18.1, R21.1, R22.1, R23.1, R24.1, R5.2, R6.2, SD.VDD, U$10.VON1, U$11.2, U$13.3V3, U$18.MR, U$18.VCC, U$19.MR, U$19.VCC, U$20.MR, U$20.VCC, U$6.NC/3V3
- new net 3: R3.2, U$23.D, U$24.GND
- new net BKU-KHEAT: U$2.Q0
- new net BUSY: U$1.BUSY, U$13.IO35
- new net CS-RA: U$1.NSS, U$13.IO21
- new net CS-SR: U$13.IO19, U$18.STCP, U$19.STCP, U$2.STCP, U$20.STCP
- new net DIO1: U$1.DIO1, U$13.IO32
- new net GND-OUT: BSK1.11, BSK1.9, BSK2.9, BSK3.14, BSK3.9, BSK4.9, R33.2, U$21.11, U$21.5, U$21.7, U$21.9
- new net GND-RADIO: R19.2, U$4.D
- new net GND-SD: R15.1, U$3.D
- new net MISO: U$1.MISO, U$13.SVP
- new net MOSI: U$1.MOSI, U$13.IO23, U$18.DS
- new net N$1: U$2.DS, U$20.Q7S
- new net N$11: R14.1, R31.2, U$3.G
- new net N$2: LED_B1.C, R3.1
- new net N$36: R32.1, R4.1, U$23.G
- new net N$5: R15.2, SD.VSS
- new net N$6: R16.1, R17.2, U$4.G
- new net NRST: R1.1, U$1.NRST, U$13.IO33
- new net RADIO: R17.1, U$2.Q2
- new net RX-EN: U$1.RXEN, U$13.IO26
- new net SCK: U$1.SCK, U$13.IO22, U$18.SHCP, U$19.SHCP, U$2.SHCP, U$20.SHCP
- new net SD: R31.1, U$2.Q1
- new net TX-EN: U$1.TXEN, U$13.IO25
- net 1W: now also U$13.IO27; no longer U$13.IO21
- net 3V3: now also C12.2, C3.1, C33.1, C6.1, LED-B.A, LED-G.A, R1.2, R10.1, R11.1, R13.2, R18.1, R21.1, R22.1, R23.1, R24.1, R5.2, R6.2, SD.VDD, U$10.VON1, U$11.2, U$13.3V3, U$18.MR, U$18.VCC, U$19.MR, U$19.VCC, U$2.MR, U$2.VCC, U$20.MR, U$20.VCC, U$21.3
- net 5V: now also LED_B1.A, U$1.VCC, U$24.5V; no longer RADIO.VCC, U$8.EN1, U$8.EN2, U$8.VS, U$8.VSS
- net B1-CMD: now also U$18.Q3
- net B1-KHEAT: now also R32.2, U$18.Q0
- net B1-KVCC: now also U$18.Q1
- net B1-ROZE: now also U$18.Q2
- net B2-CMD: now also U$18.Q7
- net B2-KHEAT: now also U$18.Q4
- net B2-KVCC: now also U$18.Q5
- net B2-ROZE: now also U$18.Q6
- net B3-CMD: now also U$19.Q3
- net B3-KHEAT: now also U$19.Q0
- net B3-KVCC: now also U$19.Q1
- net B3-ROZE: now also U$19.Q2
- net B4-CMD: now also U$19.Q7
- net B4-KHEAT: now also U$19.Q4
- net B4-KVCC: now also U$19.Q5
- net B4-ROZE: now also U$19.Q6
- net B5-KHEAT: now also U$20.Q0
- net BUS+: now also U$21.1, U$21.2; no longer U$6.3V3/BUS
- net DAT0: now also U$21.14; no longer JP1.2
- net EN: now also U$21.4; no longer U$6.NRST/EN
- net GND: now also R14.2, R16.2, R19.1, R33.1, R4.2, R7.1, U$1.GND, U$2.GND, U$2.OE, U$23.S, U$3.S, U$4.S; no longer BSK1.11, BSK1.9, BSK2.9, BSK3.9, BSK4.9, JP1.1, JTAG.1, R27.2, R29.2, RADIO.GND, RADIO.M0, SD.VSS, U$6.GND, U$7.GND, U$8.GND, U$8.HEAT
- net IO0-E: now also U$21.13; no longer U$6.NC/GPIO
- net MTCK: no longer JTAG.5
- net MTDI: no longer JTAG.6
- net MTDO: no longer JTAG.3
- net MTMS: no longer JTAG.4
- net N$3: now also LED-G.C, R7.2; no longer LED-B#2.A, U$7.5V, U$8.OUT4
- net N$4: now also LED-B.C; no longer LED1.C
- net PL1-KVCC: now also U$20.Q2
- net PL2-KVCC: now also U$20.Q3
- net PL3-KVCC: now also U$20.Q4
- net PL4-KVCC: now also U$20.Q5
- net PL5-KVCC: now also U$20.Q6
- net PL6-KVCC: now also U$20.Q7
- net RX-E: now also U$21.6; no longer U$6.SWD/RXD
- net RX-R: now also U$21.10; no longer RADIO.TXD, U$13.IO35, U$6.RX0
- net SCL-TM: now also BSK2.10, BSK3.12, BSK4.10
- net SDA-TM: now also BSK2.11, BSK3.13, BSK4.11
- net SINS-KVCC: now also BSK3.11, U$20.Q1; no longer BSK3.14
- net TIME: now also U$13.IO18; no longer U$13.IO19
- net TX-E: now also U$21.8; no longer U$6.SWC/TXD
- net TX-R: now also U$21.12; no longer RADIO.RXD, U$13.IO32, U$6.TX0
Other:
- moved on the sheet: BSK1, BSK2, BSK4, C1, C12, C14, C15, C16, C17, C3, C33, C4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
