File: schematics/board/Debug.sch (EAGLE design)
At the start: 29 parts, among them T1 2n7002, T2 2n7002

Commit message: Отладочная плата Debug
Parts:
- removed JP1: (no value), pinhead:PINHD-1X2
- removed RADIO: (no value), pinhead:PINHD-1X4
- removed U$1, U$2: USB-C, CanCubeSat:USB-C
- added DAT0: (no value), switch-omron:10-XX
- added POWER: (no value), pinhead:PINHD-1X3
- added U$12, U$21: FFC-CONNECT68611, CanCubeSat:FFC-CONNECT68611
Connections:
- removed net M1: JP1.2, RADIO.4, U$1.NC/M1
- removed net RX: DEBUG_STM32.3, U$2.RX0
- removed net RX1: RADIO.3, U$1.RX0
- removed net RXD: DOWNLOAD_ESP32.3, U$1.SWD/RXD
- removed net TX: DEBUG_STM32.2, U$2.TX0
- removed net TX1: RADIO.2, U$1.TX0
- removed net TXD: DOWNLOAD_ESP32.2, U$1.SWC/TXD
- new net 5V: POWER.1, U$21.11
- new net DAT0: DAT0.P, DAT0.P1, U$21.10
- new net RX-E: DOWNLOAD_ESP32.3, U$21.6
- new net RX-S: DEBUG_STM32.3, U$12.4
- new net TX-E: DOWNLOAD_ESP32.2, U$21.8
- new net TX-S: DEBUG_STM32.2, U$12.6
- net 3V3: now also POWER.2, U$21.3; no longer JP5.2, JP7.2, LED1.A, U$2.3V3/BUS
- net 3V3-S: now also JP5.2, JP7.2, LED1.A, U$12.1, U$12.2; no longer JP1.1, U$1.NC/3V3
- net BUS: now also U$21.1, U$21.2; no longer U$1.3V3/BUS
- net EN: now also U$21.4; no longer U$1.NRST/EN
- net GND: now also DAT0.S, DAT0.S1, POWER.3, U$12.3, U$12.5, U$12.7, U$12.9, U$21.5, U$21.7; no longer RADIO.1, U$1.GND, U$2.GND
- net IO0: now also U$21.9; no longer U$1.NC/GPIO
- net NRST: now also U$12.11; no longer U$2.NRST/EN
- net SWC: now also U$12.10; no longer U$2.SWC/TXD
- net SWD: now also U$12.8; no longer U$2.SWD/RXD
Other:
- moved on the sheet: DOWNLOAD_ESP32, JP5, JP6, JP7, JP8, LED1, LED2, R3, R4

Commit message: Добавлены герберы плат BKU и Debug
Parts:
- U$12, U$21: value FFC-CONNECT68611 -> FFC-CONNECT; device CanCubeSat:FFC-CONNECT68611 -> CanCubeSat:FFC-CONNECT
Connections:
- net RX-S: now also DEBUG_STM32.2; no longer DEBUG_STM32.3
- net SWC: now also DOWNLOAD_STM32.3; no longer DOWNLOAD_STM32.2
- net SWD: now also DOWNLOAD_STM32.2; no longer DOWNLOAD_STM32.3
- net TX-S: now also DEBUG_STM32.3; no longer DEBUG_STM32.2
Other:
- moved on the sheet: U$12, U$21
Changed lines of the file:
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@@
 <part name="LED2" library="led" library_urn="urn:adsk.eagle:library:259" deviceset="LED" device="CHIPLED_0603" package3d_urn="urn:adsk.eagle:package:15822/2"/>
 <part name="LED1" library="led" library_urn="urn:adsk.eagle:library:259" deviceset="LED" device="CHIPLED_0603" package3d_urn="urn:adsk.eagle:package:15822/2"/>
-<part name="U$21" library="CanCubeSat" deviceset="FFC-CONNECT" device="68611"/>
-<part name="U$12" library="CanCubeSat" deviceset="FFC-CONNECT" device="68611"/>
+<part name="U$21" library="CanCubeSat" deviceset="FFC-CONNECT" device="" value="FFC-CONNECT"/>
+<part name="U$12" library="CanCubeSat" deviceset="FFC-CONNECT" device="" value="FFC-CONNECT"/>
 <part name="POWER" library="pinhead" library_urn="urn:adsk.eagle:library:325" deviceset="PINHD-1X3" device="" package3d_urn="urn:adsk.eagle:package:22458/2"/>
 <part name="DAT0" library="switch-omron" library_urn="urn:adsk.eagle:library:377" deviceset="10-XX" device="" package3d_urn="urn:adsk.eagle:package:27496/1"/>
@@
 <net name="SWC" class="0">
 <segment>
+<wire x1="147.32" y1="116.84" x2="147.32" y2="96.52" width="0.1524" layer="91"/>
+<label x="147.32" y="96.52" size="1.778" layer="95" rot="R90"/>
+<pinref part="U$12" gate="G$1" pin="10"/>
+</segment>
+<segment>
+<pinref part="DOWNLOAD_STM32" gate="A" pin="3"/>
+<wire x1="149.86" y1="35.56" x2="149.86" y2="22.86" width="0.1524" layer="91"/>
+<label x="149.86" y="27.94" size="1.778" layer="95" rot="R90"/>
+</segment>
+</net>
+<net name="SWD" class="0">
+<segment>
+<wire x1="142.24" y1="116.84" x2="142.24" y2="96.52" width="0.1524" layer="91"/>
+<label x="142.24" y="96.52" size="1.778" layer="95" rot="R90"/>
+<pinref part="U$12" gate="G$1" pin="8"/>
+</segment>
+<segment>
 <pinref part="DOWNLOAD_STM32" gate="A" pin="2"/>
 <wire x1="152.4" y1="35.56" x2="152.4" y2="22.86" width="0.1524" layer="91"/>
 <label x="152.4" y="27.94" size="1.778" layer="95" rot="R90"/>
-</segment>
-<segment>
-<wire x1="147.32" y1="116.84" x2="147.32" y2="96.52" width="0.1524" layer="91"/>
-<label x="147.32" y="96.52" size="1.778" layer="95" rot="R90"/>
-<pinref part="U$12" gate="G$1" pin="10"/>
-</segment>
-</net>
-<net name="SWD" class="0">
-<segment>
-<pinref part="DOWNLOAD_STM32" gate="A" pin="3"/>
-<wire x1="149.86" y1="35.56" x2="149.86" y2="22.86" width="0.1524" layer="91"/>
-<label x="149.86" y="27.94" size="1.778" layer="95" rot="R90"/>
-</segment>
-<segment>
-<wire x1="142.24" y1="116.84" x2="142.24" y2="96.52" width="0.1524" layer="91"/>
-<label x="142.24" y="96.52" size="1.778" layer="95" rot="R90"/>
-<pinref part="U$12" gate="G$1" pin="8"/>
 </segment>
 </net>
@@
 </segment>
 <segment>
+<pinref part="DEBUG_STM32" gate="A" pin="2"/>
+<wire x1="129.54" y1="22.86" x2="129.54" y2="35.56" width="0.1524" layer="91"/>
+<label x="129.54" y="27.94" size="1.778" layer="95" rot="R90"/>
+</segment>
+</net>
+<net name="TX-S" class="0">
+<segment>
+<wire x1="137.16" y1="116.84" x2="137.16" y2="96.52" width="0.1524" layer="91"/>
+<label x="137.16" y="96.52" size="1.778" layer="95" rot="R90"/>
+<pinref part="U$12" gate="G$1" pin="6"/>
+</segment>
+<segment>
 <pinref part="DEBUG_STM32" gate="A" pin="3"/>
 <wire x1="127" y1="22.86" x2="127" y2="35.56" width="0.1524" layer="91"/>
@@
 </segment>
 </net>
-<net name="TX-S" class="0">
-<segment>
-<wire x1="137.16" y1="116.84" x2="137.16" y2="96.52" width="0.1524" layer="91"/>
-<label x="137.16" y="96.52" size="1.778" layer="95" rot="R90"/>
-<pinref part="U$12" gate="G$1" pin="6"/>
-</segment>
-<segment>
-<pinref part="DEBUG_STM32" gate="A" pin="2"/>
-<wire x1="129.54" y1="22.86" x2="129.54" y2="35.56" width="0.1524" layer="91"/>
-<label x="129.54" y="27.94" size="1.778" layer="95" rot="R90"/>
-</segment>
-</net>
