File: schematics/board/Debug.brd (EAGLE design)
At the start: 84 x 54 mm, 29 parts, among them T1 2n7002, T2 2n7002

Commit message: Отладочная плата Debug
Parts:
- removed JP1: (no value), pinhead:1X02
- removed RADIO: (no value), pinhead:1X04
- removed U$1, U$2: USB-C, CanCubeSat:USB-C
- added DAT0: (no value), switch-omron:B3F-10XX
- added POWER: (no value), pinhead:1X03
- added U$12, U$21: FFC-CONNECT68611, CanCubeSat:68611
- moved R1 4.24 mm to (16.3, 25.6)
- moved R2 4.24 mm to (16.4, 37.8)
- moved T2 4.24 mm to (18.6, 31.6)
- moved T1 4.24 mm to (14.0, 31.6)
- moved EN 2.62 mm to (8.90, 25.7)
- moved ENABLE 2.62 mm to (8.90, 34.7)
- moved C1 1.50 mm to (41.5, 9.00)
- moved C2 1.50 mm to (41.5, 13.0)
- moved C3 1.50 mm to (41.5, 17.0)
- moved GPIO0 1.50 mm to (41.5, 35.0)
- moved IO0 1.50 mm to (41.5, 26.0)
Connections:
- removed net M1: JP1.2, RADIO.4, U$1.NC/M1
- removed net RX: DEBUG_STM32.3, U$2.RX0
- removed net RX1: RADIO.3, U$1.RX0
- removed net RXD: DOWNLOAD_ESP32.3, U$1.SWD/RXD
- removed net TX: DEBUG_STM32.2, U$2.TX0
- removed net TX1: RADIO.2, U$1.TX0
- removed net TXD: DOWNLOAD_ESP32.2, U$1.SWC/TXD
- new net 5V: POWER.1, U$21.P$11
- new net DAT0: DAT0.3, DAT0.4, U$21.P$10
- new net RX-E: DOWNLOAD_ESP32.3, U$21.P$6
- new net RX-S: DEBUG_STM32.3, U$12.P$4
- new net TX-E: DOWNLOAD_ESP32.2, U$21.P$8
- new net TX-S: DEBUG_STM32.2, U$12.P$6
- net 3V3: now also POWER.2, U$21.P$3; no longer JP5.2, JP7.2, LED1.A, U$2.3V3/BUS0, U$2.3V3/BUS1
- net 3V3-S: now also JP5.2, JP7.2, LED1.A, U$12.P$1, U$12.P$2; no longer JP1.1, U$1.NC/3V3
- net BUS: now also U$21.P$1, U$21.P$2; no longer U$1.3V3/BUS0, U$1.3V3/BUS1
- net EN: now also U$21.P$4; no longer U$1.NRST/EN
- net GND: now also DAT0.1, DAT0.2, POWER.3, U$12.P$3, U$12.P$5, U$12.P$7, U$12.P$9, U$21.P$5, U$21.P$7; no longer RADIO.1, U$1.GND0, U$1.GND1, U$2.GND0, U$2.GND1
- net IO0: now also U$21.P$9; no longer U$1.NC/GPIO
- net NRST: now also U$12.P$11; no longer U$2.NRST/EN
- net SWC: now also U$12.P$10; no longer U$2.SWC/TXD
- net SWD: now also U$12.P$8; no longer U$2.SWD/RXD
Routing:
- net RX1: track 56.3 -> 0.00 mm
- net 5V: track 0.00 -> 53.3 mm
- net M1: track 46.4 -> 0.00 mm, vias 1 -> 0
- net TX-E: track 0.00 -> 43.9 mm
- net RX-E: track 0.00 -> 41.9 mm
- net TX1: track 40.8 -> 0.00 mm
- net TX-S: track 0.00 -> 39.4 mm
- net RX-S: track 0.00 -> 39.1 mm
- net RX: track 38.9 -> 0.00 mm, vias 1 -> 0
- net TX: track 38.5 -> 0.00 mm
- net TXD: track 36.1 -> 0.00 mm
- net RXD: track 35.7 -> 0.00 mm
- net DAT0: track 0.00 -> 35.1 mm
- net 3V3-S: track 21.1 -> 39.1 mm
- net 3V3: track 48.0 -> 63.8 mm, vias 1 -> 2
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Other:
- outline, holes or cut-outs redrawn
- board text added: "3V3-E"
- board text added: "5V"
- board text added: "ESP32 DAT0 (LOW)"
- board text added: "to ESP32"
- board text added: "to STM32"
- board text removed: "M1"
- board text removed: "RADIO"
- board text removed: "RADIO M1 (HIGH)"
- board text removed: "RX1"
- board text removed: "TX1"
- board text removed: "USB-C to ESP32"
- board text removed: "USB-C to STM32"

Commit message: Добавлены герберы плат BKU и Debug
Parts:
- U$12, U$21: value FFC-CONNECT68611 -> FFC-CONNECT; device CanCubeSat:68611 -> CanCubeSat:SLW15S
- moved U$12 0.40 mm to (55.3, 48.0), turned to 0 degrees
- moved U$21 0.40 mm to (28.8, 48.0), turned to 0 degrees
Connections:
- net 3V3: now also U$21.3; no longer U$21.P$3
- net 3V3-S: now also U$12.1, U$12.2; no longer U$12.P$1, U$12.P$2
- net 5V: now also U$21.11; no longer U$21.P$11
- net BUS: now also U$21.1, U$21.2; no longer U$21.P$1, U$21.P$2
- net DAT0: now also U$21.10; no longer U$21.P$10
- net EN: now also U$21.4; no longer U$21.P$4
- net GND: now also U$12.3, U$12.5, U$12.7, U$12.9, U$21.5, U$21.7; no longer U$12.P$3, U$12.P$5, U$12.P$7, U$12.P$9, U$21.P$5, U$21.P$7
- net IO0: now also U$21.9; no longer U$21.P$9
- net NRST: now also U$12.11; no longer U$12.P$11
- net RX-E: now also U$21.6; no longer U$21.P$6
- net RX-S: now also DEBUG_STM32.2, U$12.4; no longer DEBUG_STM32.3, U$12.P$4
- net SWC: now also DOWNLOAD_STM32.3, U$12.10; no longer DOWNLOAD_STM32.2, U$12.P$10
- net SWD: now also DOWNLOAD_STM32.2, U$12.8; no longer DOWNLOAD_STM32.3, U$12.P$8
- net TX-E: now also U$21.8; no longer U$21.P$8
- net TX-S: now also DEBUG_STM32.3, U$12.6; no longer DEBUG_STM32.2, U$12.P$6
Routing:
- net TX-E: track 43.9 -> 71.5 mm
- net SWD: track 42.2 -> 64.7 mm
- net TX-S: track 39.4 -> 57.1 mm
- net RX-E: track 41.9 -> 58.4 mm
- net SWC: track 43.4 -> 59.6 mm
- net DAT0: track 35.1 -> 49.2 mm, vias 0 -> 1
- net RX-S: track 39.1 -> 51.0 mm
- net GND: track 297.9 -> 290.2 mm, vias 1 -> 2
- net BUS: track 61.5 -> 56.3 mm
- net EN: track 87.0 -> 90.8 mm
- net IO0: track 73.1 -> 70.2 mm, vias 3 -> 1
- net 3V3: track 63.8 -> 61.6 mm, vias 2 -> 1
- net NRST: track 80.5 -> 78.3 mm
- net RTS: track 37.6 -> 35.9 mm
- net 3V3-S: track 39.1 -> 39.8 mm
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
Commit message: Исправлены герберы плат
Routing:
- net TX-E: track 71.5 -> 70.5 mm
Changed lines of the file:
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@@
 <contactref element="IO0" pad="4"/>
 <contactref element="C1" pad="2"/>
-<wire x1="42.75" y1="35" x2="42.77" y2="35" width="0.3" layer="16"/>
 <wire x1="42.375" y1="11.875" x2="42.375" y2="9" width="0.3" layer="1"/>
 <wire x1="42.375" y1="21.25" x2="42.375" y2="11.875" width="0.3" layer="16"/>
@@
 <wire x1="43.75" y1="29.25" x2="43.7606" y2="29.2512" width="0.3" layer="1"/>
 <wire x1="43.75" y1="22.75" x2="43.7606" y2="22.7488" width="0.3" layer="1"/>
-<wire x1="43.75" y1="29.375" x2="43.7606" y2="29.2512" width="0.3" layer="1"/>
 <via x="42.375" y="11.875" extent="1-16" drill="0.35"/>
 <contactref element="T2" pad="1"/>
@@
 <wire x1="7.86" y1="11.3" x2="5.95" y2="13.21" width="0.3" layer="16"/>
 <wire x1="25.6394" y1="29.6512" x2="25.6394" y2="23.1488" width="0.3" layer="1"/>
-<wire x1="54.3" y1="47" x2="54.3" y2="42.71" width="0.8" layer="1"/>
-<wire x1="54.3" y1="42.71" x2="52.45" y2="40.86" width="0.8" layer="1"/>
+<wire x1="54.3" y1="47" x2="54.3" y2="42.41" width="0.8" layer="1"/>
+<wire x1="54.3" y1="42.41" x2="52.75" y2="40.86" width="0.8" layer="1"/>
+<wire x1="52.75" y1="40.86" x2="52.45" y2="40.86" width="0.8" layer="1"/>
 <wire x1="52.45" y1="40.86" x2="49.615" y2="38.025" width="0.4" layer="1"/>
-<wire x1="40.23" y1="35" x2="40.23" y2="35.325" width="0.4" layer="1"/>
 <wire x1="25.6394" y1="23.1488" x2="20.92" y2="18.4294" width="0.5" layer="1"/>
 <wire x1="20.92" y1="18.4294" x2="20.92" y2="11.5" width="0.5" layer="1"/>
@@
 <wire x1="39.2" y1="49.7" x2="39.2" y2="41.7" width="0.3" layer="16"/>
 <contactref element="DOWNLOAD_ESP32" pad="2"/>
-<wire x1="23.46" y1="11.5" x2="23.46" y2="12.5" width="0.3" layer="1"/>
 <wire x1="34.9" y1="10.1" x2="32.3" y2="7.5" width="0.3" layer="16"/>
 <wire x1="32.3" y1="7.5" x2="25.6" y2="7.5" width="0.3" layer="16"/>
