File: schematics/board/RADIO.sch (EAGLE design)
At the start: 2 parts

Commit message: Готова плата RADIO и переделана плата AB
Parts:
- removed JP1: (no value), pinheadCS:PINHD-1X7
- removed RADIO: RADIO, CanCubeSat:RADIO
- added C1: 0.1uF, rcl:C-EUC0603
- added JP2: (no value), pinhead:PINHD-1X4
- added JP3: (no value), pinhead:PINHD-1X2
- added JP4: (no value), pinhead:PINHD-1X7
- added R1, R2, R3: 5k1, resistor:R-US_R0603
- added U$1: E22-400M30S, CanCubeSat:E22-400M30S
Connections:
- removed net AUX: JP1.3, RADIO.AUX
- removed net M1: JP1.6, RADIO.M1
- removed net RXD: JP1.5, RADIO.RXD
- removed net TXD: JP1.4, RADIO.TXD
- new net 3V3: JP4.1, R1.2
- new net BUSY: JP4.3, U$1.BUSY
- new net CS-RA: JP2.1, U$1.NSS
- new net DIO1: JP4.4, U$1.DIO1
- new net DIO2: JP4.5, U$1.DIO2
- new net MISO: JP2.4, U$1.MISO
- new net MOSI: JP2.3, U$1.MOSI
- new net NRST: JP4.2, R1.1, U$1.NRST
- new net RX-EN: JP4.7, R2.1, U$1.RXEN
- new net SCK: JP2.2, U$1.SCK
- new net TX-EN: JP4.6, R3.1, U$1.TXEN
- net 5V: now also C1.1, JP3.1, U$1.VCC; no longer JP1.2, RADIO.VCC
- net GND: now also C1.2, JP3.2, R2.2, R3.2, U$1.GND; no longer JP1.1, JP1.7, RADIO.GND, RADIO.M0
